File: AstroCam.kicad_pcb (KiCad board)
At the start: 2 copper layers, 114.3 x 61 mm, 113 parts, among them U1 AD9974, U10 LMR62014, U11 CXD3400N, U12 ICX825AQA, U3 LM25088, U4 TPS2420, U6 LM3674, U7 TPS56x200, U8 TPS56x200, U9 TPS56x200

Commit message: initial experimentation with size constraints
Parts:
- removed C60, C61: 47F/3Mohm, w_smd_cap:c_0603
- removed C62: 220nF/220Mohm, w_smd_cap:c_0603
- removed C63, C64, C66: 0.1u, w_smd_cap:c_0603
- removed C67: 2200pF, w_smd_cap:c_0603
- removed C68, C69: 0.1, w_smd_cap:c_0603
- removed C70, C72: 0.01, w_smd_cap:c_0603
- removed U4: TPS2420, w_smd_qfn:pvqfn-n16
- added C11: 1.0F/11mOhm, w_smd_cap:c_0603, F.Cu at (143.8, 162.8)
- added C13: 2.20uF/2.80Mohm, w_smd_cap:c_0603, F.Cu at (180.0, 130.2)
- added C18: 1.0F, w_smd_cap:c_0603, F.Cu at (165.0, 142.8)
- added C22: 10.0F/3.0mOhm, w_smd_cap:c_0603, F.Cu at (171.5, 130.2)
- added C24: 2.2F/4.9Mohm, w_smd_cap:c_0603, F.Cu at (180.0, 132.0)
- added C44: 3.3/20V, w_smd_cap:c_0805, F.Cu at (160.0, 150.0)
- added C5: 220nF, w_smd_cap:c_0603, F.Cu at (90.6, 138.0)
- added C6: 470pF, w_smd_cap:c_0603, F.Cu at (160.0, 167.2)
- added P1: CONN_01X02, w_pin_strip:pin_strip_2, F.Cu at (184.3, 148.4)
- added P2: CONN_01X08, w_smd_strip:bb02-hp08, B.Cu at (99.6, 163.9)
- added P3: CONN_02X12, w_smd_strip:bb02-hp24, F.Cu at (100.3, 149.4)
- added Q1: Q_NMOS_DGS, w_smd_trans:sot23, F.Cu at (94.8, 136.0)
- added U5: LM3674, w_smd_trans:sot23-5, F.Cu at (120.5, 138.0)
- C1, C9: value 0.1uF -> 56nF
- C10: value 0.1uF -> 10.0uF/9.0Mohm
- C12: value 0.1u -> 68pF
- C14: value 0.1uF -> 1.5nF
- C15, C26, C27, C8: value 0.1uF -> 100nF
- C16: value 0.1u -> 1.0F/20Mohm
- C17: value 0.1uF -> 15F; footprint w_smd_cap:c_0603 -> w_smd_cap:c_0805
- C19: value 0.1uF -> 1.0F
- C2: value 0.1uF -> 10.0F/9Mohm
- C20: value 0.1uF -> 4.7F/5.0mOhm
- C21, C23: value 0.1uF -> 10.0F/3.0mOhm
- C25: value 0.1uF -> 9.0pF
- C28: value 56nF -> 100nF
- C29: value 10.0F/9Mohm -> 270pF
- C3: value 0.1uF -> 4.7F/6Mohm
- C30: value 4.7F/6Mohm -> 4.7F/2Mohm
- C31: value 1.0uF -> 10F/9Mohm
- C32: value 220nF -> 47F/3Mohm
- C33: value 470pF -> 47F/3Mohm
- C34: value 22nF -> 47F/3Mohm
- C35: value 100nF -> 220nF/220Mohm
- C36: value 56nF -> 0.1u
- C37: value 10.0uF/9.0Mohm -> 0.1u
- C38: value 1.0F/11mOhm -> 1/35V; footprint w_smd_cap:c_0603 -> w_smd_cap:c_0805
- C39: value 68pF -> 0.1u
- C4: value 0.1uF -> 1.0uF
- C40: value 2.20uF/2.80Mohm -> 2200pF
- C41: value 1.5nF -> 0.1
- C42: value 100nF -> 0.1
- C43: value 1.0F/20Mohm -> 0.01
- C45: value 1.0F -> 0.01; footprint w_smd_cap:c_0603 -> w_smd_cap:c_0805
- C46: value 1.0F -> 3.3/20V; footprint w_smd_cap:c_0603 -> w_smd_cap:c_0805
- C47: value 4.7F/5.0mOhm -> 3.3/20V; footprint w_smd_cap:c_0603 -> w_smd_cap:c_0805
- C48, C49, C50: value 10.0F/3.0mOhm -> 0.1uF
- C51: value 2.2F/4.9Mohm -> 0.1uF
- C52: value 9.0pF -> 0.1uF
- C53, C54, C55: value 100nF -> 0.1uF
- C56: value 270pF -> 0.1uF
- C57: value 4.7F/2Mohm -> 4.7uF
- C58: value 10F/9Mohm -> 0.1u
- C59: value 47F/3Mohm -> 0.1u
- C7: value 0.1uF -> 22nF
- D1: footprint w_smd_diode:sod523 -> w_smd_diode:sod80c
- D2, D3: footprint w_smd_diode:sod323 -> w_smd_diode:sod80c
- D4: footprint w_pth_diodes:diode_do41 -> w_smd_diode:sod123
- L1: footprint w_smd_inductors:inductor_smd_0603 -> w_smd_inductors:inductor_smd_0805
- R1, R10, R11, R12, R13, R14, R15, R16, R17, R18, R19, R2, R20, R21, R22, R23, R24, R25, R26, R27, R28, R3, R4, R5, R6, R7, R8, R9: footprint w_smd_resistors:r_0603 -> w_smd_resistors:r_0805
- U1: value AD9974 -> LMZ10500; footprint w_smd_bga:tfbga100-std -> camera:llp-8
- U10: value LMR62014 -> CXD3400N; footprint w_smd_trans:sot23-5 -> w_smd_dil:tssop-20; moved to B.Cu
- U11: value CXD3400N -> ICX825AQA; footprint w_smd_dil:ssop-16 -> camera:ICX825; moved to B.Cu
- U12: value ICX825AQA -> ADDI7013; footprint camera:ICX825 -> camera:csp-bga-bc-76-3
- U3: value LM25088 -> TPS2420; footprint w_smd_dil:tssop-16 -> w_smd_qfn:pvqfn-n16
- U6: value LM3674 -> TPS56x200; footprint w_smd_trans:sot23-5 -> w_smd_trans:sot23-6
- U9: value TPS56x200 -> LMR62014; footprint w_smd_trans:sot23-6 -> w_smd_trans:sot23-5
- moved C21 144.5 mm to (101.5, 167.2)
- moved L8 143.3 mm to (193.2, 168.8)
- moved L2 140.2 mm to (193.2, 154.0)
- moved R2 139.0 mm to (160.0, 165.0)
- moved C10 136.5 mm to (165.0, 158.5)
- moved U6 133.0 mm to (101.5, 164.8)
- moved R9 132.3 mm to (144.0, 165.0)
- moved C57 124.9 mm to (165.0, 162.0)
- moved L6 124.7 mm to (155.2, 160.0)
- moved U3 123.9 mm to (139.8, 163.2)
- moved C19 122.1 mm to (169.8, 150.0)
- moved C29 122.0 mm to (151.2, 167.2)
- moved R17 121.6 mm to (148.0, 165.0)
- moved R23 121.4 mm to (162.2, 131.2)
- moved C50 121.4 mm to (160.0, 155.0)
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Connections:
- C1 pad 1: /power-supply/1V8 -> Net-(C1-Pad1)
- C1 pad 2: GND -> /camera/-7V
- C10 pad 1: /LDO_OUT_A -> /h-driver/3V3
- C10 pad 2: GND -> /camera/GND
- C12 pad 1: /power-supply/3V3 -> Net-(C12-Pad1)
- C12 pad 2: GND -> Net-(C12-Pad2)
- C14 pad 1: GND -> Net-(C14-Pad1)
- C14 pad 2: /power-supply/3V3 -> Net-(C12-Pad1)
- C15 pad 1: GND -> Net-(C15-Pad1)
- C15 pad 2: /power-supply/3V3 -> Net-(C15-Pad2)
- C16 pad 1: GND -> /power-supply/5V5
- C16 pad 2: /power-supply/3V3 -> /camera/-7V
- C17 pad 1: /LDO_OUT_B -> /camera/GND
- C17 pad 2: GND -> /camera/-7V
- C19 pad 1: /power-supply/3V3 -> Net-(C19-Pad1)
- C19 pad 2: GND -> /camera/-7V
- C2 pad 1: Net-(C2-Pad1) -> /power-supply/5V5
- C2 pad 2: GND -> /camera/GND
- C20 pad 1: /power-supply/3V3 -> /power-supply/5V5
- C20 pad 2: GND -> /camera/GND
- C21 pad 1: /power-supply/1V8 -> /power-supply/5V5
- C21 pad 2: GND -> /camera/GND
- C23 pad 1: Net-(C23-Pad1) -> /power-supply/5V5
- C23 pad 2: Net-(C23-Pad2) -> /camera/GND
- C25 pad 1: /power-supply/1V8 -> /power-supply/2V5
- C25 pad 2: GND -> Net-(C25-Pad2)
- C26 pad 1: Net-(C23-Pad1) -> Net-(C26-Pad1)
- C26 pad 2: GND -> Net-(C26-Pad2)
- C27 pad 1: Net-(C23-Pad2) -> Net-(C27-Pad1)
- C27 pad 2: GND -> Net-(C27-Pad2)
- C28 pad 2: /camera/-7V -> Net-(C28-Pad2)
- C29 pad 1: /power-supply/5V5 -> Net-(C29-Pad1)
- C29 pad 2: GND -> Net-(C29-Pad2)
- C3 pad 1: Net-(C3-Pad1) -> /power-supply/5V5
- C3 pad 2: GND -> /camera/GND
- C30 pad 1: /power-supply/5V5 -> Net-(C29-Pad2)
- C30 pad 2: GND -> /camera/GND
- C31 pad 1: /power-supply/V_BATT -> /power-supply/2V5
- C31 pad 2: GND -> /camera/GND
- C32 pad 1: /power-supply/5V5 -> /power-supply/1V2_1
- C32 pad 2: GND -> /camera/GND
- C33 pad 1: Net-(C33-Pad1) -> /power-supply/1V2_2
- C33 pad 2: GND -> /camera/GND
- C34 pad 1: Net-(C34-Pad1) -> /h-driver/1V8
- C34 pad 2: /camera/-7V -> /camera/GND
- C35 pad 1: Net-(C35-Pad1) -> /camera/12V
- C35 pad 2: /camera/-7V -> /camera/GND
- C36 pad 1: Net-(C36-Pad1) -> /camera/-7V
- C36 pad 2: /camera/-7V -> /camera/GND
- C37 pad 1: /power-supply/3V3 -> /camera/GND
- C37 pad 2: GND -> /camera/12V
- C38 pad 2: GND -> Net-(C38-Pad2)
- C39 pad 1: Net-(C39-Pad1) -> Net-(C38-Pad1)
- C39 pad 2: Net-(C39-Pad2) -> /camera/SUB
- C4 pad 1: Net-(C2-Pad1) -> /power-supply/V_BATT
- C4 pad 2: Net-(C3-Pad1) -> /camera/GND
- C40 pad 1: /power-supply/5V5 -> /camera/SUB
- C40 pad 2: GND -> /camera/GND
- C41 pad 2: Net-(C39-Pad1) -> /h-driver/RG1
- C42 pad 2: Net-(C42-Pad2) -> /h-driver/RG2
- C43 pad 1: /power-supply/5V5 -> /camera/GND
- C43 pad 2: /camera/-7V -> /camera/12V
- C45 pad 1: GND -> /camera/GND
- C45 pad 2: /camera/-7V -> /camera/12V
- C46 pad 1: Net-(C46-Pad1) -> /camera/12V
- C46 pad 2: /camera/-7V -> /camera/GND
- C47 pad 1: /power-supply/5V5 -> /camera/GND
- C47 pad 2: GND -> /camera/-7V
- C48 pad 1: /power-supply/5V5 -> /h-driver/3V3
- C48 pad 2: GND -> /camera/GND
- C49 pad 1: /power-supply/5V5 -> /h-driver/1V8
- C49 pad 2: GND -> /camera/GND
- C50 pad 1: /power-supply/5V5 -> /h-driver/3V3
- C50 pad 2: GND -> /camera/GND
- C51 pad 1: /power-supply/5V5 -> /h-driver/1V8
- C51 pad 2: GND -> /camera/GND
- C52 pad 1: /power-supply/2V5 -> /h-driver/3V3
- C52 pad 2: Net-(C52-Pad2) -> /camera/GND
- C53 pad 1: Net-(C53-Pad1) -> /h-driver/1V8
- C53 pad 2: Net-(C53-Pad2) -> /camera/GND
- C54 pad 1: Net-(C54-Pad1) -> /h-driver/3V3
- C54 pad 2: Net-(C54-Pad2) -> /camera/GND
- C55 pad 1: Net-(C55-Pad1) -> /camera/GND
- C55 pad 2: Net-(C55-Pad2) -> /h-driver/1V8
- C56 pad 1: Net-(C56-Pad1) -> /h-driver/3V3
- C56 pad 2: Net-(C56-Pad2) -> /camera/GND
- C57 pad 1: Net-(C56-Pad2) -> /h-driver/3V3
- C57 pad 2: GND -> /camera/GND
- C58 pad 1: /power-supply/2V5 -> /camera/CCD_OUT1
- C58 pad 2: GND -> Net-(C58-Pad2)
- C59 pad 1: /power-supply/1V2_1 -> /camera/CCD_OUT2
- C59 pad 2: GND -> Net-(C59-Pad2)
- C7 pad 1: /power-supply/3V3 -> Net-(C7-Pad1)
- C7 pad 2: GND -> /camera/-7V
- C8 pad 1: /power-supply/1V8 -> Net-(C8-Pad1)
- C8 pad 2: Net-(C8-Pad2) -> /camera/-7V
- C9 pad 1: /power-supply/3V3 -> Net-(C9-Pad1)
- C9 pad 2: GND -> /camera/-7V
- D1 pad 2: GND -> /camera/GND
- D2 pad 1: Net-(C42-Pad1) -> Net-(C15-Pad1)
- D3 pad 1: Net-(C56-Pad2) -> Net-(C29-Pad2)
- D4 pad 1: Net-(C65-Pad1) -> Net-(C38-Pad1)
- L1 pad 1: Net-(C42-Pad1) -> Net-(C15-Pad1)
- L1 pad 2: GND -> /camera/GND
- L3 pad 1: GND -> /camera/GND
- L3 pad 2: Net-(C46-Pad1) -> Net-(C19-Pad1)
- L6 pad 1: Net-(C53-Pad2) -> Net-(C26-Pad2)
- L7 pad 1: Net-(C54-Pad2) -> Net-(C27-Pad2)
- L8 pad 1: Net-(C55-Pad2) -> Net-(C28-Pad2)
- L8 pad 2: /power-supply/1V8 -> /h-driver/1V8
- L9 pad 1: Net-(C56-Pad2) -> Net-(C29-Pad2)
- R1 pad 2: Net-(C33-Pad1) -> Net-(C6-Pad1)
- R10 pad 2: GND -> /camera/GND
- R11 pad 1: Net-(C41-Pad1) -> Net-(C14-Pad1)
- R11 pad 2: Net-(C39-Pad2) -> Net-(C12-Pad2)
- R13 pad 2: GND -> /camera/GND
- R14 pad 1: GND -> /camera/GND
- R14 pad 2: Net-(C39-Pad1) -> Net-(C12-Pad1)
- R15 pad 1: Net-(C39-Pad1) -> Net-(C12-Pad1)
- R17 pad 1: Net-(C56-Pad1) -> Net-(C29-Pad1)
- R17 pad 2: GND -> /camera/GND
- R18 pad 1: Net-(C56-Pad2) -> Net-(C29-Pad2)
- R18 pad 2: Net-(C56-Pad1) -> Net-(C29-Pad1)
- R19 pad 1: Net-(C52-Pad2) -> Net-(C25-Pad2)
- R19 pad 2: GND -> /camera/GND
- R2 pad 1: Net-(C33-Pad1) -> Net-(C6-Pad1)
- R2 pad 2: GND -> /camera/GND
- R20 pad 2: Net-(C52-Pad2) -> Net-(C25-Pad2)
- R22 pad 2: GND -> /camera/GND
- R24 pad 2: GND -> /camera/GND
- R25 pad 1: /power-supply/1V8 -> /h-driver/1V8
- R26 pad 2: GND -> /camera/GND
- R27 pad 1: Net-(C65-Pad1) -> Net-(C38-Pad1)
- R27 pad 2: GND -> /camera/GND
- R28 pad 1: Net-(R28-Pad1) -> /camera/SUB
- R28 pad 2: GND -> /camera/GND
- R3 pad 1: Net-(C28-Pad1) -> Net-(C1-Pad1)
- R4 pad 2: Net-(C35-Pad1) -> Net-(C8-Pad1)
- R5 pad 2: Net-(C28-Pad1) -> Net-(C1-Pad1)
- R9 pad 2: GND -> /camera/GND
- U10 pad 1: GND -> /camera/5V0
- U10 pad 2: (no net) -> Net-(P2-Pad1)
- U10 pad 3: Net-(C56-Pad1) -> Net-(P2-Pad2)
- U10 pad 4: Net-(R16-Pad2) -> /camera/GND
- U10 pad 5: /power-supply/5V5 -> Net-(P2-Pad3)
- U11 pad 1: /camera/5V0 -> /camera/CCD_OUT2
- U11 pad 10: /camera/XV4 -> /camera/VT3
- U11 pad 11: GND -> /camera/VT4
- U11 pad 12: /camera/VT1 -> /camera/GND
- U11 pad 13: /camera/VT2 -> /camera/GND
- U11 pad 14: /camera/VT3 -> /camera/CCD_OUT1
- U11 pad 16: Net-(U11-Pad16) -> Net-(C41-Pad1)
- U11 pad 2: /camera/XSUB -> /camera/GND
- U11 pad 3: /camera/XV2 -> /camera/GND
- U11 pad 4: GND -> /camera/SUB
- U11 pad 5: /camera/XSGV2 -> /camera/GND
- U11 pad 6: /camera/XV3 -> /camera/GND
- U11 pad 7: GND -> /camera/-7V
- U11 pad 8: /camera/XSGV3 -> /camera/VT1
- U11 pad 9: /camera/XV1 -> /camera/VT2
- U3 pad 1: (no net) -> /power-supply/V_BATT
- U3 pad 10: (no net) -> /power-supply/5V5
- U3 pad 11: (no net) -> /power-supply/5V5
- U3 pad 12: (no net) -> /power-supply/5V5
- U3 pad 13: (no net) -> Net-(R13-Pad1)
- U3 pad 14: (no net) -> Net-(R8-Pad2)
- U3 pad 15: (no net) -> Net-(R6-Pad2)
- U3 pad 16: (no net) -> /camera/GND
- U3 pad 2: (no net) -> /power-supply/V_BATT
- U3 pad 3: (no net) -> /power-supply/V_BATT
- U3 pad 4: (no net) -> /power-supply/V_BATT
- U3 pad 5: (no net) -> /camera/GND
- U3 pad 6: (no net) -> /camera/GND
- U3 pad 7: (no net) -> Net-(R9-Pad1)
- U3 pad 8: (no net) -> Net-(R10-Pad1)
- U3 pad 9: (no net) -> Net-(C11-Pad1)
- U6 pad 1: /power-supply/5V5 -> /camera/GND
- U6 pad 2: GND -> Net-(C26-Pad2)
- U6 pad 4: Net-(C52-Pad2) -> Net-(R21-Pad2)
- U6 pad 5: Net-(L5-Pad1) -> /power-supply/5V5
- U7 pad 1: GND -> /camera/GND
- U7 pad 2: Net-(C53-Pad2) -> Net-(C27-Pad2)
- U7 pad 4: Net-(R21-Pad2) -> Net-(R23-Pad2)
- U7 pad 6: Net-(C53-Pad1) -> Net-(C27-Pad1)
- U8 pad 1: GND -> /camera/GND
- U8 pad 2: Net-(C54-Pad2) -> Net-(C28-Pad2)
- U8 pad 4: Net-(R23-Pad2) -> Net-(R25-Pad2)
- U8 pad 6: Net-(C54-Pad1) -> Net-(C28-Pad1)
- U9 pad 1: GND -> Net-(D3-Pad2)
- U9 pad 2: Net-(C55-Pad2) -> (no net)
- U9 pad 3: /power-supply/5V5 -> Net-(C29-Pad1)
- U9 pad 4: Net-(R25-Pad2) -> Net-(R16-Pad2)
Routing:
- net GND: track 16.9 -> 0.00 mm, vias 3 -> 0
- net /LDO_OUT_B: track 4.14 -> 0.00 mm
Other:
- board size 114.3 x 61 mm -> 115 x 40 mm
- rule trace_min: 0.1 -> 0.2
- rule via_min_drill: 0.1 -> 0.3
- rule via_min_size: 0.2 -> 0.4

Commit message: More work on schematic
Parts:
- removed L2: 2.0uH/0.024Ohm, w_smd_inductors:inductor_smd_0805
- removed P3: CONN_02X12, w_smd_strip:bb02-hp24
- C11, C25, C4: footprint w_smd_cap:c_0603 -> Capacitors_SMD:C_0805_HandSoldering
- C20, C31: footprint w_smd_cap:c_0603 -> Capacitors_SMD:C_0603_HandSoldering
- C39: value 0.1u -> 0.1uF
- C40: value 2200pF -> 2.2uF
- C49, C52, C53, C54, C55, C56, C57, C58, C59: moved to B.Cu
- D1: footprint w_smd_diode:sod80c -> Diodes_SMD:Diode-SMB_Handsoldering
- L5: footprint w_smd_inductors:inductor_smd_0805 -> camera:Inductor_SMD_2016
- P2: value CONN_01X08 -> CONN_01X24; footprint w_smd_strip:bb02-hp08 -> camera:FFC-24-0.5mm; moved to F.Cu
- R10, R13, R6, R8, R9: footprint w_smd_resistors:r_0805 -> Resistors_SMD:R_0805_HandSoldering
- R19, R20: footprint w_smd_resistors:r_0805 -> Resistors_SMD:R_0402
- U10: moved to F.Cu
- U3: footprint w_smd_qfn:pvqfn-n16 -> Housings_DFN_QFN:QFN-16-1EP_4x4mm_Pitch0.65mm
- moved L8 94.0 mm to (117.8, 112.8)
- moved C56 88.6 mm to (90.1, 112.9)
- moved C29 87.4 mm to (97.5, 98.3)
- moved C53 81.1 mm to (91.4, 115.2), turned to 270 degrees
- moved C57 81.0 mm to (99.4, 114.5), turned to 270 degrees
- moved C50 80.2 mm to (93.8, 109.8)
- moved C52 80.1 mm to (97.3, 112.2)
- moved C15 79.9 mm to (89.8, 130.3)
- moved C54 79.2 mm to (98.0, 114.5), turned to 270 degrees
- moved C30 78.2 mm to (107.0, 100.8)
- moved R18 77.2 mm to (113.0, 98.0)
- moved C6 76.7 mm to (92.8, 130.3)
- moved R17 74.7 mm to (110.2, 100.5)
- moved C10 74.3 mm to (124.8, 96.0)
- moved C55 73.4 mm to (96.4, 116.5), turned to 180 degrees
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Connections:
- C55 pad 1: /camera/GND -> /h-driver/1V8
- C55 pad 2: /h-driver/1V8 -> /camera/GND
- P2 pad 1: Net-(P2-Pad1) -> /h-driver/CLI
- P2 pad 2: Net-(P2-Pad2) -> /h-driver/GP01
- P2 pad 3: Net-(P2-Pad3) -> /h-driver/GP02
- P2 pad 4: Net-(P2-Pad4) -> /h-driver/GP03
- P2 pad 5: Net-(P2-Pad5) -> /h-driver/GP04
- P2 pad 6: Net-(P2-Pad6) -> /camera/GND
- P2 pad 7: Net-(P2-Pad7) -> /h-driver/SCK
- P2 pad 8: /camera/GND -> /h-driver/SDATA
- U10 pad 10: Net-(P2-Pad7) -> /camera/XV4
- U10 pad 12: /camera/VT1 -> /camera/VT4
- U10 pad 13: /camera/VT2 -> /camera/VT1
- U10 pad 17: /camera/VT4 -> /camera/VT2
- U10 pad 2: Net-(P2-Pad1) -> /camera/XSHT
- U10 pad 3: Net-(P2-Pad2) -> /camera/XV2
- U10 pad 5: Net-(P2-Pad3) -> /camera/XSGV2
- U10 pad 6: Net-(P2-Pad4) -> /camera/XV3
- U10 pad 8: Net-(P2-Pad5) -> /camera/XSGV3
- U10 pad 9: Net-(P2-Pad6) -> /camera/XV1
- U12 pad B1: Net-(P3-Pad23) -> /h-driver/CLI
- U12 pad C1: Net-(P3-Pad21) -> /h-driver/GP01
- U12 pad C2: Net-(P3-Pad3) -> /h-driver/SL
- U12 pad D1: Net-(P3-Pad19) -> /h-driver/GP02
- U12 pad D2: Net-(P3-Pad7) -> /h-driver/SCK
- U12 pad D6: (no net) -> /camera/GND
- U12 pad E2: Net-(P3-Pad5) -> /h-driver/SDATA
- U12 pad F1: Net-(P3-Pad17) -> /h-driver/GP03
- U12 pad F2: Net-(P3-Pad13) -> /h-driver/SYNC
- U12 pad G1: Net-(P3-Pad15) -> /h-driver/GP04
- U12 pad G2: Net-(P3-Pad9) -> /h-driver/HD
- U12 pad H2: Net-(P3-Pad11) -> /h-driver/VD
- U12 pad K1: Net-(P3-Pad24) -> /h-driver/A0+
- U12 pad K10: Net-(P3-Pad2) -> /h-driver/B1-
- U12 pad K2: Net-(P3-Pad22) -> /h-driver/A0-
- U12 pad K3: Net-(P3-Pad20) -> /h-driver/A1+
- U12 pad K4: Net-(P3-Pad18) -> /h-driver/A1-
- U12 pad K5: Net-(P3-Pad14) -> /h-driver/TCLK+
- U12 pad K6: Net-(P3-Pad12) -> /h-driver/TCLK-
- U12 pad K7: Net-(P3-Pad8) -> /h-driver/B0+
- U12 pad K8: Net-(P3-Pad6) -> /h-driver/B0-
- U12 pad K9: Net-(P3-Pad4) -> /h-driver/B1+
Routing:
- net /camera/GND: track 0.00 -> 101.7 mm, vias 0 -> 1
- net /h-driver/3V3: track 0.00 -> 31.1 mm, vias 0 -> 4
- net /power-supply/V_BATT: track 0.00 -> 24.0 mm
- net Net-(R8-Pad2): track 0.00 -> 13.5 mm
- net Net-(C25-Pad2): track 0.00 -> 12.1 mm
- net /h-driver/1V8: track 0.00 -> 12.1 mm, vias 0 -> 2
- net /h-driver/B1-: track 0.00 -> 10.5 mm
- net /power-supply/2V5: track 0.00 -> 10.1 mm
- net /h-driver/B1+: track 0.00 -> 9.99 mm
- net /h-driver/B0-: track 0.00 -> 9.44 mm
- net /h-driver/B0+: track 0.00 -> 8.92 mm
- net /h-driver/VD: track 0.00 -> 8.90 mm, vias 0 -> 2
- net /h-driver/TCLK-: track 0.00 -> 8.38 mm
- net /h-driver/GP03: track 0.00 -> 8.33 mm
- net /h-driver/GP04: track 0.00 -> 8.33 mm
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Other:
- board size 115 x 40 mm -> 63.5 x 38.1 mm
- rule trace_min: 0.2 -> 0.1
- rule via_min_drill: 0.3 -> 0.1
- rule via_min_size: 0.4 -> 0.1

Commit message: Work on proto breakout.
Parts:
- removed C1, C9: 56nF, w_smd_cap:c_0603
- removed C10: 10.0uF/9.0Mohm, w_smd_cap:c_0603
- removed C11: 1.0F/11mOhm, Capacitors_SMD:C_0805_HandSoldering
- removed C12: 68pF, w_smd_cap:c_0603
- removed C13: 2.20uF/2.80Mohm, w_smd_cap:c_0603
- removed C14: 1.5nF, w_smd_cap:c_0603
- removed C15, C26, C27, C28, C8: 100nF, w_smd_cap:c_0603
- removed C16: 1.0F/20Mohm, w_smd_cap:c_0603
- removed C17: 15F, w_smd_cap:c_0805
- removed C18, C19: 1.0F, w_smd_cap:c_0603
- removed C2: 10.0F/9Mohm, w_smd_cap:c_0603
- removed C20: 4.7F/5.0mOhm, Capacitors_SMD:C_0603_HandSoldering
- removed C21, C22, C23: 10.0F/3.0mOhm, w_smd_cap:c_0603
- removed C24: 2.2F/4.9Mohm, w_smd_cap:c_0603
- removed C25: 9.0pF, Capacitors_SMD:C_0805_HandSoldering
- removed C29: 270pF, w_smd_cap:c_0603
- removed C3: 4.7F/6Mohm, w_smd_cap:c_0603
- removed C30: 4.7F/2Mohm, w_smd_cap:c_0603
- removed C31: 10F/9Mohm, Capacitors_SMD:C_0603_HandSoldering
- removed C32, C33, C34: 47F/3Mohm, w_smd_cap:c_0603
- removed C35: 220nF/220Mohm, w_smd_cap:c_0603
- removed C36, C37, C58, C59: 0.1u, w_smd_cap:c_0603
- removed C4: 1.0uF, Capacitors_SMD:C_0805_HandSoldering
- removed C5: 220nF, w_smd_cap:c_0603
- removed C50, C51, C52, C53, C54, C55, C56: 0.1uF, w_smd_cap:c_0603
- removed C57: 4.7uF, w_smd_cap:c_0603
- removed C6: 470pF, w_smd_cap:c_0603
- removed C7: 22nF, w_smd_cap:c_0603
- removed D1: 9V/5W, Diodes_SMD:Diode-SMB_Handsoldering
- removed D2: ZENERsmall, w_smd_diode:sod80c
- removed D3: ZENER, w_smd_diode:sod80c
- removed D4: D, w_smd_diode:sod123
- removed L1: 22H, w_smd_inductors:inductor_smd_0805
- removed L3: 100nH, w_smd_inductors:inductor_smd_0805
- removed L4: 12.0H/210Mohm, w_smd_inductors:inductor_smd_0805
- removed L5: 2.2H/140ohm, camera:Inductor_SMD_2016
- removed L6, L7: 1.5H/14.4mOhm, w_smd_inductors:inductor_smd_0805
- removed L8: 2.2H/13.0mOhm, w_smd_inductors:inductor_smd_0805
- removed L9: 100nH/20Mohm, w_smd_inductors:inductor_smd_0805
- removed P1: CONN_01X02, w_pin_strip:pin_strip_2
- removed Q1: Q_NMOS_DGS, w_smd_trans:sot23
- removed R1: 80.6k, w_smd_resistors:r_0805
- removed R10: 68.1k, Resistors_SMD:R_0805_HandSoldering
- removed R11: 27k, w_smd_resistors:r_0805
- removed R12: 82M/1W, w_smd_resistors:r_0805
- removed R13: 53.6k, Resistors_SMD:R_0805_HandSoldering
- removed R14: 7.87k, w_smd_resistors:r_0805
- removed R15: 1.65k, w_smd_resistors:r_0805
- removed R16: 1M, w_smd_resistors:r_0805
- removed R17: 13.3k, w_smd_resistors:r_0805
- removed R18: 118k, w_smd_resistors:r_0805
- removed R19: 100k/63.0mW, Resistors_SMD:R_0402
- removed R2: 105k, w_smd_resistors:r_0805
- removed R20: 402.0k/63mW, Resistors_SMD:R_0402
- removed R21, R23: 5.76k, w_smd_resistors:r_0805
- removed R22, R24, R26: 10.0k, w_smd_resistors:r_0805
- removed R25: 13.7k, w_smd_resistors:r_0805
- removed R27: 100k, w_smd_resistors:r_0805
- removed R28: 1M0, w_smd_resistors:r_0805
- removed R3: 3.57k, w_smd_resistors:r_0805
- removed R4: 453k, w_smd_resistors:r_0805
- removed R5: 10k, w_smd_resistors:r_0805
- removed R6, R8: 10.0k, Resistors_SMD:R_0805_HandSoldering
- removed R7: 10.2k, w_smd_resistors:r_0805
- removed R9: 51.1k, Resistors_SMD:R_0805_HandSoldering
- removed U1: LMZ10500, camera:llp-8
- removed U10: CXD3400N, w_smd_dil:tssop-20
- removed U12: ADDI7013, camera:csp-bga-bc-76-3
- removed U3: TPS2420, Housings_DFN_QFN:QFN-16-1EP_4x4mm_Pitch0.65mm
- removed U5: LM3674, w_smd_trans:sot23-5
- removed U6, U7, U8: TPS56x200, w_smd_trans:sot23-6
- removed U9: LMR62014, w_smd_trans:sot23-5
- added P3: CONN_01X10, w_pin_strip:pin_strip_10, F.Cu at (97.8, 105.6)
- added P4: CONN_01X03, w_pin_strip:pin_strip_3, F.Cu at (114.3, 94.1)
- added P5: CONN_01X12, w_pin_strip:pin_strip_12, F.Cu at (95.3, 94.1)
- added P6: CONN_01X03, w_pin_strip:pin_strip_3, F.Cu at (114.3, 105.6)
- added P7: CONN_01X03, w_pin_strip:pin_strip_3, F.Cu at (76.2, 94.1)
- added REF**: Logo, Symbols:Symbol_OSHW-Logo_SilkScreen, F.Cu at (114.3, 99.1)
- C38: value 1/35V -> 0.1uF; footprint w_smd_cap:c_0805 -> w_smd_cap:c_0603
- C40: value 2.2uF -> 0.1uF
- C41, C42: value 0.1 -> 0.1uF
- C43: value 0.01 -> 0.1uF
- C44, C46: value 3.3/20V -> 0.1uF; footprint w_smd_cap:c_0805 -> w_smd_cap:c_0603
- C45: value 0.01 -> 0.1uF; footprint w_smd_cap:c_0805 -> w_smd_cap:c_0603
- C47: value 3.3/20V -> 4.7uF; footprint w_smd_cap:c_0805 -> w_smd_cap:c_0603
- C48: value 0.1uF -> 0.1u
- C49: value 0.1uF -> 0.1u; moved to F.Cu
- P2: value CONN_01X24 -> CONN_01X05; footprint camera:FFC-24-0.5mm -> w_pin_strip:pin_strip_5
- U11: value ICX825AQA -> ADDI7013; footprint camera:ICX825 -> camera:csp-bga-bc-76-3; moved to F.Cu
- moved U11 62.0 mm to (93.2, 100.0)
- moved C41 59.6 mm to (85.4, 102.3)
- moved C42 53.5 mm to (99.9, 98.7), turned to 180 degrees
- moved C46 44.0 mm to (88.7, 99.0)
- moved C43 39.4 mm to (85.4, 101.1)
- moved C47 37.8 mm to (99.9, 102.0), turned to 180 degrees
- moved C45 35.8 mm to (102.8, 98.6), turned to 180 degrees
- moved C44 31.8 mm to (88.7, 100.1)
- moved C40 31.2 mm to (99.9, 99.8), turned to 180 degrees
- moved C49 21.0 mm to (85.1, 97.4), turned to 90 degrees
- moved C48 19.4 mm to (83.5, 97.3), turned to 90 degrees
- moved P2 12.5 mm to (78.8, 105.6), turned to 0 degrees
- moved C38 9.83 mm to (99.9, 101.0), turned to 180 degrees
- moved C39 6.47 mm to (102.8, 101.4), turned to 180 degrees
Connections:
- C38 pad 1: Net-(C38-Pad1) -> /h-driver/3V3
- C38 pad 2: Net-(C38-Pad2) -> /h-driver/GND
- C39 pad 1: Net-(C38-Pad1) -> /h-driver/1V8
- C39 pad 2: /camera/SUB -> /h-driver/GND
- C40 pad 1: /camera/SUB -> /h-driver/3V3
- C40 pad 2: /camera/GND -> /h-driver/GND
- C41 pad 1: Net-(C41-Pad1) -> /h-driver/1V8
- C41 pad 2: /h-driver/RG1 -> /h-driver/GND
- C42 pad 1: Net-(C42-Pad1) -> /h-driver/3V3
- C42 pad 2: /h-driver/RG2 -> /h-driver/GND
- C43 pad 1: /camera/GND -> /h-driver/1V8
- C43 pad 2: /camera/12V -> /h-driver/GND
- C44 pad 1: /camera/12V -> /h-driver/3V3
- C44 pad 2: /camera/GND -> /h-driver/GND
- C45 pad 1: /camera/GND -> /h-driver/1V8
- C45 pad 2: /camera/12V -> /h-driver/GND
- C46 pad 1: /camera/12V -> /h-driver/3V3
- C46 pad 2: /camera/GND -> /h-driver/GND
- C47 pad 1: /camera/GND -> /h-driver/3V3
- C47 pad 2: /camera/-7V -> /h-driver/GND
- C48 pad 1: /h-driver/3V3 -> /h-driver/IN_A+
- C48 pad 2: /camera/GND -> Net-(C48-Pad2)
- C49 pad 1: /h-driver/1V8 -> /h-driver/IN_B+
- C49 pad 2: /camera/GND -> Net-(C49-Pad2)
Routing:
- net /camera/GND: track 101.7 -> 0.00 mm, vias 1 -> 0
- net /h-driver/GND: track 0.00 -> 96.9 mm, vias 0 -> 8
- net /h-driver/1V8: track 12.1 -> 60.0 mm, vias 2 -> 5
- net /power-supply/V_BATT: track 24.0 -> 0.00 mm
- net /h-driver/SDATA: track 7.24 -> 28.0 mm, vias 2 -> 1
- net /h-driver/HD: track 6.92 -> 27.6 mm
- net /h-driver/VD: track 8.90 -> 29.6 mm
- net /h-driver/3V3: track 31.1 -> 50.4 mm, vias 4 -> 7
- net /h-driver/RG1: track 0.00 -> 18.3 mm
- net /h-driver/SCK: track 7.18 -> 25.3 mm, vias 2 -> 1
- net /h-driver/IN_A-: track 0.00 -> 17.3 mm
- net /h-driver/SYNC: track 6.99 -> 22.7 mm, vias 2 -> 1
- net /h-driver/SL: track 7.29 -> 22.6 mm, vias 2 -> 1
- net /h-driver/HL1: track 0.00 -> 15.1 mm
- net Net-(R8-Pad2): track 13.5 -> 0.00 mm
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- added copper zone on B.Cu, net /h-driver/GND
- added copper zone on F.Cu, net /h-driver/GND
Other:
- board size 63.5 x 38.1 mm -> 45.7 x 14 mm
- board text added: "Proto V0.1"

Commit message: Lot's of back and forward with vendor.
Parts:
- removed C38, C39, C40, C41, C42, C43, C44, C45, C46: 0.1uF, w_smd_cap:c_0603
- removed C47: 4.7uF, w_smd_cap:c_0603
- removed C48, C49: 0.1u, w_smd_cap:c_0603
- removed P2: CONN_01X05, w_pin_strip:pin_strip_5
- removed P3: CONN_01X10, w_pin_strip:pin_strip_10
- removed P4, P6, P7: CONN_01X03, w_pin_strip:pin_strip_3
- removed P5: CONN_01X12, w_pin_strip:pin_strip_12
- removed REF**: Logo, Symbols:Symbol_OSHW-Logo_SilkScreen
- removed U11: ADDI7013, camera:csp-bga-bc-76-3
- added C1: 1.0uF, Capacitors_SMD:C_0805_HandSoldering, F.Cu at (102.4, 95.6)
- added C10: 0.1uF, Capacitors_SMD:C_0805_HandSoldering, F.Cu at (125.8, 73.0)
- added C11: 10uF, Capacitors_SMD:C_0805_HandSoldering, F.Cu at (99.9, 65.3)
- added C14: 10.0F/3.0mOhm, w_smd_cap:c_0603, F.Cu at (131.4, 92.0)
- added C15: 10.0F/9Mohm, w_smd_cap:c_0603, F.Cu at (109.3, 69.3)
- added C16: 470pF, w_smd_cap:c_0603, F.Cu at (112.0, 75.2)
- added C2: 1.0uF, Capacitors_SMD:C_0805_HandSoldering, F.Cu at (129.4, 77.7)
- added C20: 100nF, w_smd_cap:c_0603, F.Cu at (131.4, 95.2)
- added C21: 10.0uF/9.0Mohm, w_smd_cap:c_0603, F.Cu at (113.7, 70.2)
- added C25: 47F/3Mohm, w_smd_cap:c_0603, F.Cu at (127.0, 98.4)
- added C3: 47pF, Capacitors_SMD:C_0805_HandSoldering, F.Cu at (133.1, 84.1)
- added C4: 2.20uF/2.80Mohm, w_smd_cap:c_0603, F.Cu at (102.7, 69.0)
- added C5: 47pF, Capacitors_SMD:C_0805_HandSoldering, F.Cu at (133.1, 69.7)
- added C6: 1.0uF, Capacitors_SMD:C_0805_HandSoldering, F.Cu at (129.4, 80.1)
- added C7: 100nF, Capacitors_SMD:C_0805_HandSoldering, F.Cu at (130.3, 66.0)
- added C8: 1.0F/11mOhm, Capacitors_SMD:C_0805_HandSoldering, F.Cu at (111.4, 81.6)
- added C9: 4.7uF, Capacitors_SMD:C_0805_HandSoldering, F.Cu at (126.6, 66.6)
- added D1: 9V/5W, Diodes_SMD:Diode-SMB_Handsoldering, F.Cu at (104.4, 90.6)
- added L1: 15uH, w_smd_inductors:inductor_smd_0805, F.Cu at (130.0, 82.8)
- added L2: 15uH, w_smd_inductors:inductor_smd_0805, F.Cu at (125.8, 80.5)
- added L3: 2.0uH/0.024Ohm, w_smd_inductors:inductor_smd_0805, F.Cu at (99.2, 72.8)
- added L4: 10uH, w_smd_inductors:inductor_smd_0805, F.Cu at (125.8, 76.9)
- added L8: 2.2H/13.0mOhm, w_smd_inductors:inductor_smd_0805, F.Cu at (130.0, 98.8)
- added P8: CONN_01X06, w_pin_strip:pin_socket_6, F.Cu at (118.0, 99.5)
- added P9: CONN_01X02, w_pin_strip:pin_socket_2, F.Cu at (100.3, 99.6)
- added R1: 10.0k, Resistors_SMD:R_0805_HandSoldering, F.Cu at (99.4, 86.6)
- added R16: 13.7k, w_smd_resistors:r_0805, F.Cu at (126.8, 89.6)
- added R17: 10.0k, w_smd_resistors:r_0805, F.Cu at (129.2, 89.8)
- added R2: 324k, w_smd_resistors:r_0603, F.Cu at (131.1, 69.7)
- added R3: 10.0k, Resistors_SMD:R_0805_HandSoldering, F.Cu at (99.4, 82.6)
- added R4: 51.1k, Resistors_SMD:R_0805_HandSoldering, F.Cu at (111.5, 86.2)
- added R5: 68.1k, Resistors_SMD:R_0805_HandSoldering, F.Cu at (111.5, 84.0)
- added R6: 53.6k, Resistors_SMD:R_0805_HandSoldering, F.Cu at (99.4, 78.6)
- added R7: 324k, w_smd_resistors:r_0603, F.Cu at (127.3, 69.7)
- added R8: 80.6k, w_smd_resistors:r_0805, F.Cu at (108.4, 75.2)
- added R9: 105k, w_smd_resistors:r_0805, F.Cu at (110.3, 76.8)
- added U1: TPS2420, camera:S-PVQFN-N16, F.Cu at (105.7, 84.6)
- added U2: LT3487, w_smd_qfn:dfn10-3x3, F.Cu at (129.7, 73.9)
- added U3: TPS63002, Housings_DFN_QFN:DFN-10-1EP_3x3mm_Pitch0.5mm, F.Cu at (99.5, 69.2)
- added U7: TPS56x200, w_smd_trans:sot23-6, F.Cu at (128.0, 94.0)
- added U8: LMZ10500, camera:llp-8, F.Cu at (109.7, 72.0)
Routing:
- net /power-supply/GND: track 0.00 -> 182.7 mm, vias 0 -> 22
- net /power-supply/5V5: track 0.00 -> 142.0 mm, vias 0 -> 7
- net /h-driver/GND: track 96.9 -> 0.00 mm, vias 8 -> 0
- net /power-supply/5V0: track 0.00 -> 63.0 mm
- net /h-driver/1V8: track 60.0 -> 0.00 mm, vias 5 -> 0
- net /h-driver/3V3: track 50.4 -> 0.00 mm, vias 7 -> 0
- net /power-supply/3V3: track 0.00 -> 42.1 mm, vias 0 -> 2
- net /power-supply/+12V: track 0.00 -> 34.5 mm, vias 0 -> 4
- net /power-supply/V_BAT: track 0.00 -> 32.1 mm
- net /h-driver/VD: track 29.6 -> 0.00 mm, vias 2 -> 0
- net /power-supply/1V8: track 0.00 -> 29.4 mm
- net /power-supply/-7V: track 0.00 -> 29.4 mm, vias 0 -> 2
- net /h-driver/SDATA: track 28.0 -> 0.00 mm, vias 1 -> 0
- net /h-driver/HD: track 27.6 -> 0.00 mm, vias 2 -> 0
- net /h-driver/SCK: track 25.3 -> 0.00 mm, vias 1 -> 0
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- added copper zone on F.Cu, net /power-supply/+12V
- added copper zone on F.Cu, net /power-supply/-7V
- added copper zone on F.Cu, net /power-supply/1V8
- added copper zone on F.Cu, net /power-supply/3V3
- added copper zone on F.Cu, net /power-supply/5V5
- added copper zone on B.Cu, net /power-supply/GND
- added copper zone on F.Cu, net /power-supply/GND
- added copper zone on B.Cu, net /power-supply/PAD
- added copper zone on F.Cu, net /power-supply/V_BAT
- removed copper zone on B.Cu, net /h-driver/GND
- removed copper zone on F.Cu, net /h-driver/GND
Other:
- board size 45.7 x 14 mm -> 40 x 40 mm
- net class Default: clearance 0.2 -> 0.1524; trace_width 0.25 -> 0.254; via_dia 0.6 -> 0.604774; via_drill 0.4 -> 0.299974
- rule trace_clearance: 0.2 -> 0.1524
- rule trace_min: 0.1 -> 0.1524
- rule via_min_drill: 0.1 -> 0.299974
- rule via_min_size: 0.1 -> 0.604774
- board text added: "+"
- board text added: "-"
- board text added: "-7.0V"
- board text added: "1.8V"
- board text added: "12.0V"
- board text added: "3.3V"
- board text added: "5.0V"
- board text added: "5.5V"
- board text removed: "Proto V0.1"
