File: AstroCam.kicad_pcb (KiCad board)
At the start: 2 copper layers, 40 x 40 mm, 41 parts, among them P8 CONN_01X06, P9 CONN_01X02, U1 TPS2420, U2 LT3487, U3 TPS63002, U7 TPS56x200, U8 LMZ10500

Commit message: lots of work
Parts:
- added C12, C13, C26, C27: 0.1u, Capacitors_SMD:C_0603, F.Cu at (227.5, 93.0)
- added C28: 1u/35V, Capacitors_SMD:c_elec_4x5.3, F.Cu at (227.5, 93.0)
- added C29: 0.1uF, Capacitors_SMD:C_0603, F.Cu at (227.5, 93.0)
- added C30: 2200pF, Capacitors_SMD:C_0603, F.Cu at (227.5, 93.0)
- added C31, C32: 0.1, Capacitors_SMD:C_0603, F.Cu at (227.5, 93.0)
- added C33, C35: 0.01, Capacitors_SMD:C_0603, F.Cu at (227.5, 93.0)
- added C34, C36, C37: 3.3/20V, Capacitors_SMD:c_elec_4x5.3, F.Cu at (227.5, 93.0)
- added C38, C39, C40, C41, C42, C43, C44, C45, C46: 0.1uF, Capacitors_SMD:C_0603_HandSoldering, F.Cu at (227.5, 93.0)
- added C47: 4.7uF, Capacitors_SMD:C_0603_HandSoldering, F.Cu at (227.5, 93.0)
- added C48, C49: 0.1u, Capacitors_SMD:C_0603_HandSoldering, F.Cu at (227.5, 93.0)
- added D2: D, Diodes_SMD:SOD-123, F.Cu at (227.5, 93.0)
- added P1: CONN_01X02, Pin_Headers:Pin_Header_Straight_1x02, F.Cu at (227.5, 93.0)
- added P10: CONN_01X14, Pin_Headers:Pin_Header_Straight_1x14, F.Cu at (227.5, 93.0)
- added P2, P3: CONN_01X18, Pin_Headers:Pin_Header_Straight_1x18, F.Cu at (227.5, 93.0)
- added P4: CONN_01X04, Socket_Strips:Socket_Strip_Straight_1x04, F.Cu at (227.5, 93.0)
- added P5: CONN_01X01, Socket_Strips:Socket_Strip_Straight_1x01, F.Cu at (227.5, 93.0)
- added Q1, Q3: 2SC5095, w_smd_trans:sot323, F.Cu at (227.5, 93.0)
- added Q2, Q4: MT3S20TU, w_smd_trans:sot323, F.Cu at (227.5, 93.0)
- added R10, R11, R14, R15: 10K, Resistors_SMD:R_0603_HandSoldering, F.Cu at (227.5, 93.0)
- added R12, R20: 1.17K, Resistors_SMD:R_0603_HandSoldering, F.Cu at (227.5, 93.0)
- added R13, R21: 1.74K, Resistors_SMD:R_0603_HandSoldering, F.Cu at (227.5, 93.0)
- added R18: 100k, Resistors_SMD:R_0603_HandSoldering, F.Cu at (227.5, 93.0)
- added R19: 1M0, Resistors_SMD:R_0603_HandSoldering, F.Cu at (227.5, 93.0)
- added R22: 10.0k, Resistors_SMD:R_0603_HandSoldering, F.Cu at (227.5, 93.0)
- added U10: ICX825AQA, camera:ICX825, F.Cu at (227.5, 93.0)
- added U11: ADDI7013, camera:csp-bga-bc-76-3, F.Cu at (227.5, 93.0)
- added U4: TXB0104, Housings_SSOP:TSSOP-14_4.4x5mm_Pitch0.65mm, F.Cu at (227.5, 93.0)
- added U9: CXD3400N, w_smd_dil:tssop-20, F.Cu at (227.5, 93.0)
- C14: value 10.0F/3.0mOhm -> 10.0uF; footprint w_smd_cap:c_0603 -> Capacitors_SMD:C_0805_HandSoldering
- C15: value 10.0F/9Mohm -> 10.0uF; footprint w_smd_cap:c_0603 -> Capacitors_SMD:C_0805_HandSoldering
- C16: footprint w_smd_cap:c_0603 -> Capacitors_SMD:C_0402
- C20: value 100nF -> 0.1uF; footprint w_smd_cap:c_0603 -> Capacitors_SMD:C_0603_HandSoldering
- C21: value 10.0uF/9.0Mohm -> 10.0uF; footprint w_smd_cap:c_0603 -> Capacitors_SMD:C_0805_HandSoldering
- C25: value 47F/3Mohm -> 47uF; footprint w_smd_cap:c_0603 -> Capacitors_SMD:C_1206_HandSoldering
- C4: value 2.20uF/2.80Mohm -> 2.2uF; footprint w_smd_cap:c_0603 -> Capacitors_SMD:C_0603_HandSoldering
- C8: value 1.0F/11mOhm -> 1.0uF/11mOhm
- L3: value 2.0uH/0.024Ohm -> 2.0uH
- L8: value 2.2H/13.0mOhm -> 2.2uH
- P8: footprint w_pin_strip:pin_socket_6 -> Pin_Headers:Pin_Header_Straight_1x06
- P9: footprint w_pin_strip:pin_socket_2 -> Pin_Headers:Pin_Header_Straight_1x02
- R16, R17, R8, R9: footprint w_smd_resistors:r_0805 -> Resistors_SMD:R_0402
- R2, R7: footprint w_smd_resistors:r_0603 -> Resistors_SMD:R_0603_HandSoldering
- R3, R4, R5, R6: footprint Resistors_SMD:R_0805_HandSoldering -> Resistors_SMD:R_0603_HandSoldering
- U1: footprint camera:S-PVQFN-N16 -> Housings_DFN_QFN:QFN-16-1EP_4x4mm_Pitch0.65mm
- U7: footprint w_smd_trans:sot23-6 -> Housings_SOT-23_SOT-143_TSOT-6:SOT-23-6
- moved R16 9.81 mm to (130.3, 98.8), turned to 180 degrees
- moved C25 9.62 mm to (132.0, 90.2)
- moved L8 9.60 mm to (128.3, 89.4), turned to 0 degrees
- moved R17 9.05 mm to (127.9, 98.8), turned to 180 degrees
- moved P8 6.35 mm to (111.6, 99.5), turned to 90 degrees
- moved C14 3.74 mm to (127.7, 92.0), turned to 0 degrees
- moved U7 1.54 mm to (127.6, 95.5), turned to 270 degrees
- moved P9 1.27 mm to (99.1, 99.6), turned to 90 degrees
- moved C20 0.86 mm to (130.6, 95.5), turned to 90 degrees
- moved R7 0.27 mm to (127.5, 69.9), turned to 180 degrees
- turned C15 to 0 degrees
- turned C16 to 0 degrees
- turned C21 to 90 degrees
- turned C4 to 90 degrees
- turned R2 to 270 degrees
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Connections:
- net Net-(C16-Pad1) renamed /power-supply/VCON
- net Net-(C7-Pad1) renamed /power-supply/SOFT_START
- C1 pad 2: /power-supply/GND -> GND
- C11 pad 2: /power-supply/GND -> GND
- C14 pad 2: /power-supply/GND -> GND
- C15 pad 2: /power-supply/GND -> GND
- C16 pad 2: /power-supply/GND -> GND
- C2 pad 2: /power-supply/GND -> GND
- C21 pad 2: /power-supply/GND -> GND
- C25 pad 2: /power-supply/GND -> GND
- C3 pad 2: /power-supply/GND -> GND
- C4 pad 2: /power-supply/GND -> GND
- C7 pad 2: /power-supply/GND -> GND
- C8 pad 2: /power-supply/GND -> GND
- C9 pad 2: /power-supply/GND -> GND
- D1 pad 2: /power-supply/GND -> GND
- P9 pad 2: /power-supply/GND -> GND
- R17 pad 2: /power-supply/GND -> GND
- R4 pad 2: /power-supply/GND -> GND
- R5 pad 2: /power-supply/GND -> GND
- R6 pad 2: /power-supply/GND -> GND
- R9 pad 2: /power-supply/GND -> GND
- U1 pad 16: /power-supply/GND -> GND
- U1 pad 5: /power-supply/GND -> GND
- U1 pad 6: /power-supply/GND -> GND
- U2 pad 11: /power-supply/GND -> GND
- U3 pad 11: /power-supply/GND -> GND
- U3 pad 3: /power-supply/GND -> GND
- U3 pad 9: /power-supply/GND -> GND
- U7 pad 1: /power-supply/GND -> GND
- U8 pad 4: /power-supply/GND -> GND
- U8 pad 6: /power-supply/GND -> GND
- U8 pad 9: /power-supply/GND -> GND
Routing:
- net /power-supply/GND: track 182.7 -> 0.00 mm, vias 22 -> 0
- net GND: track 0.00 -> 164.6 mm, vias 0 -> 25
- net /power-supply/3V3: track 42.1 -> 19.8 mm
- net /power-supply/5V5: track 142.0 -> 160.3 mm
- net Net-(C20-Pad1): track 7.51 -> 2.01 mm
- net /power-supply/1V8: track 29.4 -> 27.5 mm
- net /power-supply/V_BAT: track 32.1 -> 33.7 mm
- net /power-supply/VCON: track 5.85 -> 7.01 mm
- net /power-supply/FBP: track 3.66 -> 2.85 mm
- net /power-supply/FBN: track 7.39 -> 6.59 mm
- net /power-supply/CAP: track 10.0 -> 9.31 mm
- net Net-(C20-Pad2): track 8.40 -> 9.05 mm, vias 0 -> 2
- net Net-(R16-Pad2): track 5.03 -> 4.45 mm
- added copper zone on B.Cu, net GND
- added copper zone on F.Cu, net GND
- removed copper zone on F.Cu, net /power-supply/1V8
- removed copper zone on B.Cu, net /power-supply/GND
- removed copper zone on F.Cu, net /power-supply/GND
- removed copper zone on B.Cu, net /power-supply/PAD
