File: AstroCam.sch (KiCad schematic (older format))
At the start: 30 parts, among them P1 CONN_01X02, P2 CONN_02X03, U1 AD9974

Commit message: initial experimentation with size constraints
Parts:
- removed C1, C10, C14, C15, C17, C19, C2, C20, C23, C25, C26, C27, C3, C4, C7, C9: 0.1uF, w_smd_cap:c_0603, symbol C_Small
- removed C11, C13, C18, C22, C24, C5, C6: 4.7uF, symbol CP1_Small
- removed C12, C16: 0.1u, w_smd_cap:c_0603, symbol C_Small
- removed C21, C8: 0.1uF, w_smd_cap:c_0603, symbol C
- removed P2: CONN_02X03, symbol CONN_02X03
- removed U1: AD9974, w_smd_bga:tfbga100-std, symbol AD9974
- P1: footprint (none) -> w_pin_strip:pin_strip_2
Connections:
- net labels removed: 1V8, 3V0, CCD_OUT1, CCD_OUT2, CLK_A, CLK_B, DATA_A, DATA_B, GND, H1A, H1B, H2A, H2B, H3A, H3B, H4A, H4B, HD_A, HD_B, LDO_OUT_A, LDO_OUT_B, RG_A, RG_B, SCK_A, SCK_B, SDATA_A, SDATA_B, SL_A, SL_B, VD_A, VD_B, V_BATT
- wire segments 127 -> 63
- no-connect marks 8 -> 0
Other:
- note removed: "Horizontal & Vertical Clock Pulses from FPGA\n"
- moved on the sheet: P1

Commit message: Work on proto breakout.
Changed lines of the file:
@@
 $Descr A4 11693 8268
 encoding utf-8
-Sheet 1 4
+Sheet 1 5
 Title ""
 Date ""
@@
 F8 "1V2_2" I R 3850 4250 60
 F9 "1V8" I R 3850 3950 60
-F10 "12V" I R 3850 3050 60
-F11 "5V0" I R 3850 3500 60
-F12 "5V5" I R 3850 3350 60
+F10 "5V0" I R 3850 3500 60
+F11 "5V5" I R 3850 3350 60
+F12 "12V" I R 3850 3050 60
 $EndSheet
 $Sheet
@@
 Wire Wire Line
 	4450 2900 4450 4300
+$Sheet
+S 8350 3150 1800 1400
+U 557FDF11
+F0 "Save" 60
+F1 "Save.sch" 60
+$EndSheet
 $EndSCHEMATC

Commit message: more work
Changed lines of the file:
@@
 F12 "12V" I R 3850 3050 60
-$EndSheet
-$Sheet
-S 4500 1850 1100 1200
-U 557AFA5B
-F0 "camera" 60
-F1 "camera.sch" 60
-F2 "RG_A" I L 4500 1950 60
-F3 "RG_B" I L 4500 2050 60
-F4 "LH1_1" I R 5600 1950 60
-F5 "H1S_1" I R 5600 2050 60
-F6 "H1T_1" I R 5600 2150 60
-F7 "H2S_1" I R 5600 2250 60
-F8 "H2T_1" I R 5600 2350 60
-F9 "LH1_2" I R 5600 2500 60
-F10 "H1S_2" I R 5600 2600 60
-F11 "H1T_2" I R 5600 2700 60
-F12 "H2S_2" I R 5600 2800 60
-F13 "H2T_2" I R 5600 2900 60
-F14 "CCD_OUT1" I L 4500 2800 60
-F15 "CCD_OUT2" I L 4500 2900 60
-F16 "12V" I L 4500 2250 60
-F17 "-7V" I L 4500 2350 60
-F18 "GND" I L 4500 2550 60
-F19 "5V0" I L 4500 2450 60
 $EndSheet
 $Comp
@@
 F1 "Save.sch" 60
 $EndSheet
+$Sheet
+S 4500 1850 1100 1200
+U 557AFA5B
+F0 "camera" 60
+F1 "camera.sch" 60
+$EndSheet
 $EndSCHEMATC

Commit message: lots of work
Parts:
- P1: footprint w_pin_strip:pin_strip_2 -> Pin_Headers:Pin_Header_Straight_1x02
Changed lines of the file:
@@
 F 0 "P1" H 2150 3450 50  0000 C CNN
 F 1 "CONN_01X02" V 2250 3300 50  0000 C CNN
-F 2 "w_pin_strip:pin_strip_2" H 2150 3300 60  0001 C CNN
+F 2 "Pin_Headers:Pin_Header_Straight_1x02" H 2150 3300 60  0001 C CNN
 F 3 "" H 2150 3300 60  0000 C CNN
 	1    2150 3300
