File: breakout-addi.kicad_pcb (KiCad board)
At the start: 2 copper layers, 45.7 x 15.2 mm, 20 parts, among them P2 CONN_01X05, P3 CONN_01X10, P4 CONN_01X03, P5 CONN_01X12, P6 CONN_01X03, P7 CONN_01X03, U11 ADDI7013

Commit message: more work
Parts:
- removed P4, P6, P7: CONN_01X03, w_pin_strip:pin_strip_3
- removed P5: CONN_01X12, w_pin_strip:pin_strip_12
- P2: value CONN_01X05 -> CONN_01X18; footprint w_pin_strip:pin_strip_5 -> w_pin_strip:pin_strip_18
- P3: value CONN_01X10 -> CONN_01X18; footprint w_pin_strip:pin_strip_10 -> w_pin_strip:pin_strip_18
- moved P2 16.5 mm to (57.9, 58.4)
- moved P3 13.0 mm to (57.9, 45.7)
Connections:
- P3 pad 1: /h-driver/A0+ -> /h-driver/1V8
- P3 pad 10: /h-driver/B1- -> /h-driver/H4
- P3 pad 2: /h-driver/A0- -> /h-driver/3V3
- P3 pad 3: /h-driver/A1+ -> /h-driver/GND
- P3 pad 4: /h-driver/A1- -> /h-driver/IN_A-
- P3 pad 5: /h-driver/TCLK+ -> /h-driver/IN_A+
- P3 pad 6: /h-driver/TCLK- -> /h-driver/IN_B+
- P3 pad 7: /h-driver/B0+ -> /h-driver/IN_B-
- P3 pad 8: /h-driver/B0- -> /h-driver/RG2
- P3 pad 9: /h-driver/B1+ -> /h-driver/HL2
Routing:
- net /h-driver/GND: track 74.0 -> 96.2 mm, vias 5 -> 8
- net /h-driver/A1+: track 22.8 -> 5.51 mm
- net /h-driver/A1-: track 22.8 -> 5.51 mm
- net /h-driver/A0-: track 15.2 -> 7.68 mm
- net /h-driver/A0+: track 14.9 -> 7.60 mm
- net /h-driver/TCLK+: track 14.4 -> 8.84 mm
- net /h-driver/TCLK-: track 14.4 -> 8.92 mm
- net /h-driver/1V8: track 60.0 -> 62.7 mm
- net /h-driver/B0+: track 14.1 -> 13.2 mm
- net /h-driver/B0-: track 14.1 -> 13.3 mm
- net /h-driver/SYNC: track 29.3 -> 28.5 mm
- net /h-driver/HD: track 26.7 -> 25.9 mm
- net /h-driver/B1-: track 17.6 -> 17.0 mm
Other:
- outline, holes or cut-outs redrawn

Commit message: lots of work
Parts:
- removed REF**: Logo, Symbols:Symbol_OSHW-Logo_SilkScreen
- added G***: LOGO, w_logo:Logo_silk_OSHW_6x6mm, F.Cu at (78.0, 51.4)
- C38, C39, C40, C41, C42, C43, C44, C45, C46, C47, C48, C49: footprint w_smd_cap:c_0603 -> Capacitors_SMD:C_0603_HandSoldering
- moved C47 21.6 mm to (41.3, 49.1)
- moved C41 18.8 mm to (66.8, 53.2)
- moved C42 15.2 mm to (47.9, 54.1), turned to 0 degrees
- moved C38 14.6 mm to (47.9, 52.5), turned to 0 degrees
- moved C46 12.2 mm to (62.7, 53.2)
- moved C44 11.8 mm to (62.7, 51.5)
- moved C43 3.33 mm to (47.9, 55.8)
- moved C39 3.24 mm to (66.8, 49.9), turned to 0 degrees
- moved C45 2.02 mm to (66.8, 51.5), turned to 0 degrees
- moved C48 1.84 mm to (47.6, 49.9), turned to 0 degrees
- moved C40 1.42 mm to (62.8, 49.9), turned to 0 degrees
- moved C49 0.60 mm to (47.6, 48.2), turned to 0 degrees
Connections:
- C38 pad 2: /h-driver/GND -> GND
- C39 pad 2: /h-driver/GND -> GND
- C40 pad 2: /h-driver/GND -> GND
- C41 pad 2: /h-driver/GND -> GND
- C42 pad 2: /h-driver/GND -> GND
- C43 pad 2: /h-driver/GND -> GND
- C44 pad 2: /h-driver/GND -> GND
- C45 pad 2: /h-driver/GND -> GND
- C46 pad 2: /h-driver/GND -> GND
- C47 pad 2: /h-driver/GND -> GND
- P3 pad 1: /h-driver/1V8 -> GND
- P3 pad 2: /h-driver/3V3 -> /h-driver/1V8
- P3 pad 3: /h-driver/GND -> /h-driver/3V3
- U11 pad A1: /h-driver/GND -> GND
- U11 pad B2: /h-driver/GND -> GND
- U11 pad B3: /h-driver/GND -> GND
- U11 pad B4: /h-driver/GND -> GND
- U11 pad B5: /h-driver/GND -> GND
- U11 pad B6: /h-driver/GND -> GND
- U11 pad B7: /h-driver/GND -> GND
- U11 pad B8: /h-driver/GND -> GND
- U11 pad B9: /h-driver/GND -> GND
- U11 pad C9: /h-driver/GND -> GND
- U11 pad D4: /h-driver/GND -> GND
- U11 pad D5: /h-driver/GND -> GND
- U11 pad D6: /h-driver/GND -> GND
- U11 pad D7: /h-driver/GND -> GND
- U11 pad D9: /h-driver/GND -> GND
- U11 pad E4: /h-driver/GND -> GND
- U11 pad E7: /h-driver/GND -> GND
- U11 pad E9: /h-driver/GND -> GND
- U11 pad F4: /h-driver/GND -> GND
- U11 pad F7: /h-driver/GND -> GND
- U11 pad F9: /h-driver/GND -> GND
- U11 pad G4: /h-driver/GND -> GND
- U11 pad G5: /h-driver/GND -> GND
- U11 pad G6: /h-driver/GND -> GND
- U11 pad G7: /h-driver/GND -> GND
- U11 pad J3: /h-driver/GND -> GND
- U11 pad J4: /h-driver/GND -> GND
- U11 pad J7: /h-driver/GND -> GND
- U11 pad J8: /h-driver/GND -> GND
Routing:
- net /h-driver/GND: track 96.2 -> 0.00 mm, vias 8 -> 0
- net GND: track 0.00 -> 39.1 mm, vias 0 -> 4
- net /h-driver/1V8: track 62.7 -> 55.2 mm
- net /h-driver/3V3: track 48.3 -> 54.8 mm
- net /h-driver/VD: track 24.2 -> 30.5 mm
- net /h-driver/GP04: track 10.8 -> 16.2 mm
- net /h-driver/HD: track 25.9 -> 30.5 mm
- net Net-(C48-Pad2): track 12.4 -> 7.79 mm
- net /h-driver/GP03: track 13.5 -> 16.3 mm
- net /h-driver/IN_A+: track 2.60 -> 5.12 mm
- net /h-driver/IN_B+: track 3.06 -> 5.51 mm
- net /h-driver/SYNC: track 28.5 -> 30.5 mm
- net /h-driver/SCK: track 25.3 -> 27.0 mm
- net /h-driver/SL: track 22.8 -> 24.4 mm
- net Net-(C49-Pad2): track 10.7 -> 9.24 mm
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- added copper zone on B.Cu, net GND
- added copper zone on F.Cu, net GND
- removed copper zone on B.Cu, net /h-driver/GND
- removed copper zone on F.Cu, net /h-driver/GND
Other:
- board text added: "CCD/ADC Proto V0.3"
- board text removed: "CCD/ADC Proto V0.2"
