File: camera.sch (KiCad schematic (older format))
At the start: 17 parts, among them U11 CXD3400N, U12 ICX825AQA

Commit message: initial experimentation with size constraints
Parts:
- added P2: CONN_01X08, w_smd_strip:bb02-hp08, symbol CONN_01X08
- C38: renamed from C65; footprint (none) -> w_smd_cap:c_0805
- C44: renamed from C71; footprint (none) -> w_smd_cap:c_0805
- C45: renamed from C72; footprint w_smd_cap:c_0603 -> w_smd_cap:c_0805
- C46: renamed from C73; footprint (none) -> w_smd_cap:c_0805
- C47: renamed from C74; footprint (none) -> w_smd_cap:c_0805
- D4: footprint w_pth_diodes:diode_do41 -> w_smd_diode:sod123
- R27, R28: footprint w_smd_resistors:r_0603 -> w_smd_resistors:r_0805
- U10: renamed from U11; footprint w_smd_dil:ssop-16 -> w_smd_dil:tssop-20
- renumbered C63 to C36, C64 to C37, C66 to C39, C67 to C40, C68 to C41, C69 to C42, C70 to C43, U12 to U11
Connections:
- net labels removed: XSGV2, XSGV3, XSUB, XV1, XV2, XV3, XV4
- wire segments 66 -> 78
Changed lines of the file:
@@
 $Descr A4 11693 8268
 encoding utf-8
-Sheet 3 3
+Sheet 3 4
 Title ""
 Date ""
@@
 $EndDescr
 $Comp
-L ICX825AQA U12
+L ICX825AQA U11
 U 1 1 557B0BF2
 P 7750 2900
-F 0 "U12" H 7350 3700 60  0000 C CNN
+F 0 "U11" H 7350 3700 60  0000 C CNN
 F 1 "ICX825AQA" H 7750 2900 60  0000 C CNN
 F 2 "camera:ICX825" H 7750 2900 60  0001 C CNN
@@
 GND
 $Comp
-L CXD3400N U11
+L CXD3400N U10
 U 1 1 557B0C28
 P 3300 2950
-F 0 "U11" H 2850 3800 50  0000 L CNN
+F 0 "U10" H 2850 3800 50  0000 L CNN
 F 1 "CXD3400N" H 3450 2150 50  0000 L CNN
-F 2 "w_smd_dil:ssop-16" H 3300 2950 60  0001 C CNN
+F 2 "w_smd_dil:tssop-20" H 3300 2950 60  0001 C CNN
 F 3 "" H 3300 2950 60  0000 C CNN
 	1    3300 2950
@@
 Text Label 3300 2000 1    60   ~ 0
 5V0
-Text Label 2700 1200 0    60   ~ 0
+Text Label 2350 1000 0    60   ~ 0
 12V
 NoConn ~ 3900 2450
-Text HLabel 2300 2250 0    60   Input ~ 0
-XSUB
-Text HLabel 2300 2450 0    60   Input ~ 0
-XV2
-Text HLabel 2300 2650 0    60   Input ~ 0
-XSGV2
-Text HLabel 2300 2750 0    60   Input ~ 0
-XV3
 Text Label 2700 2550 2    60   ~ 0
 GND
@@
 GND
 Wire Wire Line
-	2300 2750 2700 2750
-Wire Wire Line
-	2300 2650 2700 2650
-Wire Wire Line
-	2300 2450 2700 2450
-Wire Wire Line
-	2300 2250 2700 2250
-Text HLabel 2300 2950 0    60   Input ~ 0
-XSGV3
-Text HLabel 2300 3050 0    60   Input ~ 0
-XV1
-Text HLabel 2300 3150 0    60   Input ~ 0
-XV4
-Wire Wire Line
-	2300 3150 2700 3150
-Wire Wire Line
-	2300 3050 2700 3050
-Wire Wire Line
-	2300 2950 2700 2950
+	1250 2750 2700 2750
+Wire Wire Line
+	1250 2650 2700 2650
+Wire Wire Line
+	1700 2450 2700 2450
+Wire Wire Line
+	1600 2250 2700 2250
+Wire Wire Line
+	1500 3150 2700 3150
+Wire Wire Line
+	1600 3050 2700 3050
+Wire Wire Line
+	1700 2950 2700 2950
 Wire Wire Line
 	2250 3450 2700 3450
@@
 -7V
 $Comp
-L C_Small C63
+L C_Small C36
 U 1 1 557B0E82
 P 2350 3600
-F 0 "C63" H 2360 3670 50  0000 L CNN
+F 0 "C36" H 2360 3670 50  0000 L CNN
 F 1 "0.1u" H 2360 3520 50  0000 L CNN
 F 2 "w_smd_cap:c_0603" H 2350 3600 60  0001 C CNN
@@
 12V
 $Comp
-L C_Small C64
+L C_Small C37
 U 1 1 557B0EEE
 P 2600 4050
-F 0 "C64" H 2610 4120 50  0000 L CNN
+F 0 "C37" H 2610 4120 50  0000 L CNN
 F 1 "0.1u" H 2610 3970 50  0000 L CNN
 F 2 "w_smd_cap:c_0603" H 2600 4050 60  0001 C CNN
@@
 Connection ~ 2600 4200
 $Comp
-L CP1_Small C65
+L CP1_Small C38
 U 1 1 557B105F
 P 4100 2250
-F 0 "C65" H 4110 2320 50  0000 L CNN
+F 0 "C38" H 4110 2320 50  0000 L CNN
 F 1 "1/35V" H 4110 2170 50  0000 L CNN
-F 2 "" H 4100 2250 60  0001 C CNN
+F 2 "w_smd_cap:c_0805" H 4100 2250 60  0001 C CNN
 F 3 "" H 4100 2250 60  0000 C CNN
 	1    4100 2250
@@
 F 0 "D4" H 4300 2130 50  0000 L CNN
 F 1 "D" H 4200 1970 50  0000 L CNN
-F 2 "w_pth_diodes:diode_do41" V 4350 2050 60  0001 C CNN
+F 2 "w_smd_diode:sod123" V 4350 2050 60  0001 C CNN
 F 3 "" V 4350 2050 60  0000 C CNN
 	1    4350 2050
@@
 F 0 "R27" H 4380 2470 50  0000 L CNN
 F 1 "100k" H 4380 2410 50  0000 L CNN
-F 2 "w_smd_resistors:r_0603" H 4350 2450 60  0001 C CNN
+F 2 "w_smd_resistors:r_0805" H 4350 2450 60  0001 C CNN
 F 3 "" H 4350 2450 60  0000 C CNN
 	1    4350 2450
@@
 VT1
 $Comp
-L C_Small C66
+L C_Small C39
 U 1 1 557B1301
 P 4650 2250
-F 0 "C66" H 4660 2320 50  0000 L CNN
+F 0 "C39" H 4660 2320 50  0000 L CNN
 F 1 "0.1u" H 4660 2170 50  0000 L CNN
 F 2 "w_smd_cap:c_0603" H 4650 2250 60  0001 C CNN
@@
 $EndComp
 Wire Wire Line
-	4750 2250 5250 2250
-$Comp
-L C_Small C67
+	4750 2250 5350 2250
+$Comp
+L C_Small C40
 U 1 1 557B1390
 P 4850 2450
-F 0 "C67" H 4860 2520 50  0000 L CNN
+F 0 "C40" H 4860 2520 50  0000 L CNN
 F 1 "2200pF" H 4860 2370 50  0000 L CNN
 F 2 "w_smd_cap:c_0603" H 4850 2450 60  0001 C CNN
@@
 F 0 "R28" H 5230 2470 50  0000 L CNN
 F 1 "1M0" H 5230 2410 50  0000 L CNN
-F 2 "w_smd_resistors:r_0603" H 5200 2450 60  0001 C CNN
+F 2 "w_smd_resistors:r_0805" H 5200 2450 60  0001 C CNN
 F 3 "" H 5200 2450 60  0000 C CNN
 	1    5200 2450
@@
 	5200 2650 5200 2550
 Connection ~ 4850 2650
-Wire Wire Line
-	5200 2250 5200 2350
 Text Label 8400 2800 0    60   ~ 0
 SUB
-Text Label 5250 2250 0    60   ~ 0
+Text Label 5350 2250 0    60   ~ 0
 SUB
 Text Label 7600 3800 3    60   ~ 0
@@
 	8400 2900 9200 2900
 $Comp
-L CP1_Small C74
+L CP1_Small C47
 U 1 1 557B16E0
 P 9000 3100
-F 0 "C74" H 9010 3170 50  0000 L CNN
+F 0 "C47" H 9010 3170 50  0000 L CNN
 F 1 "3.3/20V" H 9010 3020 50  0000 L CNN
-F 2 "" H 9000 3100 60  0001 C CNN
+F 2 "w_smd_cap:c_0805" H 9000 3100 60  0001 C CNN
 F 3 "" H 9000 3100 60  0000 C CNN
 	1    9000 3100
@@
 	6550 2300 6700 2300
 $Comp
-L C_Small C68
+L C_Small C41
 U 1 1 557B19FB
 P 6800 2300
-F 0 "C68" H 6810 2370 50  0000 L CNN
+F 0 "C41" H 6810 2370 50  0000 L CNN
 F 1 "0.1" H 6810 2220 50  0000 L CNN
 F 2 "w_smd_cap:c_0603" H 6800 2300 60  0001 C CNN
@@
 $EndComp
 $Comp
-L C_Small C69
+L C_Small C42
 U 1 1 557B1A55
 P 6800 3000
-F 0 "C69" H 6810 3070 50  0000 L CNN
+F 0 "C42" H 6810 3070 50  0000 L CNN
 F 1 "0.1" H 6810 2920 50  0000 L CNN
 F 2 "w_smd_cap:c_0603" H 6800 3000 60  0001 C CNN
@@
 12V
 $Comp
-L C_Small C70
+L C_Small C43
 U 1 1 557B1E47
 P 7050 1750
-F 0 "C70" H 7060 1820 50  0000 L CNN
+F 0 "C43" H 7060 1820 50  0000 L CNN
 F 1 "0.01" H 7060 1670 50  0000 L CNN
 F 2 "w_smd_cap:c_0603" H 7050 1750 60  0001 C CNN
@@
 $EndComp
 $Comp
-L CP1_Small C71
+L CP1_Small C44
 U 1 1 557B1EB1
 P 7250 1750
-F 0 "C71" H 7260 1820 50  0000 L CNN
+F 0 "C44" H 7260 1820 50  0000 L CNN
 F 1 "3.3/20V" H 7260 1670 50  0000 L CNN
-F 2 "" H 7250 1750 60  0001 C CNN
+F 2 "w_smd_cap:c_0805" H 7250 1750 60  0001 C CNN
 F 3 "" H 7250 1750 60  0000 C CNN
 	1    7250 1750
@@
 12V
 $Comp
-L CP1_Small C73
+L CP1_Small C46
 U 1 1 557B2356
 P 8200 1750
-F 0 "C73" H 8210 1820 50  0000 L CNN
+F 0 "C46" H 8210 1820 50  0000 L CNN
 F 1 "3.3/20V" H 8210 1670 50  0000 L CNN
-F 2 "" H 8200 1750 60  0001 C CNN
+F 2 "w_smd_cap:c_0805" H 8200 1750 60  0001 C CNN
 F 3 "" H 8200 1750 60  0000 C CNN
 	1    8200 1750
@@
 $EndComp
 $Comp
-L C_Small C72
+L C_Small C45
 U 1 1 557B23B2
 P 8000 1750
-F 0 "C72" H 8010 1820 50  0000 L CNN
+F 0 "C45" H 8010 1820 50  0000 L CNN
 F 1 "0.01" H 8010 1670 50  0000 L CNN
-F 2 "w_smd_cap:c_0603" H 8000 1750 60  0001 C CNN
+F 2 "w_smd_cap:c_0805" H 8000 1750 60  0001 C CNN
 F 3 "" H 8000 1750 60  0000 C CNN
 	1    8000 1750
@@
 	9200 2550 8400 2550
 Wire Wire Line
-	2700 1200 2450 1200
-Text HLabel 2450 1200 0    60   Input ~ 0
+	2700 1000 2250 1000
+Text HLabel 2250 1000 0    60   Input ~ 0
 12V
-Text HLabel 2450 1350 0    60   Input ~ 0
+Text HLabel 2250 1350 0    60   Input ~ 0
 -7V
-Text HLabel 2450 1500 0    60   Input ~ 0
-GND
-Wire Wire Line
-	2450 1350 2700 1350
-Wire Wire Line
-	2450 1500 2700 1500
-Text Label 2700 1350 0    60   ~ 0
+Text HLabel 2250 1700 0    60   Input ~ 0
+GND
+Wire Wire Line
+	2250 1350 2700 1350
+Wire Wire Line
+	2250 1700 2700 1700
+Text Label 2300 1350 0    60   ~ 0
 -7V
-Text Label 2700 1500 0    60   ~ 0
-GND
+Text Label 2300 1700 0    60   ~ 0
+GND
+$Comp
+L PWR_FLAG #FLG05
+U 1 1 557FC97D
+P 2700 1000
+F 0 "#FLG05" H 2700 1095 50  0001 C CNN
+F 1 "PWR_FLAG" H 2700 1180 50  0000 C CNN
+F 2 "" H 2700 1000 60  0000 C CNN
+F 3 "" H 2700 1000 60  0000 C CNN
+	1    2700 1000
+	-1   0    0    1
+$EndComp
 $Comp
 L PWR_FLAG #FLG06
-U 1 1 557FC97D
-P 2700 1200
-F 0 "#FLG06" H 2700 1295 50  0001 C CNN
-F 1 "PWR_FLAG" H 2700 1380 50  0000 C CNN
-F 2 "" H 2700 1200 60  0000 C CNN
-F 3 "" H 2700 1200 60  0000 C CNN
-	1    2700 1200
-	1    0    0    -1
-$EndComp
-$Comp
-L PWR_FLAG #FLG07
 U 1 1 557FC9B3
 P 2700 1350
-F 0 "#FLG07" H 2700 1445 50  0001 C CNN
+F 0 "#FLG06" H 2700 1445 50  0001 C CNN
 F 1 "PWR_FLAG" H 2700 1530 50  0000 C CNN
 F 2 "" H 2700 1350 60  0000 C CNN
 F 3 "" H 2700 1350 60  0000 C CNN
 	1    2700 1350
-	1    0    0    -1
-$EndComp
+	-1   0    0    1
+$EndComp
+$Comp
+L PWR_FLAG #FLG07
+U 1 1 557FC9E9
+P 2700 1700
+F 0 "#FLG07" H 2700 1795 50  0001 C CNN
+F 1 "PWR_FLAG" H 2700 1880 50  0000 C CNN
+F 2 "" H 2700 1700 60  0000 C CNN
+F 3 "" H 2700 1700 60  0000 C CNN
+	1    2700 1700
+	-1   0    0    1
+$EndComp
+Text HLabel 3250 1000 0    60   Input ~ 0
+5V0
+Wire Wire Line
+	3250 1000 3600 1000
+Text Label 3600 1000 0    60   ~ 0
+5V0
 $Comp
 L PWR_FLAG #FLG08
-U 1 1 557FC9E9
-P 2700 1500
-F 0 "#FLG08" H 2700 1595 50  0001 C CNN
-F 1 "PWR_FLAG" H 2700 1680 50  0000 C CNN
-F 2 "" H 2700 1500 60  0000 C CNN
-F 3 "" H 2700 1500 60  0000 C CNN
-	1    2700 1500
-	1    0    0    -1
-$EndComp
-Text HLabel 3300 1200 0    60   Input ~ 0
-5V0
-Wire Wire Line
-	3300 1200 3500 1200
-Text Label 3500 1200 0    60   ~ 0
-5V0
-$Comp
-L PWR_FLAG #FLG09
 U 1 1 557FCCCA
-P 3500 1200
-F 0 "#FLG09" H 3500 1295 50  0001 C CNN
-F 1 "PWR_FLAG" H 3500 1380 50  0000 C CNN
-F 2 "" H 3500 1200 60  0000 C CNN
-F 3 "" H 3500 1200 60  0000 C CNN
-	1    3500 1200
-	-1   0    0    1
-$EndComp
+P 3600 1000
+F 0 "#FLG08" H 3600 1095 50  0001 C CNN
+F 1 "PWR_FLAG" H 3600 1180 50  0000 C CNN
+F 2 "" H 3600 1000 60  0000 C CNN
+F 3 "" H 3600 1000 60  0000 C CNN
+	1    3600 1000
+	-1   0    0    1
+$EndComp
+Wire Wire Line
+	5200 2250 5200 2350
+Connection ~ 5200 2250
+$Comp
+L CONN_01X08 P2
+U 1 1 557D9F8F
+P 1050 2800
+F 0 "P2" H 1050 3250 50  0000 C CNN
+F 1 "CONN_01X08" V 1150 2800 50  0000 C CNN
+F 2 "w_smd_strip:bb02-hp08" H 1050 2800 60  0001 C CNN
+F 3 "" H 1050 2800 60  0000 C CNN
+	1    1050 2800
+	-1   0    0    -1
+$EndComp
+Wire Wire Line
+	1250 2450 1600 2450
+Wire Wire Line
+	1600 2450 1600 2250
+Wire Wire Line
+	1250 2550 1700 2550
+Wire Wire Line
+	1700 2550 1700 2450
+Wire Wire Line
+	1250 2850 1700 2850
+Wire Wire Line
+	1700 2850 1700 2950
+Wire Wire Line
+	1250 2950 1600 2950
+Wire Wire Line
+	1600 2950 1600 3050
+Wire Wire Line
+	1250 3050 1500 3050
+Wire Wire Line
+	1500 3050 1500 3150
+Wire Wire Line
+	1250 3150 1400 3150
+Wire Wire Line
+	1400 3150 1400 3300
+Text Label 1400 3300 0    60   ~ 0
+GND
 $EndSCHEMATC

Commit message: More work on schematic
Parts:
- removed P2: CONN_01X08, w_smd_strip:bb02-hp08, symbol CONN_01X08
- C39: value 0.1u -> 0.1uF
- C40: value 2200pF -> 2.2uF
Connections:
- net labels added: XSGV2, XSGV3, XSHT, XV1, XV2, XV3, XV4
- wire segments 78 -> 66
Changed lines of the file:
@@
 EESchema Schematic File Version 2
+LIBS:AstroCam-rescue
 LIBS:power
 LIBS:device
@@
 GND
 Wire Wire Line
-	1250 2750 2700 2750
-Wire Wire Line
-	1250 2650 2700 2650
-Wire Wire Line
-	1700 2450 2700 2450
+	1600 2450 2700 2450
 Wire Wire Line
 	1600 2250 2700 2250
 Wire Wire Line
-	1500 3150 2700 3150
+	1600 3150 2700 3150
 Wire Wire Line
 	1600 3050 2700 3050
 Wire Wire Line
-	1700 2950 2700 2950
+	1600 2950 2700 2950
 Wire Wire Line
 	2250 3450 2700 3450
@@
 GND
 Text Label 3900 2550 0    60   ~ 0
-VT4
+VT2
 NoConn ~ 3900 2750
 Text Label 3900 2850 0    60   ~ 0
 VT3
 Text Label 3900 3050 0    60   ~ 0
-VT2
+VT1
 Text Label 3900 3150 0    60   ~ 0
-VT1
+VT4
 $Comp
 L C_Small C39
@@
 P 4650 2250
 F 0 "C39" H 4660 2320 50  0000 L CNN
-F 1 "0.1u" H 4660 2170 50  0000 L CNN
+F 1 "0.1uF" H 4660 2170 50  0000 L CNN
 F 2 "w_smd_cap:c_0603" H 4650 2250 60  0001 C CNN
 F 3 "" H 4650 2250 60  0000 C CNN
@@
 P 4850 2450
 F 0 "C40" H 4860 2520 50  0000 L CNN
-F 1 "2200pF" H 4860 2370 50  0000 L CNN
+F 1 "2.2uF" H 4860 2370 50  0000 L CNN
 F 2 "w_smd_cap:c_0603" H 4850 2450 60  0001 C CNN
 F 3 "" H 4850 2450 60  0000 C CNN
@@
 GND
 $Comp
-L PWR_FLAG #FLG05
+L PWR_FLAG #FLG5
 U 1 1 557FC97D
 P 2700 1000
-F 0 "#FLG05" H 2700 1095 50  0001 C CNN
+F 0 "#FLG5" H 2700 1095 50  0001 C CNN
 F 1 "PWR_FLAG" H 2700 1180 50  0000 C CNN
 F 2 "" H 2700 1000 60  0000 C CNN
@@
 $EndComp
 $Comp
-L PWR_FLAG #FLG06
+L PWR_FLAG #FLG6
 U 1 1 557FC9B3
 P 2700 1350
-F 0 "#FLG06" H 2700 1445 50  0001 C CNN
+F 0 "#FLG6" H 2700 1445 50  0001 C CNN
 F 1 "PWR_FLAG" H 2700 1530 50  0000 C CNN
 F 2 "" H 2700 1350 60  0000 C CNN
@@
 $EndComp
 $Comp
-L PWR_FLAG #FLG07
+L PWR_FLAG #FLG7
 U 1 1 557FC9E9
 P 2700 1700
-F 0 "#FLG07" H 2700 1795 50  0001 C CNN
+F 0 "#FLG7" H 2700 1795 50  0001 C CNN
 F 1 "PWR_FLAG" H 2700 1880 50  0000 C CNN
 F 2 "" H 2700 1700 60  0000 C CNN
@@
 5V0
 $Comp
-L PWR_FLAG #FLG08
+L PWR_FLAG #FLG8
 U 1 1 557FCCCA
 P 3600 1000
-F 0 "#FLG08" H 3600 1095 50  0001 C CNN
+F 0 "#FLG8" H 3600 1095 50  0001 C CNN
 F 1 "PWR_FLAG" H 3600 1180 50  0000 C CNN
 F 2 "" H 3600 1000 60  0000 C CNN
@@
 	5200 2250 5200 2350
 Connection ~ 5200 2250
-$Comp
-L CONN_01X08 P2
-U 1 1 557D9F8F
-P 1050 2800
-F 0 "P2" H 1050 3250 50  0000 C CNN
-F 1 "CONN_01X08" V 1150 2800 50  0000 C CNN
-F 2 "w_smd_strip:bb02-hp08" H 1050 2800 60  0001 C CNN
-F 3 "" H 1050 2800 60  0000 C CNN
-	1    1050 2800
-	-1   0    0    -1
-$EndComp
-Wire Wire Line
-	1250 2450 1600 2450
-Wire Wire Line
-	1600 2450 1600 2250
-Wire Wire Line
-	1250 2550 1700 2550
-Wire Wire Line
-	1700 2550 1700 2450
-Wire Wire Line
-	1250 2850 1700 2850
-Wire Wire Line
-	1700 2850 1700 2950
-Wire Wire Line
-	1250 2950 1600 2950
-Wire Wire Line
-	1600 2950 1600 3050
-Wire Wire Line
-	1250 3050 1500 3050
-Wire Wire Line
-	1500 3050 1500 3150
-Wire Wire Line
-	1250 3150 1400 3150
-Wire Wire Line
-	1400 3150 1400 3300
-Text Label 1400 3300 0    60   ~ 0
-GND
+Wire Wire Line
+	1600 2750 2700 2750
+Text HLabel 1600 2250 0    60   Input ~ 0
+XSHT
+Text HLabel 1600 2450 0    60   Input ~ 0
+XV2
+Text HLabel 1600 2650 0    60   Input ~ 0
+XSGV2
+Wire Wire Line
+	1600 2650 2700 2650
+Text HLabel 1600 2750 0    60   Input ~ 0
+XV3
+Text HLabel 1600 2950 0    60   Input ~ 0
+XSGV3
+Text HLabel 1600 3050 0    60   Input ~ 0
+XV1
+Text HLabel 1600 3150 0    60   Input ~ 0
+XV4
 $EndSCHEMATC

Commit message: Work on proto breakout.
Parts:
- renumbered C36 to C26, C37 to C27, C38 to C28, C39 to C29, C40 to C30, C41 to C31, C42 to C32, C43 to C33, C44 to C34, C45 to C35, C46 to C36, C47 to C37, D4 to D2, R27 to R18, R28 to R19, U11 to U10, U10 to U9
Other:
- moved on the sheet: C26, C27, C28, C29, C30, D2, R18, R19, U9

Commit message: Lot's of back and forward with vendor.
Parts:
- added P10: CONN_01X14, w_pin_strip:pin_strip_14, symbol CONN_01X14
- added P11: CONN_01X12, w_pin_strip:pin_strip_12, symbol CONN_01X12
Connections:
- net labels added: RG_1, RG_2
- net labels removed: RG_A, RG_B
- wire segments 66 -> 62
Changed lines of the file:
@@
 Text Label 7850 1950 1    60   ~ 0
 GND
-Text Label 2350 1000 0    60   ~ 0
-12V
 Text Label 8400 2800 0    60   ~ 0
 SUB
@@
 Text Label 9200 2900 0    60   ~ 0
 -7V
-Text HLabel 6550 2300 0    60   Input ~ 0
-RG_A
-Text HLabel 6550 3000 0    60   Input ~ 0
-RG_B
 Wire Wire Line
 	6550 2300 6700 2300
@@
 Wire Wire Line
 	6900 2300 7050 2300
-Text HLabel 6550 2400 0    60   Input ~ 0
-LH1_1
-Text HLabel 6550 2500 0    60   Input ~ 0
-H1S_1
-Text HLabel 6550 2600 0    60   Input ~ 0
-H1T_1
-Text HLabel 6550 2700 0    60   Input ~ 0
-H2S_1
-Text HLabel 6550 2800 0    60   Input ~ 0
-H2T_1
 Wire Wire Line
 	6550 2400 7050 2400
@@
 Wire Wire Line
 	6550 2800 7050 2800
-Text HLabel 6550 3100 0    60   Input ~ 0
-LH1_2
-Text HLabel 6550 3200 0    60   Input ~ 0
-H1S_2
-Text HLabel 6550 3300 0    60   Input ~ 0
-H1T_2
-Text HLabel 6550 3400 0    60   Input ~ 0
-H2S_2
-Text HLabel 6550 3500 0    60   Input ~ 0
-H2T_2
 Wire Wire Line
 	6550 3100 7050 3100
@@
 Wire Wire Line
 	8400 2400 9200 2400
-Text HLabel 9200 2400 2    60   Input ~ 0
-CCD_OUT1
-Text HLabel 9200 2550 2    60   Input ~ 0
-CCD_OUT2
 Wire Wire Line
 	9200 2550 8400 2550
 Wire Wire Line
-	2700 1000 2250 1000
-Text HLabel 2250 1000 0    60   Input ~ 0
-12V
-Text HLabel 2250 1350 0    60   Input ~ 0
--7V
-Text HLabel 2250 1700 0    60   Input ~ 0
-GND
-Wire Wire Line
-	2250 1350 2700 1350
-Wire Wire Line
-	2250 1700 2700 1700
-Text Label 2300 1350 0    60   ~ 0
--7V
-Text Label 2300 1700 0    60   ~ 0
-GND
-Text HLabel 3250 1000 0    60   Input ~ 0
-5V0
-Wire Wire Line
-	3250 1000 3600 1000
-Text Label 3600 1000 0    60   ~ 0
-5V0
-Text HLabel 1600 4050 0    60   Input ~ 0
-XV4
-Text HLabel 1600 3950 0    60   Input ~ 0
-XV1
-Text HLabel 1600 3850 0    60   Input ~ 0
-XSGV3
-Text HLabel 1600 3650 0    60   Input ~ 0
-XV3
-Wire Wire Line
 	1600 3550 2700 3550
-Text HLabel 1600 3550 0    60   Input ~ 0
-XSGV2
-Text HLabel 1600 3350 0    60   Input ~ 0
-XV2
-Text HLabel 1600 3150 0    60   Input ~ 0
-XSHT
 Wire Wire Line
 	1600 3650 2700 3650
@@
 	1    0    0    -1
 $EndComp
+Text Label 1850 3150 0    60   ~ 0
+XSHT
+Text Label 1850 3350 0    60   ~ 0
+XV2
+Text Label 1850 3550 0    60   ~ 0
+XSGV2
+Text Label 1850 3650 0    60   ~ 0
+XV3
+Text Label 1850 3850 0    60   ~ 0
+XSGV3
+Text Label 1850 3950 0    60   ~ 0
+XV1
+Text Label 1850 4050 0    60   ~ 0
+XV4
+Text Label 8800 2400 0    60   ~ 0
+CCD_OUT1
+Text Label 8750 2550 0    60   ~ 0
+CCD_OUT2
+Text Label 6550 2300 0    60   ~ 0
+RG_1
+Text Label 6550 2400 0    60   ~ 0
+LH1_1
+Text Label 6550 2500 0    60   ~ 0
+H1S_1
+Text Label 6550 2600 0    60   ~ 0
+H1T_1
+Text Label 6550 2700 0    60   ~ 0
+H2S_1
+Text Label 6550 2800 0    60   ~ 0
+H2T_1
+Text Label 6550 3000 0    60   ~ 0
+RG_2
+Text Label 6550 3100 0    60   ~ 0
+LH1_2
+Text Label 6550 3200 0    60   ~ 0
+H1S_2
+Text Label 6550 3300 0    60   ~ 0
+H1T_2
+Text Label 6550 3400 0    60   ~ 0
+H2S_2
+Text Label 6550 3500 0    60   ~ 0
+H2T_2
+Text Label 4650 750  0    60   ~ 0
+12V
+Text Label 4650 850  0    60   ~ 0
+-7V
+Text Label 4650 950  0    60   ~ 0
+GND
+Text Label 4650 1050 0    60   ~ 0
+5V0
+Text Label 4650 1650 0    60   ~ 0
+XSHT
+Text Label 4650 1250 0    60   ~ 0
+XV1
+Text Label 4650 1350 0    60   ~ 0
+XV2
+Text Label 4650 1450 0    60   ~ 0
+XV3
+Text Label 4650 1550 0    60   ~ 0
+XV4
+Text Label 4650 1750 0    60   ~ 0
+XSGV2
+Text Label 4650 1850 0    60   ~ 0
+XSGV3
+Text Label 4650 1950 0    60   ~ 0
+CCD_OUT1
+Text Label 4650 1150 0    60   ~ 0
+CCD_OUT2
+Text Label 5700 750  0    60   ~ 0
+RG_1
+Text Label 5700 850  0    60   ~ 0
+LH1_1
+Text Label 5700 950  0    60   ~ 0
+H1S_1
+Text Label 5700 1050 0    60   ~ 0
+H1T_1
+Text Label 5700 1150 0    60   ~ 0
+H2S_1
+Text Label 5700 1250 0    60   ~ 0
+H2T_1
+Text Label 5700 1850 0    60   ~ 0
+RG_2
+Text Label 5700 1750 0    60   ~ 0
+LH1_2
+Text Label 5700 1650 0    60   ~ 0
+H1S_2
+Text Label 5700 1550 0    60   ~ 0
+H1T_2
+Text Label 5700 1450 0    60   ~ 0
+H2S_2
+Text Label 5700 1350 0    60   ~ 0
+H2T_2
+$Comp
+L CONN_01X12 P11
+U 1 1 5584CDCA
+P 5500 1300
+F 0 "P11" H 5500 1950 50  0000 C CNN
+F 1 "CONN_01X12" V 5600 1300 50  0000 C CNN
+F 2 "w_pin_strip:pin_strip_12" H 5500 1300 60  0001 C CNN
+F 3 "" H 5500 1300 60  0000 C CNN
+	1    5500 1300
+	-1   0    0    -1
+$EndComp
+$Comp
+L CONN_01X14 P10
+U 1 1 5584CE51
+P 4450 1400
+F 0 "P10" H 4450 2150 50  0000 C CNN
+F 1 "CONN_01X14" V 4550 1400 50  0000 C CNN
+F 2 "w_pin_strip:pin_strip_14" H 4450 1400 60  0001 C CNN
+F 3 "" H 4450 1400 60  0000 C CNN
+	1    4450 1400
+	-1   0    0    -1
+$EndComp
+Text Label 4650 2050 0    60   ~ 0
+GND
 $EndSCHEMATC

Commit message: more work
Parts:
- added C? (x2): 0.1u, symbol C
- added C?: 1.0u, symbol C
- added Q1, Q3: 2SC5095, w_smd_trans:sot323, symbol Q_NPN_BEC
- added Q2, Q4: MT3S20TU, w_smd_trans:sot323, symbol Q_NPN_BEC
- added R10, R11, R14, R15: 10K, w_smd_resistors:r_0805, symbol R
- added R12, R20: 1.17K, w_smd_resistors:r_0805, symbol R
- added R13, R21: 1.74K, w_smd_resistors:r_0805, symbol R
- added R? (x2): R, symbol R
- added U?: SN74LVC8T245, symbol SN74LVC8T245
- C28: value 1/35V -> 1u/35V
- C30: value 2.2uF -> 2200pF
Connections:
- net labels added: 3V3, B1, B2, E1, E2, H1, H2, H3, H4, HL1, HL2, RG1, RG2, VOUT1, VOUT2
- wire segments 62 -> 149
Other:
- moved on the sheet: C26, C27, C28, C29, C30, C31, C32, D2, R18, R19, U9

Commit message: lots of work
Parts:
- removed C?: 1.0u, symbol C
- removed P11: CONN_01X12, w_pin_strip:pin_strip_12, symbol CONN_01X12
- removed R?: R, symbol R
- removed U?: SN74LVC8T245, symbol SN74LVC8T245
- added P4: CONN_01X04, Socket_Strips:Socket_Strip_Straight_1x04, symbol CONN_01X04
- added P5: CONN_01X01, Socket_Strips:Socket_Strip_Straight_1x01, symbol CONN_01X01
- added U4: TXB0104, Housings_SSOP:TSSOP-14_4.4x5mm_Pitch0.65mm, symbol TXB0104
- C12, C13: renamed from C?; footprint (none) -> Capacitors_SMD:C_0603
- C26, C27, C29, C30, C31, C32, C33: footprint w_smd_cap:c_0603 -> Capacitors_SMD:C_0603
- C28, C34, C36, C37: footprint w_smd_cap:c_0805 -> Capacitors_SMD:c_elec_4x5.3
- C35: footprint w_smd_cap:c_0805 -> Capacitors_SMD:C_0603
- D2: footprint w_smd_diode:sod123 -> Diodes_SMD:SOD-123
- P10: footprint w_pin_strip:pin_strip_14 -> Pin_Headers:Pin_Header_Straight_1x14
- R10, R11, R12, R13, R14, R15, R18, R19, R20, R21: footprint w_smd_resistors:r_0805 -> Resistors_SMD:R_0603_HandSoldering
- R22: renamed from R?; value R -> 10.0k; footprint (none) -> Resistors_SMD:R_0603_HandSoldering
Connections:
- net labels added: ENH, HL, OH1, OH2, OHL, ORG, RG
- net labels removed: H3, H4, HL1, HL2, RG1, RG2
- wire segments 149 -> 107
Other:
- moved on the sheet: C12, C13, C26, C27, C28, C29, C30, C32, C35, C36, D2, R18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
