File: h-driver.sch (KiCad schematic (older format))
At the start: 14 parts, among them P3 CONN_02X12, U12 ADDI7013

Commit message: More work on schematic
Parts:
- added P2: CONN_01X24, camera:FFC-24-0.5mm, symbol CONN_01X24
- P3: footprint w_smd_strip:bb02-hp24 -> camera:FFC-24-0.5mm
Connections:
- net labels added: A0+, A0-, A1+, A1-, B0+, B0-, B1+, B1-, CLI, GP01, GP02, GP03, GP04, HD, SCK, SDATA, SL, SYNC, TCLK+, TCLK-, VD
- wire segments 84 -> 90
- no-connect marks 2 -> 0
Other:
- moved on the sheet: C54
Changed lines of the file:
@@
 EESchema Schematic File Version 2
+LIBS:AstroCam-rescue
 LIBS:power
 LIBS:device
@@
 U 1 1 557AD8F3
 P 2100 2200
+AR Path="/557AD8F3" Ref="U12"  Part="1"
+AR Path="/557AD230/557AD8F3" Ref="U12"  Part="1"
 F 0 "U12" H 2100 2950 60  0000 C CNN
 F 1 "ADDI7013" H 2100 2200 60  0000 C CNN
@@
 U 2 1 557B0AAF
 P 6450 2200
+AR Path="/557B0AAF" Ref="U12"  Part="2"
+AR Path="/557AD230/557B0AAF" Ref="U12"  Part="2"
 F 0 "U12" H 6450 2950 60  0000 C CNN
 F 1 "ADDI7013" H 6450 2200 60  0000 C CNN
@@
 U 3 1 557B0FDF
 P 2100 4550
+AR Path="/557B0FDF" Ref="U12"  Part="3"
+AR Path="/557AD230/557B0FDF" Ref="U12"  Part="3"
 F 0 "U12" H 2100 5300 60  0000 C CNN
 F 1 "ADDI7013" H 2100 4550 60  0000 C CNN
@@
 	1    0    0    -1
 $EndComp
-Text Label 3550 2750 0    60   ~ 0
+Text Label 3250 3100 0    60   ~ 0
 GND
 $Comp
-L C_Small C52
-U 1 1 557B2B4B
+L C_Small C54
+U 1 1 557B320A
 P 2150 6050
-F 0 "C52" H 2160 6120 50  0000 L CNN
+F 0 "C54" H 2160 6120 50  0000 L CNN
 F 1 "0.1uF" H 2160 5970 50  0000 L CNN
 F 2 "w_smd_cap:c_0603" H 2150 6050 60  0001 C CNN
 F 3 "" H 2150 6050 60  0000 C CNN
 	1    2150 6050
-	1    0    0    -1
-$EndComp
-$Comp
-L C_Small C54
-U 1 1 557B320A
-P 2450 6050
-F 0 "C54" H 2460 6120 50  0000 L CNN
-F 1 "0.1uF" H 2460 5970 50  0000 L CNN
-F 2 "w_smd_cap:c_0603" H 2450 6050 60  0001 C CNN
-F 3 "" H 2450 6050 60  0000 C CNN
-	1    2450 6050
 	1    0    0    -1
 $EndComp
@@
 F 3 "" H 2450 6500 60  0000 C CNN
 	1    2450 6500
-	-1   0    0    1
+	1    0    0    -1
 $EndComp
 Text Label 1450 5900 2    60   ~ 0
@@
 U 4 1 557B715D
 P 4950 4500
+AR Path="/557B715D" Ref="U12"  Part="4"
+AR Path="/557AD230/557B715D" Ref="U12"  Part="4"
 F 0 "U12" H 4950 5250 60  0000 C CNN
 F 1 "ADDI7013" H 4950 4500 60  0000 C CNN
@@
 Text Label 4950 5700 0    60   ~ 0
 GND
-Text Notes 4550 1550 0    60   ~ 0
+Text Notes 5350 1150 0    60   ~ 0
 Analog Differential \nPair Outputs
-Text Notes 3750 1450 0    60   ~ 0
+Text Notes 2800 1200 0    60   ~ 0
 Control\n
-Text HLabel 3250 2750 0    60   Input ~ 0
+Text HLabel 3250 3100 0    60   Input ~ 0
 GND
 $Comp
 L CONN_02X12 P3
 U 1 1 557AFA24
-P 4350 2200
-F 0 "P3" H 4350 2850 50  0000 C CNN
-F 1 "CONN_02X12" V 4350 2200 50  0000 C CNN
-F 2 "w_smd_strip:bb02-hp24" H 4350 1000 60  0001 C CNN
-F 3 "" H 4350 1000 60  0000 C CNN
-	1    4350 2200
+P 1000 1400
+F 0 "P3" H 1000 2050 50  0000 C CNN
+F 1 "CONN_02X12" V 1000 1400 50  0000 C CNN
+F 2 "camera:FFC-24-0.5mm" H 1000 200 60  0001 C CNN
+F 3 "" H 1000 200 60  0000 C CNN
+	1    1000 1400
 	1    0    0    1
 $EndComp
-NoConn ~ 4600 2350
-NoConn ~ 4600 2050
-Wire Wire Line
-	3250 2750 4100 2750
-Wire Wire Line
-	3550 2750 3550 2800
 Wire Wire Line
 	7150 1650 7500 1650
@@
 Wire Wire Line
 	1850 5900 1850 5950
+Connection ~ 1850 5900
 Wire Wire Line
 	2150 5900 2150 5950
-Connection ~ 1850 5900
-Wire Wire Line
-	2450 5900 2450 5950
+Wire Wire Line
+	2750 5900 2750 5950
 Connection ~ 2150 5900
-Wire Wire Line
-	2750 5900 2750 5950
-Connection ~ 2450 5900
 Wire Wire Line
 	3050 5900 3050 5950
@@
 	2750 6150 2750 6200
 Connection ~ 2750 6200
-Wire Wire Line
-	2450 6150 2450 6200
-Connection ~ 2450 6200
 Wire Wire Line
 	2150 6150 2150 6200
@@
 Connection ~ 4850 5400
 Wire Wire Line
-	5650 5400 5650 3900
+	5650 5400 5650 3850
 Connection ~ 5050 5400
-Connection ~ 5650 5100
-Connection ~ 5650 5000
-Connection ~ 5650 4900
-Connection ~ 5650 4800
-Connection ~ 5650 4700
-Connection ~ 5650 4600
-Connection ~ 5650 4500
-Connection ~ 5650 4400
-Connection ~ 5650 4300
-Connection ~ 5650 4200
-Connection ~ 5650 4100
-Connection ~ 5650 4000
+Connection ~ 5650 5050
+Connection ~ 5650 4950
+Connection ~ 5650 4850
+Connection ~ 5650 4750
+Connection ~ 5650 4650
+Connection ~ 5650 4550
+Connection ~ 5650 4450
+Connection ~ 5650 4350
+Connection ~ 5650 4250
+Connection ~ 5650 4150
+Connection ~ 5650 4050
+Connection ~ 5650 3950
 Wire Wire Line
 	4950 5400 4950 5700
 Connection ~ 4950 5400
 Wire Wire Line
-	4600 1650 5750 1650
-Wire Wire Line
-	4600 1750 5750 1750
-Wire Wire Line
-	4600 1850 5750 1850
-Wire Wire Line
-	4600 1950 5750 1950
-Wire Wire Line
-	4600 2150 5750 2150
-Wire Wire Line
-	4600 2250 5750 2250
-Wire Wire Line
-	4600 2450 5750 2450
-Wire Wire Line
-	4600 2550 5750 2550
-Wire Wire Line
-	4600 2650 5750 2650
-Wire Wire Line
-	4600 2750 5750 2750
-Wire Wire Line
-	2800 1650 4100 1650
-Wire Wire Line
-	2800 1750 4100 1750
-Wire Wire Line
-	2800 1850 4100 1850
-Wire Wire Line
-	2800 1950 4100 1950
-Wire Wire Line
-	2800 2050 4100 2050
-Wire Wire Line
-	2800 2200 3450 2200
-Wire Wire Line
-	3450 2200 3450 2150
-Wire Wire Line
-	3450 2150 4100 2150
-Wire Wire Line
-	2800 2300 3550 2300
-Wire Wire Line
-	3550 2300 3550 2250
-Wire Wire Line
-	3550 2250 4100 2250
-Wire Wire Line
-	2800 2400 3650 2400
-Wire Wire Line
-	3650 2400 3650 2350
-Wire Wire Line
-	3650 2350 4100 2350
-Wire Wire Line
-	2800 2550 2950 2550
-Wire Wire Line
-	2950 2550 2950 2500
-Wire Wire Line
-	2950 2500 3750 2500
-Wire Wire Line
-	3750 2500 3750 2450
-Wire Wire Line
-	3750 2450 4100 2450
-Wire Wire Line
-	2800 2650 2900 2650
-Wire Wire Line
-	2900 2650 2900 2600
-Wire Wire Line
-	2900 2600 3050 2600
-Wire Wire Line
-	3050 2600 3050 2550
-Wire Wire Line
-	3050 2550 4100 2550
-Wire Wire Line
-	2800 2750 2800 2700
-Wire Wire Line
-	2800 2700 2950 2700
-Wire Wire Line
-	2950 2700 2950 2650
-Wire Wire Line
-	2950 2650 4100 2650
+	2800 2550 3700 2550
+Wire Wire Line
+	2800 2650 3800 2650
+Connection ~ 5650 5150
+$Comp
+L CONN_01X24 P2
+U 1 1 557E7FB2
+P 4250 1300
+F 0 "P2" H 4250 2550 50  0000 C CNN
+F 1 "CONN_01X24" V 4350 1300 50  0000 C CNN
+F 2 "camera:FFC-24-0.5mm" V 4250 1300 60  0000 C CNN
+F 3 "" H 4250 1300 60  0000 C CNN
+	1    4250 1300
+	0    -1   -1   0
+$EndComp
+Wire Wire Line
+	2800 1650 3100 1650
+Wire Wire Line
+	3100 1650 3100 1500
+Wire Wire Line
+	2800 1750 3200 1750
+Wire Wire Line
+	3200 1750 3200 1500
+Wire Wire Line
+	2800 1850 3300 1850
+Wire Wire Line
+	3300 1850 3300 1500
+Wire Wire Line
+	2800 1950 3400 1950
+Wire Wire Line
+	3400 1950 3400 1500
+Wire Wire Line
+	2800 2050 3500 2050
+Wire Wire Line
+	3500 2050 3500 1500
+Wire Wire Line
+	3700 2550 3700 1500
+Wire Wire Line
+	3800 2650 3800 1500
+Wire Wire Line
+	2800 2750 3900 2750
+Wire Wire Line
+	3900 2750 3900 1500
+Wire Wire Line
+	2800 2200 4000 2200
+Wire Wire Line
+	4000 2200 4000 1500
+Wire Wire Line
+	2800 2300 4100 2300
+Wire Wire Line
+	4100 2300 4100 1500
+Wire Wire Line
+	2800 2400 4200 2400
+Wire Wire Line
+	4200 2400 4200 1500
+Wire Wire Line
+	3250 3100 5400 3100
+Wire Wire Line
+	3600 3100 3600 1500
+Wire Wire Line
+	4300 3100 4300 1500
+Connection ~ 3600 3100
+Wire Wire Line
+	5400 3100 5400 1500
+Connection ~ 4300 3100
+Wire Wire Line
+	5750 1650 4400 1650
+Wire Wire Line
+	4400 1650 4400 1500
+Wire Wire Line
+	5750 1750 4500 1750
+Wire Wire Line
+	4500 1750 4500 1500
+Wire Wire Line
+	5750 1850 4600 1850
+Wire Wire Line
+	4600 1850 4600 1500
+Wire Wire Line
+	5750 1950 4700 1950
+Wire Wire Line
+	4700 1950 4700 1500
+Wire Wire Line
+	5750 2150 4800 2150
+Wire Wire Line
+	4800 2150 4800 1500
+Wire Wire Line
+	5750 2250 4900 2250
+Wire Wire Line
+	4900 2250 4900 1500
+Wire Wire Line
+	5750 2450 5000 2450
+Wire Wire Line
+	5000 2450 5000 1500
+Wire Wire Line
+	5750 2550 5100 2550
+Wire Wire Line
+	5100 2550 5100 1500
+Wire Wire Line
+	5750 2650 5200 2650
+Wire Wire Line
+	5200 2650 5200 1500
+Wire Wire Line
+	5750 2750 5300 2750
+Wire Wire Line
+	5300 2750 5300 1500
+Text Label 5500 1650 0    60   ~ 0
+A0+
+Text Label 5500 1750 0    60   ~ 0
+A0-
+Text Label 5500 1850 0    60   ~ 0
+A1+
+Text Label 5500 1950 0    60   ~ 0
+A1-
+Text Label 5500 2150 0    60   ~ 0
+TCLK+
+Text Label 5500 2250 0    60   ~ 0
+TCLK-
+Text Label 5500 2450 0    60   ~ 0
+B0+
+Text Label 5500 2550 0    60   ~ 0
+B0-
+Text Label 5500 2650 0    60   ~ 0
+B1+
+Text Label 5500 2750 0    60   ~ 0
+B1-
+Text Label 2800 1650 0    60   ~ 0
+CLI
+Text Label 2800 1750 0    60   ~ 0
+GP01
+Text Label 2800 1850 0    60   ~ 0
+GP02
+Text Label 2800 1950 0    60   ~ 0
+GP03
+Text Label 2800 2050 0    60   ~ 0
+GP04
+Text Label 2800 2200 0    60   ~ 0
+SYNC
+Text Label 2800 2300 0    60   ~ 0
+VD
+Text Label 2800 2400 0    60   ~ 0
+HD
+Text Label 2800 2550 0    60   ~ 0
+SCK
+Text Label 2800 2650 0    60   ~ 0
+SDATA
+Text Label 2800 2750 0    60   ~ 0
+SL
+$Comp
+L C_Small C52
+U 1 1 557E9A62
+P 2450 6050
+F 0 "C52" H 2460 6120 50  0000 L CNN
+F 1 "0.1uF" H 2460 5970 50  0000 L CNN
+F 2 "w_smd_cap:c_0603" H 2450 6050 60  0001 C CNN
+F 3 "" H 2450 6050 60  0000 C CNN
+	1    2450 6050
+	1    0    0    -1
+$EndComp
+Wire Wire Line
+	2450 5950 2450 5900
+Connection ~ 2450 5900
+Wire Wire Line
+	2450 6150 2450 6200
+Connection ~ 2450 6200
 $EndSCHEMATC

Commit message: Work on proto breakout.
Parts:
- removed P2: CONN_01X24, camera:FFC-24-0.5mm, symbol CONN_01X24
- removed P3: CONN_02X12, camera:FFC-24-0.5mm, symbol CONN_02X12
- added P2: CONN_01X05, w_pin_strip:pin_strip_5, symbol CONN_01X05
- added P3: CONN_01X10, w_pin_strip:pin_strip_10, symbol CONN_01X10
- added P4, P6, P7: CONN_01X03, w_pin_strip:pin_strip_3, symbol CONN_01X03
- added P5: CONN_01X12, w_pin_strip:pin_strip_12, symbol CONN_01X12
- renumbered C48 to C38, C49 to C39, C50 to C40, C51 to C41, C54 to C42, C53 to C43, C52 to C44, C55 to C45, C56 to C46, C57 to C47, C58 to C48, C59 to C49, U12 to U11
Connections:
- net labels added: IN_A+, IN_A-, IN_B+, IN_B-
- net labels removed: INPA+, INPA-, INPB+, INPB-
- wire segments 90 -> 86

Commit message: Lot's of back and forward with vendor.
Connections:
- wire segments 86 -> 89
Other:
- moved on the sheet: P5, P7
Changed lines of the file:
@@
 	1    0    0    -1
 $EndComp
-Text Label 6500 3500 0    60   ~ 0
+Text Label 3600 4350 0    60   ~ 0
 GND
 $Comp
@@
 Text Label 7200 2800 0    60   ~ 0
 IN_B-
-Text Label 6500 3600 0    60   ~ 0
-3V3
-Text Label 6500 3700 0    60   ~ 0
-1V8
-Text Label 7950 4350 2    60   ~ 0
+Text Label 3600 4450 0    60   ~ 0
+3V3
+Text Label 3600 4550 0    60   ~ 0
+1V8
+Text Label 9450 2600 2    60   ~ 0
 H1
-Text Label 7950 4250 2    60   ~ 0
+Text Label 9450 2500 2    60   ~ 0
 H2
-Text Label 7950 4150 2    60   ~ 0
+Text Label 9450 2400 2    60   ~ 0
 H3
-Text Label 7950 4050 2    60   ~ 0
+Text Label 9450 2300 2    60   ~ 0
 H4
-Text Label 7950 4450 2    60   ~ 0
+Text Label 9450 2700 2    60   ~ 0
 HL1
-Text Label 7950 3950 2    60   ~ 0
+Text Label 9450 2200 2    60   ~ 0
 HL2
-Text Label 7950 4550 2    60   ~ 0
+Text Label 9450 2800 2    60   ~ 0
 RG1
-Text Label 7950 3850 2    60   ~ 0
+Text Label 9450 2100 2    60   ~ 0
 RG2
-Text Label 7950 3550 2    60   ~ 0
+Text Label 9450 1800 2    60   ~ 0
 IN_A+
-Text Label 7950 3450 2    60   ~ 0
+Text Label 9450 1700 2    60   ~ 0
 IN_A-
-Text Label 7950 3650 2    60   ~ 0
+Text Label 9450 1900 2    60   ~ 0
 IN_B+
-Text Label 7950 3750 2    60   ~ 0
+Text Label 9450 2000 2    60   ~ 0
 IN_B-
 $Comp
 L CONN_01X12 P5
 U 1 1 55801ABA
-P 8150 4000
-F 0 "P5" H 8150 4650 50  0000 C CNN
-F 1 "CONN_01X12" V 8250 4000 50  0000 C CNN
-F 2 "w_pin_strip:pin_strip_12" H 8150 4000 60  0001 C CNN
-F 3 "" H 8150 4000 60  0000 C CNN
-	1    8150 4000
+P 9650 2250
+F 0 "P5" H 9650 2900 50  0000 C CNN
+F 1 "CONN_01X12" V 9750 2250 50  0000 C CNN
+F 2 "w_pin_strip:pin_strip_12" H 9650 2250 60  0001 C CNN
+F 3 "" H 9650 2250 60  0000 C CNN
+	1    9650 2250
 	1    0    0    -1
 $EndComp
@@
 L CONN_01X03 P7
 U 1 1 55802F4C
-P 6300 3600
-F 0 "P7" H 6300 3800 50  0000 C CNN
-F 1 "CONN_01X03" V 6400 3600 50  0000 C CNN
-F 2 "w_pin_strip:pin_strip_3" H 6300 3600 60  0001 C CNN
-F 3 "" H 6300 3600 60  0000 C CNN
-	1    6300 3600
+P 3400 4450
+F 0 "P7" H 3400 4650 50  0000 C CNN
+F 1 "CONN_01X03" V 3500 4450 50  0000 C CNN
+F 2 "w_pin_strip:pin_strip_3" H 3400 4450 60  0001 C CNN
+F 3 "" H 3400 4450 60  0000 C CNN
+	1    3400 4450
 	-1   0    0    1
 $EndComp
@@
 Wire Wire Line
 	2800 2400 4000 2400
+Text Label 6800 4600 0    60   ~ 0
+GND
+Text Label 6800 4200 0    60   ~ 0
+3V3
+Text Label 6800 5050 0    60   ~ 0
+1V8
+Wire Wire Line
+	6800 4600 6450 4600
+Wire Wire Line
+	6450 4200 6800 4200
+Wire Wire Line
+	6800 5050 6450 5050
+$Comp
+L PWR_FLAG #FLG04
+U 1 1 5580E99E
+P 6450 4600
+F 0 "#FLG04" H 6450 4695 50  0001 C CNN
+F 1 "PWR_FLAG" H 6450 4780 50  0000 C CNN
+F 2 "" H 6450 4600 60  0000 C CNN
+F 3 "" H 6450 4600 60  0000 C CNN
+	1    6450 4600
+	1    0    0    -1
+$EndComp
+$Comp
+L PWR_FLAG #FLG05
+U 1 1 5580E9DE
+P 6450 4200
+F 0 "#FLG05" H 6450 4295 50  0001 C CNN
+F 1 "PWR_FLAG" H 6450 4380 50  0000 C CNN
+F 2 "" H 6450 4200 60  0000 C CNN
+F 3 "" H 6450 4200 60  0000 C CNN
+	1    6450 4200
+	1    0    0    -1
+$EndComp
+$Comp
+L PWR_FLAG #FLG06
+U 1 1 5580EA1E
+P 6450 5050
+F 0 "#FLG06" H 6450 5145 50  0001 C CNN
+F 1 "PWR_FLAG" H 6450 5230 50  0000 C CNN
+F 2 "" H 6450 5050 60  0000 C CNN
+F 3 "" H 6450 5050 60  0000 C CNN
+	1    6450 5050
+	1    0    0    -1
+$EndComp
 $EndSCHEMATC

Commit message: more work
Parts:
- removed P2: CONN_01X05, w_pin_strip:pin_strip_5, symbol CONN_01X05
- removed P3: CONN_01X10, w_pin_strip:pin_strip_10, symbol CONN_01X10
- removed P4, P6, P7: CONN_01X03, w_pin_strip:pin_strip_3, symbol CONN_01X03
- removed P5: CONN_01X12, w_pin_strip:pin_strip_12, symbol CONN_01X12
- added P2, P3: CONN_01X18, w_pin_strip:pin_strip_18, symbol CONN_01X18
Connections:
- wire segments 89 -> 83
Changed lines of the file:
@@
 $Descr A4 11693 8268
 encoding utf-8
-Sheet 4 5
+Sheet 3 5
 Title ""
 Date ""
@@
 	1    0    0    -1
 $EndComp
-Text Label 3600 4350 0    60   ~ 0
+Text Label 10150 1350 2    60   ~ 0
 GND
 $Comp
@@
 Text Label 4950 5700 0    60   ~ 0
 GND
-Text Notes 4550 1100 0    60   ~ 0
+Text Notes 5750 1100 0    60   ~ 0
 Analog Differential \nPair Outputs
-Text Notes 3450 1050 0    60   ~ 0
+Text Notes 2200 1050 0    60   ~ 0
 Control\n
 Wire Wire Line
@@
 	4950 5400 4950 5700
 Connection ~ 4950 5400
-Wire Wire Line
-	2800 2550 3700 2550
-Wire Wire Line
-	2800 2650 3800 2650
 Connection ~ 5650 5150
 Wire Wire Line
-	2800 1650 3100 1650
-Wire Wire Line
-	3100 1650 3100 1500
-Wire Wire Line
-	2800 1750 3200 1750
-Wire Wire Line
-	3200 1750 3200 1500
-Wire Wire Line
-	2800 1850 3300 1850
-Wire Wire Line
-	3300 1850 3300 1500
-Wire Wire Line
-	2800 1950 3400 1950
-Wire Wire Line
-	3400 1950 3400 1500
-Wire Wire Line
-	2800 2050 3500 2050
-Wire Wire Line
-	3500 2050 3500 1500
-Wire Wire Line
-	2800 2750 3600 2750
-Wire Wire Line
-	2800 2200 4100 2200
-Wire Wire Line
-	5750 1650 4400 1650
-Wire Wire Line
-	4400 1650 4400 1500
-Wire Wire Line
-	5750 1750 4500 1750
-Wire Wire Line
-	4500 1750 4500 1500
-Wire Wire Line
-	5750 1850 4600 1850
-Wire Wire Line
-	4600 1850 4600 1500
-Wire Wire Line
-	5750 1950 4700 1950
-Wire Wire Line
-	4700 1950 4700 1500
-Wire Wire Line
-	5750 2150 4800 2150
-Wire Wire Line
-	4800 2150 4800 1500
-Wire Wire Line
-	5750 2250 4900 2250
-Wire Wire Line
-	4900 2250 4900 1500
-Wire Wire Line
-	5750 2450 5000 2450
-Wire Wire Line
-	5000 2450 5000 1500
-Wire Wire Line
-	5750 2550 5100 2550
-Wire Wire Line
-	5100 2550 5100 1500
-Wire Wire Line
-	5750 2650 5200 2650
-Wire Wire Line
-	5200 2650 5200 1500
-Wire Wire Line
-	5750 2750 5300 2750
-Wire Wire Line
-	5300 2750 5300 1500
+	2800 1650 3350 1650
+Wire Wire Line
+	3350 1650 3350 1350
+Wire Wire Line
+	2800 1750 3450 1750
+Wire Wire Line
+	3450 1750 3450 1350
+Wire Wire Line
+	2800 1850 3550 1850
+Wire Wire Line
+	3550 1850 3550 1350
+Wire Wire Line
+	2800 1950 3650 1950
+Wire Wire Line
+	3650 1950 3650 1350
+Wire Wire Line
+	2800 2050 3750 2050
+Wire Wire Line
+	3750 2050 3750 1350
+Wire Wire Line
+	2800 2200 5050 2200
+Wire Wire Line
+	5750 1650 3850 1650
+Wire Wire Line
+	3850 1650 3850 1350
+Wire Wire Line
+	5750 1750 3950 1750
+Wire Wire Line
+	3950 1750 3950 1350
+Wire Wire Line
+	5750 1850 4050 1850
+Wire Wire Line
+	4050 1850 4050 1350
+Wire Wire Line
+	5750 1950 4150 1950
+Wire Wire Line
+	4150 1950 4150 1350
+Wire Wire Line
+	5750 2150 4250 2150
+Wire Wire Line
+	4250 2150 4250 1350
+Wire Wire Line
+	5750 2250 4350 2250
+Wire Wire Line
+	4350 2250 4350 1350
+Wire Wire Line
+	5750 2450 4450 2450
+Wire Wire Line
+	4450 2450 4450 1350
+Wire Wire Line
+	5750 2550 4550 2550
+Wire Wire Line
+	4550 2550 4550 1350
+Wire Wire Line
+	5750 2650 4650 2650
+Wire Wire Line
+	4650 2650 4650 1350
+Wire Wire Line
+	5750 2750 4750 2750
+Wire Wire Line
+	4750 2750 4750 1350
 Text Label 5500 1650 0    60   ~ 0
 A0+
@@
 	2450 6150 2450 6200
 Connection ~ 2450 6200
-$Comp
-L CONN_01X10 P3
-U 1 1 558012C2
-P 4850 1300
-F 0 "P3" H 4850 1850 50  0000 C CNN
-F 1 "CONN_01X10" V 4950 1300 50  0000 C CNN
-F 2 "w_pin_strip:pin_strip_10" H 4850 1300 60  0001 C CNN
-F 3 "" H 4850 1300 60  0000 C CNN
-	1    4850 1300
-	0    -1   -1   0
-$EndComp
 Text Label 7200 1650 0    60   ~ 0
 H1
@@
 Text Label 7200 2800 0    60   ~ 0
 IN_B-
-Text Label 3600 4450 0    60   ~ 0
-3V3
-Text Label 3600 4550 0    60   ~ 0
-1V8
-Text Label 9450 2600 2    60   ~ 0
+Text Label 10150 1250 2    60   ~ 0
+3V3
+Text Label 10150 1150 2    60   ~ 0
+1V8
+Text Label 10150 2350 2    60   ~ 0
 H1
-Text Label 9450 2500 2    60   ~ 0
+Text Label 10150 2250 2    60   ~ 0
 H2
-Text Label 9450 2400 2    60   ~ 0
+Text Label 10150 2150 2    60   ~ 0
 H3
-Text Label 9450 2300 2    60   ~ 0
+Text Label 10150 2050 2    60   ~ 0
 H4
-Text Label 9450 2700 2    60   ~ 0
+Text Label 10150 2450 2    60   ~ 0
 HL1
-Text Label 9450 2200 2    60   ~ 0
+Text Label 10150 1950 2    60   ~ 0
 HL2
-Text Label 9450 2800 2    60   ~ 0
+Text Label 10150 2550 2    60   ~ 0
 RG1
-Text Label 9450 2100 2    60   ~ 0
+Text Label 10150 1850 2    60   ~ 0
 RG2
-Text Label 9450 1800 2    60   ~ 0
+Text Label 10150 1550 2    60   ~ 0
 IN_A+
-Text Label 9450 1700 2    60   ~ 0
+Text Label 10150 1450 2    60   ~ 0
 IN_A-
-Text Label 9450 1900 2    60   ~ 0
+Text Label 10150 1650 2    60   ~ 0
 IN_B+
-Text Label 9450 2000 2    60   ~ 0
+Text Label 10150 1750 2    60   ~ 0
 IN_B-
-$Comp
-L CONN_01X12 P5
-U 1 1 55801ABA
-P 9650 2250
-F 0 "P5" H 9650 2900 50  0000 C CNN
-F 1 "CONN_01X12" V 9750 2250 50  0000 C CNN
-F 2 "w_pin_strip:pin_strip_12" H 9650 2250 60  0001 C CNN
-F 3 "" H 9650 2250 60  0000 C CNN
-	1    9650 2250
-	1    0    0    -1
-$EndComp
-$Comp
-L CONN_01X05 P2
-U 1 1 55802A9E
-P 3300 1300
-F 0 "P2" H 3300 1600 50  0000 C CNN
-F 1 "CONN_01X05" V 3400 1300 50  0000 C CNN
-F 2 "w_pin_strip:pin_strip_5" H 3300 1300 60  0001 C CNN
-F 3 "" H 3300 1300 60  0000 C CNN
-	1    3300 1300
-	0    -1   -1   0
-$EndComp
-$Comp
-L CONN_01X03 P4
-U 1 1 55802B35
-P 3700 1650
-F 0 "P4" H 3700 1850 50  0000 C CNN
-F 1 "CONN_01X03" V 3800 1650 50  0000 C CNN
-F 2 "w_pin_strip:pin_strip_3" H 3700 1650 60  0001 C CNN
-F 3 "" H 3700 1650 60  0000 C CNN
-	1    3700 1650
-	0    -1   -1   0
-$EndComp
-Wire Wire Line
-	3600 2750 3600 1850
-Wire Wire Line
-	3700 2550 3700 1850
-Wire Wire Line
-	3800 2650 3800 1850
-$Comp
-L CONN_01X03 P6
-U 1 1 55802DCC
-P 4000 1300
-F 0 "P6" H 4000 1500 50  0000 C CNN
-F 1 "CONN_01X03" V 4100 1300 50  0000 C CNN
-F 2 "w_pin_strip:pin_strip_3" H 4000 1300 60  0001 C CNN
-F 3 "" H 4000 1300 60  0000 C CNN
-	1    4000 1300
-	0    -1   -1   0
-$EndComp
-$Comp
-L CONN_01X03 P7
-U 1 1 55802F4C
-P 3400 4450
-F 0 "P7" H 3400 4650 50  0000 C CNN
-F 1 "CONN_01X03" V 3500 4450 50  0000 C CNN
-F 2 "w_pin_strip:pin_strip_3" H 3400 4450 60  0001 C CNN
-F 3 "" H 3400 4450 60  0000 C CNN
-	1    3400 4450
-	-1   0    0    1
-$EndComp
-Wire Wire Line
-	3900 1500 3900 2300
-Wire Wire Line
-	4100 2200 4100 1500
-Wire Wire Line
-	4000 2400 4000 1500
-Wire Wire Line
-	3900 2300 2800 2300
-Wire Wire Line
-	2800 2400 4000 2400
+Wire Wire Line
+	4850 1350 4850 2300
+Wire Wire Line
+	5050 2200 5050 1350
+Wire Wire Line
+	4950 2400 4950 1350
+Wire Wire Line
+	4850 2300 2800 2300
+Wire Wire Line
+	2800 2400 4950 2400
 Text Label 6800 4600 0    60   ~ 0
 GND
@@
 	1    0    0    -1
 $EndComp
+$Comp
+L CONN_01X18 P3
+U 1 1 55886037
+P 10350 2000
+F 0 "P3" H 10350 2950 50  0000 C CNN
+F 1 "CONN_01X18" V 10450 2000 50  0000 C CNN
+F 2 "w_pin_strip:pin_strip_18" H 10350 2000 60  0001 C CNN
+F 3 "" H 10350 2000 60  0000 C CNN
+	1    10350 2000
+	1    0    0    -1
+$EndComp
+Text Label 10150 2650 2    60   ~ 0
+SL
+Text Label 10150 2850 2    60   ~ 0
+SDATA
+Text Label 10150 2750 2    60   ~ 0
+SCK
+$Comp
+L CONN_01X18 P2
+U 1 1 5588671F
+P 4200 1150
+F 0 "P2" H 4200 2100 50  0000 C CNN
+F 1 "CONN_01X18" V 4300 1150 50  0000 C CNN
+F 2 "w_pin_strip:pin_strip_18" H 4200 1150 60  0001 C CNN
+F 3 "" H 4200 1150 60  0000 C CNN
+	1    4200 1150
+	0    -1   -1   0
+$EndComp
 $EndSCHEMATC
