File: h-driver.sch (KiCad schematic (older format))
At the start: 15 parts, among them P2 CONN_01X18, P3 CONN_01X18, U11 ADDI7013

Commit message: lots of work
Parts:
- C38, C39, C40, C41, C42, C43, C44, C45, C46, C47, C48, C49: footprint w_smd_cap:c_0603 -> Capacitors_SMD:C_0603_HandSoldering
- P2, P3: footprint w_pin_strip:pin_strip_18 -> Pin_Headers:Pin_Header_Straight_1x18
Changed lines of the file:
@@
 F 0 "C48" H 8225 2600 50  0000 L CNN
 F 1 "0.1u" H 8225 2400 50  0000 L CNN
-F 2 "w_smd_cap:c_0603" H 8238 2350 30  0001 C CNN
+F 2 "Capacitors_SMD:C_0603_HandSoldering" H 8238 2350 30  0001 C CNN
 F 3 "" H 8200 2500 60  0000 C CNN
 	1    8200 2500
@@
 F 0 "C49" H 8225 2800 50  0000 L CNN
 F 1 "0.1u" H 8225 2600 50  0000 L CNN
-F 2 "w_smd_cap:c_0603" H 8238 2550 30  0001 C CNN
+F 2 "Capacitors_SMD:C_0603_HandSoldering" H 8238 2550 30  0001 C CNN
 F 3 "" H 8200 2700 60  0000 C CNN
 	1    8200 2700
@@
 F 0 "C38" H 1560 6120 50  0000 L CNN
 F 1 "0.1uF" H 1560 5970 50  0000 L CNN
-F 2 "w_smd_cap:c_0603" H 1550 6050 60  0001 C CNN
+F 2 "Capacitors_SMD:C_0603_HandSoldering" H 1550 6050 60  0001 C CNN
 F 3 "" H 1550 6050 60  0000 C CNN
 	1    1550 6050
@@
 F 0 "C40" H 1860 6120 50  0000 L CNN
 F 1 "0.1uF" H 1860 5970 50  0000 L CNN
-F 2 "w_smd_cap:c_0603" H 1850 6050 60  0001 C CNN
+F 2 "Capacitors_SMD:C_0603_HandSoldering" H 1850 6050 60  0001 C CNN
 F 3 "" H 1850 6050 60  0000 C CNN
 	1    1850 6050
@@
 F 0 "C39" H 1560 6570 50  0000 L CNN
 F 1 "0.1uF" H 1560 6420 50  0000 L CNN
-F 2 "w_smd_cap:c_0603" H 1550 6500 60  0001 C CNN
+F 2 "Capacitors_SMD:C_0603_HandSoldering" H 1550 6500 60  0001 C CNN
 F 3 "" H 1550 6500 60  0000 C CNN
 	1    1550 6500
@@
 F 0 "C41" H 1860 6570 50  0000 L CNN
 F 1 "0.1uF" H 1860 6420 50  0000 L CNN
-F 2 "w_smd_cap:c_0603" H 1850 6500 60  0001 C CNN
+F 2 "Capacitors_SMD:C_0603_HandSoldering" H 1850 6500 60  0001 C CNN
 F 3 "" H 1850 6500 60  0000 C CNN
 	1    1850 6500
@@
 F 0 "C43" H 2160 6570 50  0000 L CNN
 F 1 "0.1uF" H 2160 6420 50  0000 L CNN
-F 2 "w_smd_cap:c_0603" H 2150 6500 60  0001 C CNN
+F 2 "Capacitors_SMD:C_0603_HandSoldering" H 2150 6500 60  0001 C CNN
 F 3 "" H 2150 6500 60  0000 C CNN
 	1    2150 6500
 	1    0    0    -1
 $EndComp
-Text Label 10150 1350 2    60   ~ 0
+Text Label 10150 1150 2    60   ~ 0
 GND
 $Comp
@@
 F 0 "C42" H 2160 6120 50  0000 L CNN
 F 1 "0.1uF" H 2160 5970 50  0000 L CNN
-F 2 "w_smd_cap:c_0603" H 2150 6050 60  0001 C CNN
+F 2 "Capacitors_SMD:C_0603_HandSoldering" H 2150 6050 60  0001 C CNN
 F 3 "" H 2150 6050 60  0000 C CNN
 	1    2150 6050
@@
 F 0 "C47" H 3060 6120 50  0000 L CNN
 F 1 "4.7uF" H 3060 5970 50  0000 L CNN
-F 2 "w_smd_cap:c_0603" H 3050 6050 60  0001 C CNN
+F 2 "Capacitors_SMD:C_0603_HandSoldering" H 3050 6050 60  0001 C CNN
 F 3 "" H 3050 6050 60  0000 C CNN
 	1    3050 6050
@@
 F 0 "C46" H 2760 6120 50  0000 L CNN
 F 1 "0.1uF" H 2760 5970 50  0000 L CNN
-F 2 "w_smd_cap:c_0603" H 2750 6050 60  0001 C CNN
+F 2 "Capacitors_SMD:C_0603_HandSoldering" H 2750 6050 60  0001 C CNN
 F 3 "" H 2750 6050 60  0000 C CNN
 	1    2750 6050
@@
 F 0 "C45" H 2460 6570 50  0000 L CNN
 F 1 "0.1uF" H 2460 6420 50  0000 L CNN
-F 2 "w_smd_cap:c_0603" H 2450 6500 60  0001 C CNN
+F 2 "Capacitors_SMD:C_0603_HandSoldering" H 2450 6500 60  0001 C CNN
 F 3 "" H 2450 6500 60  0000 C CNN
 	1    2450 6500
@@
 F 0 "C44" H 2460 6120 50  0000 L CNN
 F 1 "0.1uF" H 2460 5970 50  0000 L CNN
-F 2 "w_smd_cap:c_0603" H 2450 6050 60  0001 C CNN
+F 2 "Capacitors_SMD:C_0603_HandSoldering" H 2450 6050 60  0001 C CNN
 F 3 "" H 2450 6050 60  0000 C CNN
 	1    2450 6050
@@
 Text Label 7200 2800 0    60   ~ 0
 IN_B-
+Text Label 10150 1350 2    60   ~ 0
+3V3
 Text Label 10150 1250 2    60   ~ 0
-3V3
-Text Label 10150 1150 2    60   ~ 0
 1V8
 Text Label 10150 2350 2    60   ~ 0
@@
 F 0 "P3" H 10350 2950 50  0000 C CNN
 F 1 "CONN_01X18" V 10450 2000 50  0000 C CNN
-F 2 "w_pin_strip:pin_strip_18" H 10350 2000 60  0001 C CNN
+F 2 "Pin_Headers:Pin_Header_Straight_1x18" H 10350 2000 60  0001 C CNN
 F 3 "" H 10350 2000 60  0000 C CNN
 	1    10350 2000
@@
 F 0 "P2" H 4200 2100 50  0000 C CNN
 F 1 "CONN_01X18" V 4300 1150 50  0000 C CNN
-F 2 "w_pin_strip:pin_strip_18" H 4200 1150 60  0001 C CNN
+F 2 "Pin_Headers:Pin_Header_Straight_1x18" H 4200 1150 60  0001 C CNN
 F 3 "" H 4200 1150 60  0000 C CNN
 	1    4200 1150
