File: power.sch (KiCad schematic (older format))
At the start: 83 parts, among them Q1 Q_NMOS_DGS, U10 LMR62014, U2 LMZ10500, U3 LM25088, U4 TPS2420, U5 TPS63002, U6 LM3674, U7 TPS56x200, U8 TPS56x200, U9 TPS56x200

Commit message: initial experimentation with size constraints
Parts:
- C17: renamed from C44; footprint (none) -> w_smd_cap:c_0805
- D1: footprint w_smd_diode:sod523 -> w_smd_diode:sod80c
- D2, D3: footprint w_smd_diode:sod323 -> w_smd_diode:sod80c
- L1: footprint w_smd_inductors:inductor_smd_0603 -> w_smd_inductors:inductor_smd_0805
- Q1: footprint (none) -> w_smd_trans:sot23
- R1, R10, R11, R12, R13, R14, R15, R16, R17, R18, R19, R2, R20, R21, R22, R23, R24, R25, R26, R3, R4, R5, R6, R7, R8, R9: footprint w_smd_resistors:r_0603 -> w_smd_resistors:r_0805
- U1: renamed from U2; footprint (none) -> camera:llp-8
- U2: renamed from U3; footprint w_smd_dil:tssop-16 -> camera:htssop-16
- renumbered C28 to C1, C37 to C10, C38 to C11, C39 to C12, C40 to C13, C41 to C14, C42 to C15, C43 to C16, C45 to C18, C46 to C19, C29 to C2, C47 to C20, C48 to C21, C49 to C22, C50 to C23, C51 to C24, C52 to C25, C53 to C26, C54 to C27, C55 to C28, C56 to C29, C30 to C3, C57 to C30, C58 to C31, C59 to C32, C60 to C33, C61 to C34, C62 to C35, C31 to C4, C32 to C5, C33 to C6, C34 to C7, C35 to C8, C36 to C9, U4 to U3, U5 to U4, U6 to U5, U7 to U6, U8 to U7, U9 to U8, U10 to U9

Commit message: More work on schematic
Parts:
- C11: footprint w_smd_cap:c_0603 -> Capacitors_SMD:C_0805_HandSoldering; Component (none) -> Murata GRM188R71C105KA12D
- C20, C31: footprint w_smd_cap:c_0603 -> Capacitors_SMD:C_0603_HandSoldering
- C25: footprint w_smd_cap:c_0603 -> Capacitors_SMD:C_0805_HandSoldering
- C4: footprint w_smd_cap:c_0603 -> Capacitors_SMD:C_0805_HandSoldering; Component (none) -> TDK C1608X5R1A105K
- D1: footprint w_smd_diode:sod80c -> Diodes_SMD:Diode-SMB_Handsoldering
- L5: footprint w_smd_inductors:inductor_smd_0805 -> camera:Inductor_SMD_2016
- R10, R13, R6, R8, R9: footprint w_smd_resistors:r_0805 -> Resistors_SMD:R_0805_HandSoldering
- R19, R20: footprint w_smd_resistors:r_0805 -> Resistors_SMD:R_0402
- U3: footprint w_smd_qfn:pvqfn-n16 -> Housings_DFN_QFN:QFN-16-1EP_4x4mm_Pitch0.65mm; symbol TPS2420 -> TPS2420-RESCUE-AstroCam
Changed lines of the file:
@@
 EESchema Schematic File Version 2
+LIBS:AstroCam-rescue
 LIBS:power
 LIBS:device
@@
 F 0 "C4" H 1325 1600 50  0000 L CNN
 F 1 "1.0uF" H 1325 1400 50  0000 L CNN
-F 2 "w_smd_cap:c_0603" H 1338 1350 30  0001 C CNN
+F 2 "Capacitors_SMD:C_0805_HandSoldering" H 1338 1350 30  0001 C CNN
 F 3 "" H 1300 1500 60  0000 C CNN
+F 4 "TDK C1608X5R1A105K" H 1300 1500 60  0001 C CNN "Component"
 	1    1300 1500
 	1    0    0    -1
@@
 F 0 "D1" H 1700 1600 50  0000 C CNN
 F 1 "9V/5W" H 1700 1400 50  0000 C CNN
-F 2 "w_smd_diode:sod80c" H 1700 1500 60  0001 C CNN
+F 2 "Diodes_SMD:Diode-SMB_Handsoldering" H 1700 1500 60  0001 C CNN
 F 3 "" H 1700 1500 60  0000 C CNN
 	1    1700 1500
@@
 $EndComp
 $Comp
-L TPS2420 U3
+L TPS2420-RESCUE-AstroCam U3
 U 1 1 55769CFD
 P 3300 1450
+AR Path="/55769CFD" Ref="U3"  Part="1"
+AR Path="/557696AD/55769CFD" Ref="U3"  Part="1"
 F 0 "U3" H 2850 1900 60  0000 C CNN
 F 1 "TPS2420" H 3300 1500 60  0000 C CNN
-F 2 "w_smd_qfn:pvqfn-n16" H 3350 1400 60  0001 C CNN
+F 2 "Housings_DFN_QFN:QFN-16-1EP_4x4mm_Pitch0.65mm" H 3350 1400 60  0001 C CNN
 F 3 "" H 3350 1400 60  0000 C CNN
 	1    3300 1450
@@
 F 0 "R6" V 2030 950 50  0000 C CNN
 F 1 "10.0k" V 1850 950 50  0000 C CNN
-F 2 "w_smd_resistors:r_0805" V 1880 950 30  0001 C CNN
+F 2 "Resistors_SMD:R_0805_HandSoldering" V 1880 950 30  0001 C CNN
 F 3 "" H 1950 950 30  0000 C CNN
 	1    1950 950
@@
 F 0 "R8" V 2530 1000 50  0000 C CNN
 F 1 "10.0k" V 2350 1000 50  0000 C CNN
-F 2 "w_smd_resistors:r_0805" V 2380 1000 30  0001 C CNN
+F 2 "Resistors_SMD:R_0805_HandSoldering" V 2380 1000 30  0001 C CNN
 F 3 "" H 2450 1000 30  0000 C CNN
 	1    2450 1000
@@
 F 0 "R9" V 3100 2200 50  0000 C CNN
 F 1 "51.1k" V 3000 2200 50  0000 C CNN
-F 2 "w_smd_resistors:r_0805" V 3030 2200 30  0001 C CNN
+F 2 "Resistors_SMD:R_0805_HandSoldering" V 3030 2200 30  0001 C CNN
 F 3 "" H 3100 2200 30  0000 C CNN
 	1    3100 2200
@@
 F 0 "R10" V 3300 2200 50  0000 C CNN
 F 1 "68.1k" V 3200 2200 50  0000 C CNN
-F 2 "w_smd_resistors:r_0805" V 3230 2200 30  0001 C CNN
+F 2 "Resistors_SMD:R_0805_HandSoldering" V 3230 2200 30  0001 C CNN
 F 3 "" H 3300 2200 30  0000 C CNN
 	1    3300 2200
@@
 F 0 "C11" H 3525 2300 50  0000 L CNN
 F 1 "1.0F/11mOhm" H 3525 2100 50  0000 L CNN
-F 2 "w_smd_cap:c_0603" H 3538 2050 30  0001 C CNN
+F 2 "Capacitors_SMD:C_0805_HandSoldering" H 3538 2050 30  0001 C CNN
 F 3 "" H 3500 2200 60  0000 C CNN
+F 4 "Murata GRM188R71C105KA12D" H 3500 2200 60  0001 C CNN "Component"
 	1    3500 2200
 	1    0    0    -1
@@
 F 0 "R13" V 4250 2200 50  0000 C CNN
 F 1 "53.6k" V 4150 2200 50  0000 C CNN
-F 2 "w_smd_resistors:r_0805" V 4180 2200 30  0001 C CNN
+F 2 "Resistors_SMD:R_0805_HandSoldering" V 4180 2200 30  0001 C CNN
 F 3 "" H 4250 2200 30  0000 C CNN
 	1    4250 2200
@@
 F 0 "C20" H 6975 1350 50  0000 L CNN
 F 1 "4.7F/5.0mOhm" H 6975 1150 50  0000 L CNN
-F 2 "w_smd_cap:c_0603" H 6988 1100 30  0001 C CNN
+F 2 "Capacitors_SMD:C_0603_HandSoldering" H 6988 1100 30  0001 C CNN
 F 3 "" H 6950 1250 60  0000 C CNN
 	1    6950 1250
@@
 F 0 "L5" V 8800 850 50  0000 C CNN
 F 1 "2.2H/140ohm" V 8950 850 50  0000 C CNN
-F 2 "w_smd_inductors:inductor_smd_0805" H 8850 850 60  0001 C CNN
+F 2 "camera:Inductor_SMD_2016" H 8850 850 60  0001 C CNN
 F 3 "" H 8850 850 60  0000 C CNN
 	1    8850 850
@@
 F 0 "C25" H 9325 1200 50  0000 L CNN
 F 1 "9.0pF" H 9325 1000 50  0000 L CNN
-F 2 "w_smd_cap:c_0603" H 9338 950 30  0001 C CNN
+F 2 "Capacitors_SMD:C_0805_HandSoldering" H 9338 950 30  0001 C CNN
 F 3 "" H 9300 1100 60  0000 C CNN
 	1    9300 1100
@@
 F 0 "R20" V 9680 1100 50  0000 C CNN
 F 1 "402.0k/63mW" V 9750 1100 50  0000 C CNN
-F 2 "w_smd_resistors:r_0805" V 9530 1100 30  0001 C CNN
+F 2 "Resistors_SMD:R_0402" V 9530 1100 30  0001 C CNN
 F 3 "" H 9600 1100 30  0000 C CNN
 	1    9600 1100
@@
 F 0 "R19" V 9530 1550 50  0000 C CNN
 F 1 "100k/63.0mW" V 9600 1500 50  0000 C CNN
-F 2 "w_smd_resistors:r_0805" V 9380 1550 30  0001 C CNN
+F 2 "Resistors_SMD:R_0402" V 9380 1550 30  0001 C CNN
 F 3 "" H 9450 1550 30  0000 C CNN
 	1    9450 1550
@@
 F 0 "C31" H 10225 1500 50  0000 L CNN
 F 1 "10F/9Mohm" H 10225 1300 50  0000 L CNN
-F 2 "w_smd_cap:c_0603" H 10238 1250 30  0001 C CNN
+F 2 "Capacitors_SMD:C_0603_HandSoldering" H 10238 1250 30  0001 C CNN
 F 3 "" H 10200 1400 60  0000 C CNN
 	1    10200 1400
@@
 	10250 4700 10250 4550
 Connection ~ 9850 4700
-Text Label 10800 3850 0    60   ~ 0
-1V8
 Text Label 6800 5000 2    60   ~ 0
 5V5
@@
 	10500 5900 10500 5550
 Connection ~ 10500 5000
-Text Label 10950 4750 0    60   ~ 0
-12V
 Text Label 850  2650 2    60   ~ 0
 5V5
@@
 	3450 650  3450 850
 $Comp
-L PWR_FLAG #FLG01
+L PWR_FLAG #FLG4
 U 1 1 557D748F
 P 10400 4000
-F 0 "#FLG01" H 10400 4095 50  0001 C CNN
+F 0 "#FLG4" H 10400 4095 50  0001 C CNN
 F 1 "PWR_FLAG" H 10400 4180 50  0000 C CNN
 F 2 "" H 10400 4000 60  0000 C CNN
@@
 $EndComp
 $Comp
-L PWR_FLAG #FLG02
+L PWR_FLAG #FLG3
 U 1 1 557D789B
 P 3450 5600
-F 0 "#FLG02" H 3450 5695 50  0001 C CNN
+F 0 "#FLG3" H 3450 5695 50  0001 C CNN
 F 1 "PWR_FLAG" H 3450 5780 50  0000 C CNN
 F 2 "" H 3450 5600 60  0000 C CNN
@@
 $EndComp
 $Comp
-L PWR_FLAG #FLG03
+L PWR_FLAG #FLG1
 U 1 1 557D8CC1
 P 900 650
-F 0 "#FLG03" H 900 745 50  0001 C CNN
+F 0 "#FLG1" H 900 745 50  0001 C CNN
 F 1 "PWR_FLAG" H 900 830 50  0000 C CNN
 F 2 "" H 900 650 60  0000 C CNN
@@
 	4050 3250 4150 3250
 $Comp
-L PWR_FLAG #FLG04
+L PWR_FLAG #FLG2
 U 1 1 557DC7C3
 P 900 2350
-F 0 "#FLG04" H 900 2445 50  0001 C CNN
+F 0 "#FLG2" H 900 2445 50  0001 C CNN
 F 1 "PWR_FLAG" H 900 2530 50  0000 C CNN
 F 2 "" H 900 2350 60  0000 C CNN

Commit message: Work on proto breakout.
Parts:
- removed C1: 56nF, w_smd_cap:c_0603, symbol C
- removed C12: 68pF, w_smd_cap:c_0603, symbol C
- removed C14: 1.5nF, w_smd_cap:c_0603, symbol C
- removed C15, C8: 100nF, w_smd_cap:c_0603, symbol C
- removed C16: 1.0F/20Mohm, w_smd_cap:c_0603, symbol C
- removed C17: 15F, w_smd_cap:c_0805, symbol CP1
- removed C18, C19: 1.0F, w_smd_cap:c_0603, symbol C
- removed C24: 2.2F/4.9Mohm, w_smd_cap:c_0603, symbol C_Small
- removed C29: 270pF, w_smd_cap:c_0603, symbol C
- removed C30: 4.7F/2Mohm, w_smd_cap:c_0603, symbol C
- removed C35: 220nF/220Mohm, w_smd_cap:c_0603, symbol C
- removed D2: ZENERsmall, w_smd_diode:sod80c, symbol ZENERsmall
- removed D3: ZENER, w_smd_diode:sod80c, symbol ZENER
- removed L3: 100nH, w_smd_inductors:inductor_smd_0805, symbol L_Small
- removed L4: 12.0H/210Mohm, w_smd_inductors:inductor_smd_0805, symbol INDUCTOR
- removed L9: 100nH/20Mohm, w_smd_inductors:inductor_smd_0805, symbol INDUCTOR
- removed Q1: Q_NMOS_DGS, w_smd_trans:sot23, symbol Q_NMOS_DGS
- removed R11: 27k, w_smd_resistors:r_0805, symbol R
- removed R12: 82M/1W, w_smd_resistors:r_0805, symbol R
- removed R14: 7.87k, w_smd_resistors:r_0805, symbol R
- removed R15: 1.65k, w_smd_resistors:r_0805, symbol R
- removed R16: 1M, w_smd_resistors:r_0805, symbol R
- removed R17: 13.3k, w_smd_resistors:r_0805, symbol R_Small
- removed R18: 118k, w_smd_resistors:r_0805, symbol R
- removed R3: 3.57k, w_smd_resistors:r_0805, symbol R
- removed R4: 453k, w_smd_resistors:r_0805, symbol R
- removed R5: 10k, w_smd_resistors:r_0805, symbol R
- removed U2: LM25088, camera:htssop-16, symbol LM25088
- removed U9: LMR62014, w_smd_trans:sot23-5, symbol LMR62014
- added C10: 0.1uF, Capacitors_SMD:C_0805_HandSoldering, symbol C
- added C2, C6: 1.0uF, Capacitors_SMD:C_0805_HandSoldering, symbol C
- added L2: 15uH, w_smd_inductors:inductor_smd_0805, symbol L_Small
- added L4: 10uH, w_smd_inductors:inductor_smd_0805, symbol L_Small
- added R2: 324k, w_smd_resistors:r_0603, symbol R
- added U2: LT3487, w_smd_qfn:dfn10-3x3, symbol LT3487
- C3: value 4.7F/6Mohm -> 47pF; footprint w_smd_cap:c_0603 -> Capacitors_SMD:C_0805_HandSoldering; Component (none) -> TDK C1608X5R1A105K
- C5: value 220nF -> 47pF; footprint w_smd_cap:c_0603 -> Capacitors_SMD:C_0805_HandSoldering; Component (none) -> TDK C1608X5R1A105K
- C7: value 22nF -> 100nF; footprint w_smd_cap:c_0603 -> Capacitors_SMD:C_0805_HandSoldering; Component (none) -> TDK C1608X5R1A105K
- C9: value 56nF -> 4.7uF; footprint w_smd_cap:c_0603 -> Capacitors_SMD:C_0805_HandSoldering; Component (none) -> TDK C1608X5R1A105K
- L1: value 22H -> 15uH
- R7: value 10.2k -> 324k; footprint w_smd_resistors:r_0805 -> w_smd_resistors:r_0603
- renumbered C4 to C1, C20 to C11, C21 to C12, C22 to C13, C23 to C14, C2 to C15, C6 to C16, C25 to C17, C26 to C18, C27 to C19, C28 to C20, C10 to C21, C31 to C22, C32 to C23, C33 to C24, C34 to C25, C13 to C4, C11 to C8, L2 to L3, R6 to R1, R19 to R10, R20 to R11, R21 to R12, R22 to R13, R23 to R14, R24 to R15, R25 to R16, R26 to R17, R8 to R3, R9 to R4, R10 to R5, R13 to R6, R1 to R8, R2 to R9, U3 to U1, U4 to U3, U5 to U4, U6 to U5, U7 to U6, U8 to U7, U1 to U8
Connections:
- net labels added: +12V, CAP, DN, FBN, FBP
- wire segments 256 -> 193
Other:
- moved on the sheet: C15, C16, C21, C4, L3, R8, R9, U3, U8

Commit message: Lot's of back and forward with vendor.
Parts:
- removed C12, C13: 10.0F/3.0mOhm, w_smd_cap:c_0603, symbol C_Small
- removed C17: 9.0pF, Capacitors_SMD:C_0805_HandSoldering, symbol C
- removed C18, C19: 100nF, w_smd_cap:c_0603, symbol C_Small
- removed C22: 10F/9Mohm, Capacitors_SMD:C_0603_HandSoldering, symbol C
- removed C23, C24: 47F/3Mohm, w_smd_cap:c_0603, symbol C
- removed L5: 2.2H/140ohm, camera:Inductor_SMD_2016, symbol INDUCTOR
- removed L6, L7: 1.5H/14.4mOhm, w_smd_inductors:inductor_smd_0805, symbol L_Small
- removed R10: 100k/63.0mW, Resistors_SMD:R_0402, symbol R
- removed R11: 402.0k/63mW, Resistors_SMD:R_0402, symbol R
- removed R12, R14: 5.76k, w_smd_resistors:r_0805, symbol R_Small
- removed R13, R15: 10.0k, w_smd_resistors:r_0805, symbol R_Small
- removed U1: TPS2420, Housings_DFN_QFN:QFN-16-1EP_4x4mm_Pitch0.65mm, symbol TPS2420-RESCUE-AstroCam
- removed U4: LM3674, w_smd_trans:sot23-5, symbol LM3674
- removed U5, U6: TPS56x200, w_smd_trans:sot23-6, symbol TPS56x200
- added P8: CONN_01X06, w_pin_strip:pin_socket_6, symbol CONN_01X06
- added P9: CONN_01X02, w_pin_strip:pin_socket_2, symbol CONN_01X02
- added U1: TPS2420, camera:S-PVQFN-N16, symbol TPS2420
- C11: value 4.7F/5.0mOhm -> 10uF; footprint Capacitors_SMD:C_0603_HandSoldering -> Capacitors_SMD:C_0805_HandSoldering; Component (none) -> TDK C1608X5R1A105K
- U3: footprint (none) -> Housings_DFN_QFN:DFN-10-1EP_3x3mm_Pitch0.5mm
Connections:
- net labels added: PAD, VCON, VREF, V_BAT
- net labels removed: 1V2_1, 1V2_2, 2V5, V_BATT
- wire segments 193 -> 132
Other:
- moved on the sheet: C1, C10, C14, C15, C16, C2, C20, C21, C25, C3, C4, C5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

Commit message: more work
Parts:
- R1, R17, R3: value 10.0k -> 10.0kE
- R16: value 13.7k -> 13.7kE
- R2, R7: value 324k -> 324kE
- R4: value 51.1k -> 51.1kE
- R5: value 68.1k -> 68.1kE
- R6: value 53.6k -> 53.6kE
- R8: value 80.6k -> 80.6kE
- R9: value 105k -> 105kE
Changed lines of the file:
@@
 P 2350 1550
 F 0 "R1" V 2430 1550 50  0000 C CNN
-F 1 "10.0k" V 2250 1550 50  0000 C CNN
+F 1 "10.0kE" V 2250 1550 50  0000 C CNN
 F 2 "Resistors_SMD:R_0805_HandSoldering" V 2280 1550 30  0001 C CNN
 F 3 "" H 2350 1550 30  0000 C CNN
@@
 P 2850 1600
 F 0 "R3" V 2930 1600 50  0000 C CNN
-F 1 "10.0k" V 2750 1600 50  0000 C CNN
+F 1 "10.0kE" V 2750 1600 50  0000 C CNN
 F 2 "Resistors_SMD:R_0805_HandSoldering" V 2780 1600 30  0001 C CNN
 F 3 "" H 2850 1600 30  0000 C CNN
@@
 P 3500 2800
 F 0 "R4" V 3500 2800 50  0000 C CNN
-F 1 "51.1k" V 3400 2800 50  0000 C CNN
+F 1 "51.1kE" V 3400 2800 50  0000 C CNN
 F 2 "Resistors_SMD:R_0805_HandSoldering" V 3430 2800 30  0001 C CNN
 F 3 "" H 3500 2800 30  0000 C CNN
@@
 P 3700 2800
 F 0 "R5" V 3700 2800 50  0000 C CNN
-F 1 "68.1k" V 3600 2800 50  0000 C CNN
+F 1 "68.1kE" V 3600 2800 50  0000 C CNN
 F 2 "Resistors_SMD:R_0805_HandSoldering" V 3630 2800 30  0001 C CNN
 F 3 "" H 3700 2800 30  0000 C CNN
@@
 P 4650 2800
 F 0 "R6" V 4650 2800 50  0000 C CNN
-F 1 "53.6k" V 4550 2800 50  0000 C CNN
+F 1 "53.6kE" V 4550 2800 50  0000 C CNN
 F 2 "Resistors_SMD:R_0805_HandSoldering" V 4580 2800 30  0001 C CNN
 F 3 "" H 4650 2800 30  0000 C CNN
@@
 P 9650 1900
 F 0 "R16" H 9680 1920 50  0000 L CNN
-F 1 "13.7k" H 9680 1860 50  0000 L CNN
+F 1 "13.7kE" H 9680 1860 50  0000 L CNN
 F 2 "w_smd_resistors:r_0805" H 9650 1900 60  0001 C CNN
 F 3 "" H 9650 1900 60  0000 C CNN
@@
 P 9650 2250
 F 0 "R17" H 9680 2270 50  0000 L CNN
-F 1 "10.0k" H 9680 2210 50  0000 L CNN
+F 1 "10.0kE" H 9680 2210 50  0000 L CNN
 F 2 "w_smd_resistors:r_0805" H 9650 2250 60  0001 C CNN
 F 3 "" H 9650 2250 60  0000 C CNN
@@
 P 7150 3750
 F 0 "R9" H 7180 3770 50  0000 L CNN
-F 1 "105k" H 7180 3710 50  0000 L CNN
+F 1 "105kE" H 7180 3710 50  0000 L CNN
 F 2 "w_smd_resistors:r_0805" H 7150 3750 60  0001 C CNN
 F 3 "" H 7150 3750 60  0000 C CNN
@@
 P 7150 3450
 F 0 "R8" H 7180 3470 50  0000 L CNN
-F 1 "80.6k" H 7180 3410 50  0000 L CNN
+F 1 "80.6kE" H 7180 3410 50  0000 L CNN
 F 2 "w_smd_resistors:r_0805" H 7150 3450 60  0001 C CNN
 F 3 "" H 7150 3450 60  0000 C CNN
@@
 P 2500 4750
 F 0 "R2" V 2580 4750 50  0000 C CNN
-F 1 "324k" V 2500 4750 50  0000 C CNN
+F 1 "324kE" V 2500 4750 50  0000 C CNN
 F 2 "w_smd_resistors:r_0603" V 2430 4750 30  0001 C CNN
 F 3 "" H 2500 4750 30  0000 C CNN
@@
 P 4550 4250
 F 0 "R7" V 4630 4250 50  0000 C CNN
-F 1 "324k" V 4550 4250 50  0000 C CNN
+F 1 "324kE" V 4550 4250 50  0000 C CNN
 F 2 "w_smd_resistors:r_0603" V 4480 4250 30  0001 C CNN
 F 3 "" H 4550 4250 30  0000 C CNN

Commit message: lots of work
Parts:
- C14: value 10.0F/3.0mOhm -> 10.0uF; footprint w_smd_cap:c_0603 -> Capacitors_SMD:C_0805_HandSoldering
- C15: value 10.0F/9Mohm -> 10.0uF; footprint w_smd_cap:c_0603 -> Capacitors_SMD:C_0805_HandSoldering
- C16: footprint w_smd_cap:c_0603 -> Capacitors_SMD:C_0402
- C20: value 100nF -> 0.1uF; footprint w_smd_cap:c_0603 -> Capacitors_SMD:C_0603_HandSoldering
- C21: value 10.0uF/9.0Mohm -> 10.0uF; footprint w_smd_cap:c_0603 -> Capacitors_SMD:C_0805_HandSoldering
- C25: value 47F/3Mohm -> 47uF; footprint w_smd_cap:c_0603 -> Capacitors_SMD:C_1206_HandSoldering
- C4: value 2.20uF/2.80Mohm -> 2.2uF; footprint w_smd_cap:c_0603 -> Capacitors_SMD:C_0603_HandSoldering
- C8: value 1.0F/11mOhm -> 1.0uF/11mOhm
- L3: value 2.0uH/0.024Ohm -> 2.0uH
- L8: value 2.2H/13.0mOhm -> 2.2uH
- P8: footprint w_pin_strip:pin_socket_6 -> Pin_Headers:Pin_Header_Straight_1x06
- P9: footprint w_pin_strip:pin_socket_2 -> Pin_Headers:Pin_Header_Straight_1x02
- R1: value 10.0kE -> 10.0k
- R16: value 13.7kE -> 13.7k; footprint w_smd_resistors:r_0805 -> Resistors_SMD:R_0402
- R17: value 10.0kE -> 10.0k; footprint w_smd_resistors:r_0805 -> Resistors_SMD:R_0402
- R2, R7: value 324kE -> 324k; footprint w_smd_resistors:r_0603 -> Resistors_SMD:R_0603_HandSoldering
- R3: value 10.0kE -> 10.0k; footprint Resistors_SMD:R_0805_HandSoldering -> Resistors_SMD:R_0603_HandSoldering
- R4: value 51.1kE -> 51.1k; footprint Resistors_SMD:R_0805_HandSoldering -> Resistors_SMD:R_0603_HandSoldering
- R5: value 68.1kE -> 68.1k; footprint Resistors_SMD:R_0805_HandSoldering -> Resistors_SMD:R_0603_HandSoldering
- R6: value 53.6kE -> 53.6k; footprint Resistors_SMD:R_0805_HandSoldering -> Resistors_SMD:R_0603_HandSoldering
- R8: value 80.6kE -> 80.6k; footprint w_smd_resistors:r_0805 -> Resistors_SMD:R_0402
- R9: value 105kE -> 105k; footprint w_smd_resistors:r_0805 -> Resistors_SMD:R_0402
- U1: footprint camera:S-PVQFN-N16 -> Housings_DFN_QFN:QFN-16-1EP_4x4mm_Pitch0.65mm
- U7: footprint w_smd_trans:sot23-6 -> Housings_SOT-23_SOT-143_TSOT-6:SOT-23-6
Connections:
- net labels added: SOFT_START
- net labels removed: PAD
- wire segments 132 -> 137
Other:
- moved on the sheet: C14, C8, R1, R3, R4, R5, R6
