File: pcb/breakout-addi.kicad_pcb (KiCad board)
At the start: 2 copper layers, 45.7 x 15.2 mm, 16 parts, among them P2 CONN_01X18, P3 CONN_01X18, U11 ADDI7013

Commit message: Confirm to Advanced Circuits
Parts:
- removed G***: LOGO, w_logo:Logo_silk_OSHW_6x6mm
Routing:
- net /h-driver/VD: track 30.5 -> 23.4 mm
- net /h-driver/GP04: track 16.2 -> 9.94 mm
- net /h-driver/HD: track 30.5 -> 26.0 mm
- net GND: track 39.1 -> 43.1 mm
- net /h-driver/SYNC: track 30.5 -> 28.5 mm
- net /h-driver/SL: track 24.4 -> 22.7 mm
- net /h-driver/1V8: track 55.2 -> 55.8 mm, vias 5 -> 4
Other:
- net class Default: clearance 0.1016 -> 0.127; via_dia 0.4064 -> 0.4318; via_drill 0.2032 -> 0.1778
- rule pad_to_mask_clearance: 0 -> 0.0762
- rule trace_clearance: 0.1016 -> 0.127
- rule trace_min: 0.1524 -> 0.127
- rule via_min_drill: 0.2032 -> 0.1778
- rule via_min_size: 0.4064 -> 0.4318
