File: pcb/breakout-addi.kicad_pcb (KiCad board)
At the start: 2 copper layers, 45.7 x 15.2 mm, 15 parts, among them P2 CONN_01X18, P3 CONN_01X18, U11 ADDI7013

Commit message: Cleanups
Parts:
- moved C47 1.07 mm to (41.4, 50.1), turned to 0 degrees
- moved C38 0.80 mm to (47.6, 51.8), turned to 180 degrees
- moved C42 0.68 mm to (47.6, 53.4), turned to 180 degrees
- moved C43 0.46 mm to (47.6, 55.5), turned to 180 degrees
Connections:
- net Net-(C48-Pad2) renamed /h-driver/INP_A+
- net Net-(C49-Pad2) renamed /h-driver/INP_B+
Routing:
- net (no net): track 0.00 -> 42.5 mm
- net GND: track 43.1 -> 80.9 mm, vias 4 -> 10
- net /h-driver/1V8: track 55.8 -> 58.9 mm, vias 4 -> 5
- net /h-driver/SYNC: track 28.5 -> 31.5 mm
- net /h-driver/HD: track 26.0 -> 28.9 mm
- net /h-driver/VD: track 23.4 -> 26.3 mm
- net /h-driver/SL: track 22.7 -> 25.1 mm
- net /h-driver/GP04: track 9.94 -> 11.4 mm
- net /h-driver/3V3: track 54.4 -> 53.2 mm
- net /h-driver/B1+: track 17.3 -> 16.3 mm
- net /h-driver/SDATA: track 29.5 -> 30.3 mm
- net /h-driver/SCK: track 27.0 -> 27.7 mm
- net /h-driver/IN_B-: track 7.48 -> 8.15 mm
