File: pcb/breakout-addi.kicad_pcb (KiCad board)
At the start: 2 copper layers, 45.7 x 15.2 mm, 15 parts, among them P2 CONN_01X18, P3 CONN_01X18, U11 ADDI7013

Commit message: Start up work to revive this project.
Other:
- net class Default removed
