File: pcb/experiment.kicad_pcb (KiCad board)
At the start: 2 copper layers, 37 x 38 mm, 82 parts, among them P1 CONN_01X02, P13 CONN_01X06, P14 LEDS, P15 ADJ, P16 CONN_01X02, Q5 VEC2611, Q6 VEC2607, T3 NET-TIE, U11 TPS65530

Commit message: latest
Parts:
- added CON1: BARREL_JACK, w_conn_misc:dc_socket, F.Cu at (190.3, 38.7)
- L10, L9: value 4.7 -> 4.7u
- P1: value CONN_01X02 -> USB_OTG; footprint xess:HDR_1x2 -> w_conn_pc:conn_usb_B_mini_smd
- moved P13 47.1 mm to (131.0, 63.1)
- moved T3 29.6 mm to (157.7, 46.9)
- moved P16 22.6 mm to (165.6, 42.3)
- moved P1 19.6 mm to (175.5, 39.6)
- moved hole_3mm 17.0 mm to (154.3, 39.0)
- moved hole_3mm 12.0 mm to (198.3, 39.0)
- moved hole_3mm 12.0 mm to (154.3, 83.0)
- moved L11 7.91 mm to (161.2, 60.1)
- moved C59 7.84 mm to (161.7, 54.0)
- moved C66 7.48 mm to (161.3, 64.5)
- moved C63 7.48 mm to (164.3, 68.1)
- moved C70 7.48 mm to (161.9, 70.1)
- moved R41 7.48 mm to (165.1, 65.9)
- moved C64 7.48 mm to (161.1, 68.1)
- moved R40 7.48 mm to (165.1, 64.3)
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Connections:
- net /u-ctrl/VOUT_AFE renamed /u-ctrl/VOUT_AFE_3V3
- net /u-ctrl/VOUT_BACKL renamed /u-ctrl/VOUT_BACKL_5V
- net /u-ctrl/VOUT_CORE renamed /u-ctrl/VOUT_CORE_1V2
- net /u-ctrl/VOUT_IO renamed /u-ctrl/VOUT_IO_3V3
- net /u-ctrl/VOUT_MEM renamed /u-ctrl/VOUT_MEM_1V8
- net /u-ctrl/VOUT_MOTOR renamed /u-ctrl/VOUT_MOTOR_5V
- P1 pad 2: GNDA -> Net-(P1-Pad2)
Routing:
- net /u-ctrl/VBATT: track 178.2 -> 0.00 mm, vias 7 -> 0
- net GND: track 125.7 -> 0.00 mm, vias 6 -> 0
- net /u-ctrl/VOUT_CORE_1V2: track 55.9 -> 0.00 mm, vias 1 -> 0
- net GNDA: track 54.5 -> 0.00 mm, vias 2 -> 0
- net /u-ctrl/VOUT_MOTOR_5V: track 49.2 -> 0.00 mm, vias 1 -> 0
- net /u-ctrl/VOUT_MEM_1V8: track 48.1 -> 0.00 mm, vias 1 -> 0
- net /u-ctrl/VOUT_IO_3V3: track 45.0 -> 0.00 mm, vias 1 -> 0
- net /u-ctrl/VOUT_CCD-: track 29.8 -> 0.00 mm
- net /u-ctrl/VOUT_AFE_3V3: track 25.5 -> 0.00 mm, vias 1 -> 0
- net /u-ctrl/EN_AFE: track 22.4 -> 0.00 mm, vias 2 -> 0
- net Net-(P14-Pad2): track 20.5 -> 0.00 mm, vias 1 -> 0
- net /u-ctrl/V_BADJ: track 19.3 -> 0.00 mm, vias 1 -> 0
- net /u-ctrl/VOUT_CCD+: track 16.4 -> 0.00 mm
- net /u-ctrl/VOUT_BACKL_5V: track 15.5 -> 0.00 mm
- net Net-(D4-Pad1): track 15.4 -> 0.00 mm
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- removed copper zone on F.Cu, net GND
Other:
- board size 37 x 38 mm -> 50 x 50 mm
