File: pcb/AstroCam.sch (KiCad schematic (older format))
At the start: 1 part, among them P1 CONN_01X02

Commit message: Latest, greatest.
Parts:
- removed P1: CONN_01X02, Pin_Headers:Pin_Header_Straight_1x02, symbol CONN_01X02
Connections:
- wire segments 63 -> 0
Changed lines of the file:
@@
 $EndDescr
 $Sheet
-S 2850 2950 1000 1350
+S 1650 1550 1000 1350
 U 557696AD
 F0 "power-supply" 60
 F1 "power.sch" 60
-F2 "V_BATT" I L 2850 3250 60
-F3 "GND" I L 2850 3350 60
-F4 "-7V" I R 3850 3150 60
-F5 "3V3" I R 3850 3650 60
-F6 "2V5" I R 3850 3800 60
-F7 "1V2_1" I R 3850 4100 60
-F8 "1V2_2" I R 3850 4250 60
-F9 "1V8" I R 3850 3950 60
-F10 "5V0" I R 3850 3500 60
-F11 "5V5" I R 3850 3350 60
-F12 "12V" I R 3850 3050 60
 $EndSheet
-$Comp
-L CONN_01X02 P1
-U 1 1 557EF73C
-P 2150 3300
-F 0 "P1" H 2150 3450 50  0000 C CNN
-F 1 "CONN_01X02" V 2250 3300 50  0000 C CNN
-F 2 "Pin_Headers:Pin_Header_Straight_1x02" H 2150 3300 60  0001 C CNN
-F 3 "" H 2150 3300 60  0000 C CNN
-	1    2150 3300
-	-1   0    0    1
-$EndComp
 $Sheet
-S 5400 3600 850  900
+S 4450 1550 850  900
 U 557AD230
 F0 "h-driver" 60
 F1 "h-driver.sch" 60
-F2 "H1" I R 6250 3700 60
-F3 "H2" I R 6250 3800 60
-F4 "H3" I R 6250 3900 60
-F5 "H4" I R 6250 4000 60
-F6 "HL1" I R 6250 4100 60
-F7 "HL2" I R 6250 4200 60
-F8 "RG1" I R 6250 4300 60
-F9 "RG2" I R 6250 4400 60
-F10 "INPA+" I L 5400 4050 60
-F11 "INPB+" I L 5400 4300 60
-F12 "INPA-" I L 5400 4150 60
-F13 "INPB-" I L 5400 4400 60
-F14 "3V3" I L 5400 3700 60
-F15 "1V8" I L 5400 3800 60
-F16 "GND" I L 5400 3900 60
-$EndSheet
-Wire Wire Line
-	3850 3950 4800 3950
-Wire Wire Line
-	3850 3650 4800 3650
-Wire Wire Line
-	5600 2050 6450 2050
-Wire Wire Line
-	5600 2150 6550 2150
-Wire Wire Line
-	5600 2250 6650 2250
-Wire Wire Line
-	5600 2350 6750 2350
-Wire Wire Line
-	5600 2600 6450 2600
-Wire Wire Line
-	5600 2700 6550 2700
-Wire Wire Line
-	5600 2800 6650 2800
-Wire Wire Line
-	5600 2900 6750 2900
-Wire Wire Line
-	4150 3500 3850 3500
-Wire Wire Line
-	4800 3650 4800 3700
-Wire Wire Line
-	4800 3700 5400 3700
-Wire Wire Line
-	4800 3950 4800 3800
-Wire Wire Line
-	4800 3800 5400 3800
-Wire Wire Line
-	6450 3700 6250 3700
-Wire Wire Line
-	6450 2050 6450 3700
-Connection ~ 6450 2600
-Wire Wire Line
-	6550 3800 6250 3800
-Wire Wire Line
-	6550 2150 6550 3800
-Connection ~ 6550 2700
-Wire Wire Line
-	6650 3900 6250 3900
-Wire Wire Line
-	6650 2250 6650 3900
-Connection ~ 6650 2800
-Wire Wire Line
-	6750 4000 6250 4000
-Wire Wire Line
-	6750 2350 6750 4000
-Connection ~ 6750 2900
-Wire Wire Line
-	6250 4100 6850 4100
-Wire Wire Line
-	6850 4100 6850 1950
-Wire Wire Line
-	6850 1950 5600 1950
-Wire Wire Line
-	5600 2500 6950 2500
-Wire Wire Line
-	6950 2500 6950 4200
-Wire Wire Line
-	6950 4200 6250 4200
-Wire Wire Line
-	6250 4300 7150 4300
-Wire Wire Line
-	7150 4300 7150 1550
-Wire Wire Line
-	6250 4400 7250 4400
-Wire Wire Line
-	7250 4400 7250 1450
-Wire Wire Line
-	2350 3250 2850 3250
-Wire Wire Line
-	2350 3350 2850 3350
-Wire Wire Line
-	4350 4050 5400 4050
-Wire Wire Line
-	4450 4300 5400 4300
-Wire Wire Line
-	5400 3900 5150 3900
-Wire Wire Line
-	5150 3900 5150 4550
-Wire Wire Line
-	5150 4150 5400 4150
-Connection ~ 5150 4150
-Connection ~ 5150 4400
-Wire Wire Line
-	2600 3350 2600 4550
-Wire Wire Line
-	2600 4550 5150 4550
-Connection ~ 2600 3350
-Wire Wire Line
-	5150 4400 5400 4400
-Wire Wire Line
-	4500 1950 4400 1950
-Wire Wire Line
-	4400 1950 4400 1550
-Wire Wire Line
-	4500 2050 4300 2050
-Wire Wire Line
-	4300 2050 4300 1450
-Wire Wire Line
-	4400 1550 7150 1550
-Wire Wire Line
-	4300 1450 7250 1450
-Wire Wire Line
-	3850 3050 3950 3050
-Wire Wire Line
-	3950 3050 3950 2250
-Wire Wire Line
-	3950 2250 4500 2250
-Wire Wire Line
-	4050 3150 3850 3150
-Wire Wire Line
-	4050 2350 4050 3150
-Wire Wire Line
-	4050 2350 4500 2350
-Wire Wire Line
-	4150 2450 4150 3500
-Wire Wire Line
-	4150 2450 4500 2450
-Wire Wire Line
-	4500 2550 4250 2550
-Wire Wire Line
-	4250 2550 4250 4550
-Connection ~ 4250 4550
-Wire Wire Line
-	4500 2800 4350 2800
-Wire Wire Line
-	4350 2800 4350 4050
-Wire Wire Line
-	4500 2900 4450 2900
-Wire Wire Line
-	4450 2900 4450 4300
-$Sheet
-S 8350 3150 1800 1400
-U 557FDF11
-F0 "Save" 60
-F1 "Save.sch" 60
 $EndSheet
 $Sheet
-S 4500 1850 1100 1200
+S 3050 1550 1100 1200
 U 557AFA5B
 F0 "camera" 60
 F1 "camera.sch" 60
 $EndSheet
+$Sheet
+S 5650 1550 1300 1400
+U 55E85005
+F0 "u-ctrl" 60
+F1 "u-ctrl.sch" 60
+$EndSheet
 $EndSCHEMATC

Commit message: work
Changed lines of the file:
@@
 $EndDescr
 $Sheet
-S 1650 1550 1000 1350
-U 557696AD
-F0 "power-supply" 60
-F1 "power.sch" 60
-$EndSheet
-$Sheet
-S 4450 1550 850  900
+S 5750 2650 850  900
 U 557AD230
 F0 "h-driver" 60
@@
 $EndSheet
 $Sheet
-S 3050 1550 1100 1200
-U 557AFA5B
-F0 "camera" 60
-F1 "camera.sch" 60
+S 4400 2700 1000 900
+U 568B9711
+F0 "fpga" 60
+F1 "fpga.sch" 60
 $EndSheet
 $Sheet
-S 5650 1550 1300 1400
-U 55E85005
-F0 "u-ctrl" 60
-F1 "u-ctrl.sch" 60
+S 3050 2650 950  950
+U 56ACC940
+F0 "usb-ctrl" 50
+F1 "usb-ctrl.sch" 50
+$EndSheet
+$Sheet
+S 6850 2650 1000 950
+U 56F8F5B8
+F0 "power" 50
+F1 "power.sch" 50
 $EndSheet
 $EndSCHEMATC
