File: pcb/AstroCam.sch (KiCad schematic (older format))
At the start: 1 part, among them P1 CONN_01X02

Commit message: Safety checkin.
Parts:
- P1: symbol CONN_01X02 -> AstroCam-rescue:CONN_01X02
Connections:
- wire segments 63 -> 26
- no-connect marks 0 -> 4
Other:
- moved on the sheet: P1

Commit message: A little more work.
Parts:
- removed P1: CONN_01X02, Pin_Headers:Pin_Header_Straight_1x02, symbol AstroCam-rescue:CONN_01X02
Connections:
- no-connect marks 4 -> 0
Changed lines of the file:
@@
 F1 "power.sch" 60
 $EndSheet
-$Comp
-L AstroCam-rescue:CONN_01X02 P1
-U 1 1 557EF73C
-P 1800 1700
-F 0 "P1" H 1800 1850 50  0000 C CNN
-F 1 "CONN_01X02" V 1900 1700 50  0000 C CNN
-F 2 "Pin_Headers:Pin_Header_Straight_1x02" H 1800 1700 60  0001 C CNN
-F 3 "" H 1800 1700 60  0000 C CNN
-	1    1800 1700
-	-1   0    0    1
-$EndComp
 $Sheet
 S 4650 1600 1100 1250
@@
 F9 "CCD_OUT1" O R 5750 1700 50
 F10 "CCD_OUT2" O R 5750 2000 50
-F11 "CCD_5V0A" I R 5750 2450 50
-F12 "CCD_3V3" I R 5750 2750 50
-F13 "CCD_12VA" I R 5750 2300 50
-F14 "CCD_N7VA" I R 5750 2600 50
-F15 "CCD_H1" I L 4650 1650 50
-F16 "CCD_H2" I L 4650 1750 50
-F17 "CCD_HL" I L 4650 1850 50
-F18 "CCD_RG" I L 4650 1950 50
+F11 "CCD_H1" I L 4650 1650 50
+F12 "CCD_H2" I L 4650 1750 50
+F13 "CCD_HL" I L 4650 1850 50
+F14 "CCD_RG" I L 4650 1950 50
 $EndSheet
 $Sheet
-S 6650 1150 1300 2100
+S 6700 1150 1300 2100
 U 557AD230
 F0 "h-driver" 60
 F1 "h-driver.sch" 60
-F2 "ADC_SYNC" I L 6650 2550 50
-F3 "ADC_VD" I L 6650 2350 50
-F4 "ADC_HD" I L 6650 2450 50
-F5 "ADC_SCK" I L 6650 2850 50
-F6 "ADC_SDATA" I L 6650 2950 50
-F7 "ADC_SL" I L 6650 3050 50
-F8 "ADC_INA" I L 6650 1700 50
-F9 "ADC_INB" I L 6650 2000 50
-F10 "ADC_OUT_A0+" O R 7950 2200 50
-F11 "ADC_OUT_A0-" O R 7950 2300 50
-F12 "ADC_OUT_A1+" O R 7950 2400 50
-F13 "ADC_OUT_A1-" O R 7950 2500 50
-F14 "ADC_OUT_B0+" O R 7950 2600 50
-F15 "ADC_OUT_B0-" O R 7950 2700 50
-F16 "ADC_OUT_B1+" O R 7950 2800 50
-F17 "ADC_OUT_B1-" O R 7950 2900 50
-F18 "ADC_OUT_TCLK+" O R 7950 3000 50
-F19 "ADC_OUT_TCKL-" O R 7950 3100 50
-F20 "ADC_HOR_H1" O R 7950 1250 50
-F21 "ADC_HOR_H2" O R 7950 1350 50
-F22 "ADC_HOR_H4" O R 7950 1550 50
-F23 "ADC_HOR_HL1" O R 7950 1650 50
-F24 "ADC_HOR_HL2" O R 7950 1750 50
-F25 "ADC_HOR_RG1" O R 7950 1850 50
-F26 "ADC_HOR_RG2" O R 7950 1950 50
-F27 "ADC_1V8A" I L 6650 1250 50
-F28 "ADC_1V8" I L 6650 1350 50
-F29 "ADC_3V3" I L 6650 1450 50
-F30 "ADC_HOR_H3" O R 7950 1450 50
+F2 "ADC_VD" I L 6700 2350 50
+F3 "ADC_HD" I L 6700 2450 50
+F4 "ADC_SCK" I L 6700 2850 50
+F5 "ADC_SDATA" I L 6700 2950 50
+F6 "ADC_SL" I L 6700 3050 50
+F7 "ADC_INA" I L 6700 1700 50
+F8 "ADC_INB" I L 6700 2000 50
+F9 "ADC_OUT_A0+" O R 8000 2200 50
+F10 "ADC_OUT_A0-" O R 8000 2300 50
+F11 "ADC_OUT_A1+" O R 8000 2400 50
+F12 "ADC_OUT_A1-" O R 8000 2500 50
+F13 "ADC_OUT_B0+" O R 8000 2600 50
+F14 "ADC_OUT_B0-" O R 8000 2700 50
+F15 "ADC_OUT_B1+" O R 8000 2800 50
+F16 "ADC_OUT_B1-" O R 8000 2900 50
+F17 "ADC_OUT_TCLK+" O R 8000 3000 50
+F18 "ADC_OUT_TCKL-" O R 8000 3100 50
+F19 "ADC_CLI" I L 6700 2550 50
 $EndSheet
 Wire Wire Line
-	5750 1700 6650 1700
+	5750 1700 6700 1700
 Wire Wire Line
-	5750 2000 6650 2000
-Wire Wire Line
-	8400 1250 8400 950
-Wire Wire Line
-	8400 950  4300 950
-Wire Wire Line
-	4300 950  4300 1650
-Wire Wire Line
-	4300 1650 4650 1650
-Wire Wire Line
-	8500 1350 8500 850
-Wire Wire Line
-	8500 850  4200 850
-Wire Wire Line
-	4200 850  4200 1750
-Wire Wire Line
-	4200 1750 4650 1750
-Wire Wire Line
-	7950 1650 8600 1650
-Wire Wire Line
-	8600 1650 8600 750
-Wire Wire Line
-	8600 750  4100 750
-Wire Wire Line
-	4100 750  4100 1850
-Wire Wire Line
-	4100 1850 4650 1850
-Wire Wire Line
-	7950 1850 8700 1850
-Wire Wire Line
-	8700 1850 8700 650
-Wire Wire Line
-	8700 650  4000 650
-Wire Wire Line
-	4000 650  4000 1950
-Wire Wire Line
-	4000 1950 4650 1950
-Wire Wire Line
-	7950 1450 8100 1450
-Wire Wire Line
-	7950 1550 8100 1550
-Wire Wire Line
-	7950 1750 8100 1750
-Wire Wire Line
-	7950 1950 8100 1950
-NoConn ~ 8100 1450
-NoConn ~ 8100 1550
-NoConn ~ 8100 1750
-NoConn ~ 8100 1950
-Wire Wire Line
-	8400 1250 7950 1250
-Wire Wire Line
-	7950 1350 8500 1350
+	5750 2000 6700 2000
 $EndSCHEMATC

Commit message: Work on power system and horizontal driver.
Parts:
- added J2, J3, J4, J5: PMOD, Connector_PinHeader_2.54mm:PinHeader_2x06_P2.54mm_Horizontal, symbol Connector_Generic:Conn_02x06_Odd_Even
Connections:
- net h-driver/ADC_OUT_A0+: now also J4.11 (Pin_11)
- net h-driver/ADC_OUT_A0-: now also J4.9 (Pin_9)
- net h-driver/ADC_OUT_A1+: now also J4.7 (Pin_7)
- net h-driver/ADC_OUT_A1-: now also J4.5 (Pin_5)
- net h-driver/ADC_OUT_B0+: now also J5.11 (Pin_11)
- net h-driver/ADC_OUT_B0-: now also J5.9 (Pin_9)
- net h-driver/ADC_OUT_B1+: now also J5.7 (Pin_7)
- net h-driver/ADC_OUT_B1-: now also J5.5 (Pin_5)
- net h-driver/ADC_OUT_TCKL-: now also J4.8 (Pin_8)
- net h-driver/ADC_OUT_TCLK+: now also J4.6 (Pin_6)
- new net +3V3: J2.1 (Pin_1), J2.2 (Pin_2), J3.1 (Pin_1), J3.2 (Pin_2), J4.1 (Pin_1), J4.2 (Pin_2), J5.1 (Pin_1), J5.2 (Pin_2)
- new net ADC_CLI: J5.12 (Pin_12)
- new net ADC_HD: J5.10 (Pin_10)
- new net ADC_SCK: J2.8 (Pin_8)
- new net ADC_SDATA: J2.10 (Pin_10)
- new net ADC_SL: J2.6 (Pin_6)
- new net ADC_VD: J3.6 (Pin_6)
- new net CCD_H1: J4.12 (Pin_12)
- new net CCD_H2: J4.10 (Pin_10)
- new net CCD_HL: J5.8 (Pin_8)
- new net CCD_RG: J5.6 (Pin_6)
- new net GND: J2.3 (Pin_3), J2.4 (Pin_4), J3.3 (Pin_3), J3.4 (Pin_4), J4.3 (Pin_3), J4.4 (Pin_4), J5.3 (Pin_3), J5.4 (Pin_4)
- new net XSGV1: J3.10 (Pin_10)
- new net XSGV2: J3.8 (Pin_8)
- new net XSHT: J3.12 (Pin_12)
- new net XV1: J3.11 (Pin_11)
- new net XV2: J3.9 (Pin_9)
- new net XV3: J3.7 (Pin_7)
- new net XV4: J3.5 (Pin_5)
- no-connect marks 0 -> 5
