File: pcb/breakout-camera.kicad_pcb (KiCad board)
At the start: 2 copper layers, 38.1 x 39.4 mm, 36 parts, among them P10 CONN_01X14, P4 CONN_01X04, P5 CONN_01X01, Q1 2SC5095, Q2 MT3S20TU, Q3 2SC5095, Q4 MT3S20TU, U10 ICX825AQA, U4 TXB0104, U9 CXD3400N

Commit message: More work
Parts:
- removed C27: 0.1u, Capacitors_SMD:C_0603_HandSoldering
- removed P4: CONN_01X04, Socket_Strips:Socket_Strip_Straight_1x04
- removed P5: CONN_01X01, Socket_Strips:Socket_Strip_Straight_1x01
- removed U9: CXD3400N, w_smd_dil:tssop-20
- added C17: 0.1uF, Capacitors_SMD:C_0603_HandSoldering, F.Cu at (78.7, 67.8)
- added C18: 0.1uF/25V, Capacitors_SMD:C_0603_HandSoldering, F.Cu at (64.1, 56.8)
- added C19: 0.1uF/10V, Capacitors_SMD:C_0603_HandSoldering, F.Cu at (74.7, 67.8)
- added C22: 1.0uF/25V, Capacitors_SMD:C_0603_HandSoldering, F.Cu at (64.1, 55.1)
- added C23: 4.7uF/10V, Capacitors_SMD:c_elec_4x5.3, F.Cu at (69.2, 60.3)
- added G***: LOGO, w_logo:Logo_silk_CC-BY-SA_10x4.5mm, F.Cu at (88.9, 79.3)
- added Horizontal: HORI, xess:HDR_1x6, F.Cu at (76.2, 83.8)
- added P6: POWER, xess:HDR_1x6, F.Cu at (55.8, 64.8)
- added P7: VERT, xess:xess-1X08, F.Cu at (96.5, 64.7)
- added R23: 10.0k, Resistors_SMD:R_0603_HandSoldering, F.Cu at (81.7, 61.8)
- added REF**: OSH, xess:oshw-logo2, F.Cu at (63.5, 78.7)
- added U5: ADDI9023, engstad:csp-bga-bc-40-1, F.Cu at (76.2, 63.5)
- added hole_3mm: VAL**, w_details:hole_3mm, F.Cu at (96.5, 83.8)
- added hole_3mm: VAL**, w_details:hole_3mm, F.Cu at (56.2, 83.5)
- added hole_3mm: VAL**, w_details:hole_3mm, F.Cu at (56.2, 43.5)
- added hole_3mm: VAL**, w_details:hole_3mm, F.Cu at (96.2, 43.5)
- C12, C13: footprint Capacitors_SMD:C_0603 -> Capacitors_SMD:C_0603_HandSoldering
- C33: footprint Capacitors_SMD:C_0603_HandSoldering -> Capacitors_SMD:C_0805_HandSoldering
- P10: value CONN_01X14 -> OUTP; footprint w_pin_strip:pin_strip_14 -> xess:HDR_1x2
- U10: footprint camera:ICX825 -> sony:icx-825
- moved R18 34.2 mm to (88.3, 57.0), turned to 90 degrees
- moved C29 29.1 mm to (85.2, 58.2), turned to 180 degrees
- moved D2 26.2 mm to (86.5, 61.4), turned to 180 degrees
- moved C36 24.5 mm to (70.4, 51.7)
- moved C30 24.4 mm to (81.3, 58.2)
- moved C12 23.8 mm to (69.2, 75.6), turned to 180 degrees
- moved R22 21.3 mm to (74.4, 80.6), turned to 180 degrees
- moved R19 19.0 mm to (77.2, 58.2)
- moved C28 18.9 mm to (83.8, 67.3), turned to 0 degrees
- moved C35 18.0 mm to (76.2, 51.7), turned to 180 degrees
- moved C34 15.2 mm to (69.2, 67.3)
- moved U4 13.6 mm to (76.2, 76.2), turned to 0 degrees
- moved C31 9.86 mm to (83.8, 73.0), turned to 180 degrees
- moved C32 9.38 mm to (69.2, 73.0), turned to 0 degrees
- moved C13 8.92 mm to (83.8, 74.9)
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Connections:
- net /camera/H1S_1 renamed /camera/OH1
- net /camera/H2S_1 renamed /camera/OH2
- net /camera/LH1_1 renamed /camera/OLH
- net Net-(C28-Pad1) renamed /camera/SCKP
- C28 pad 2: Net-(C28-Pad2) -> /camera/SUBCK
- P10 pad 1: /camera/12V -> /camera/CCD_OUT1
- P10 pad 2: /camera/-7V -> /camera/CCD_OUT2
Routing:
- net GND: track 140.8 -> 191.1 mm, vias 12 -> 11
- net /camera/-7V: track 25.0 -> 65.0 mm
- net /camera/VDREN: track 0.00 -> 24.6 mm, vias 0 -> 1
- net /camera/5V0: track 26.7 -> 43.8 mm, vias 2 -> 0
- net /camera/XV3: track 38.1 -> 22.2 mm
- net /camera/XSHT: track 38.1 -> 23.4 mm
- net /camera/ORG: track 34.7 -> 21.3 mm, vias 0 -> 3
- net /camera/XV1: track 38.4 -> 25.0 mm
- net /camera/XV4: track 38.1 -> 24.7 mm
- net /camera/XSGV3: track 38.1 -> 24.9 mm
- net /camera/CCD_OUT1: track 8.16 -> 21.2 mm
- net /camera/SUB: track 26.6 -> 14.4 mm
- net /camera/SUBCK: track 0.00 -> 11.5 mm, vias 0 -> 2
- net Net-(C28-Pad2): track 11.4 -> 0.00 mm
- net /camera/OLH: track 28.3 -> 17.3 mm
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Other:
- board size 38.1 x 39.4 mm -> 50 x 50 mm
- net class Power: trace_width 0.254 -> 0.381; via_dia 0.4064 -> 0.6096; via_drill 0.2032 -> 0.4064
- board text added: "-7V"
- board text added: "12V"
- board text added: "3V3"
- board text added: "5V0"
- board text added: "EDS CamProto v0.1"
- board text added: "GND"
- board text added: "H1"
- board text added: "H2"
- board text added: "HEN"
- board text added: "HL"
- board text added: "O1"
- board text added: "O2"
- board text added: "RG"
- board text added: "SG1"
- board text added: "SG2"
- board text added: "SHT"
- board text added: "V1"
- board text added: "V2"
- board text added: "V3"
- board text added: "V4"
- board text added: "VEN"

Commit message: More work
Parts:
- removed Horizontal: HORI, xess:HDR_1x6
- added C24: 0.1uF, Capacitors_SMD:C_0603, F.Cu at (89.7, 46.9)
- added C27: 0.1uF, Capacitors_SMD:C_0603, F.Cu at (88.6, 42.7)
- added C50: 0.1uF, Capacitors_SMD:C_0603, F.Cu at (67.8, 47.2)
- added C51: 0.1uF, Capacitors_SMD:C_0603, F.Cu at (92.2, 46.0)
- added C52: 0.1uF, Capacitors_SMD:C_0603, F.Cu at (59.9, 45.7)
- added C53: 47uF, Capacitors_Tantalum_SMD:TantalC_SizeA_EIA-3216_Reflow, F.Cu at (85.6, 47.0)
- added C54: 47uF, Capacitors_Tantalum_SMD:TantalC_SizeA_EIA-3216_Reflow, F.Cu at (61.9, 45.7)
- added JP1: JUMPER3, xess:xess-JP2, F.Cu at (81.2, 45.7)
- added JP2: JUMPER3, xess:xess-JP2, F.Cu at (71.1, 45.7)
- added P4: HORI, xess:HDR_1x6, F.Cu at (76.2, 83.8)
- added P5: OUTP, xess:HDR_1x2, F.Cu at (96.5, 49.5)
- added R24: 249k, Resistors_SMD:R_0603, F.Cu at (89.6, 45.3)
- added R25: 10K, Resistors_SMD:R_0603, F.Cu at (91.1, 43.2)
- added R26: 10K, Resistors_SMD:R_0603, F.Cu at (64.7, 47.2)
- added R27: 249k, Resistors_SMD:R_0603, F.Cu at (64.7, 43.7)
- added U6: ADA4800, engstad:lfcsp-cp-6-4, F.Cu at (85.6, 44.4)
- added U9: ADA4800, engstad:lfcsp-cp-6-4, F.Cu at (67.8, 44.7)
- C26: value 0.1u -> 0.1uF; footprint Capacitors_SMD:C_0603_HandSoldering -> Capacitors_SMD:C_0603
- C29, C30, C31, C32: footprint Capacitors_SMD:C_0603_HandSoldering -> Capacitors_SMD:C_0603
- P7: footprint xess:xess-1X08 -> xess:HDR_1x8
- moved C26 21.3 mm to (67.6, 42.6), turned to 0 degrees
- moved REF** 8.03 mm to (55.8, 76.2)
- moved Q3 4.12 mm to (56.7, 52.3)
- moved Q4 4.12 mm to (61.7, 52.3)
- moved R14 4.12 mm to (61.7, 54.9)
- moved R15 4.12 mm to (56.7, 54.9)
- moved R20 4.12 mm to (56.7, 49.8)
- moved R21 4.12 mm to (61.7, 49.8)
- moved P10 3.84 mm to (76.2, 43.1)
- moved Q1 2.92 mm to (87.5, 52.5)
- moved Q2 2.92 mm to (92.6, 52.5)
- moved R10 2.92 mm to (92.6, 55.0)
- moved R11 2.92 mm to (87.5, 55.0)
- moved R12 2.92 mm to (87.5, 49.9)
- moved R13 2.92 mm to (92.6, 49.9)
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Connections:
- C26 pad 1: /camera/-7V -> Net-(C26-Pad1)
- Q2 pad 2: /camera/CCD_OUT1 -> /camera/VO1
- Q4 pad 2: /camera/CCD_OUT2 -> /camera/VO2
- R13 pad 1: /camera/CCD_OUT1 -> /camera/VO1
- R21 pad 1: /camera/CCD_OUT2 -> /camera/VO2
Routing:
- net /camera/12V: track 113.6 -> 154.2 mm
- net GND: track 191.1 -> 231.3 mm, vias 11 -> 15
- net /camera/EO2: track 0.00 -> 39.6 mm, vias 0 -> 1
- net /camera/VO2: track 0.00 -> 33.9 mm
- net /camera/VO1: track 0.00 -> 32.3 mm
- net /camera/SUB: track 14.4 -> 2.64 mm
- net /camera/CCD_OUT1: track 21.2 -> 9.98 mm
- net /camera/CCD_OUT2: track 20.8 -> 10.0 mm
- net /camera/EO1: track 0.00 -> 7.60 mm
- net Net-(JP2-Pad3): track 0.00 -> 6.38 mm
- net Net-(JP1-Pad3): track 0.00 -> 4.89 mm
- net Net-(C24-Pad1): track 0.00 -> 4.88 mm
- net /camera/-7V: track 65.0 -> 60.2 mm
- net Net-(C27-Pad2): track 0.00 -> 4.19 mm
- net Net-(C26-Pad1): track 0.00 -> 3.96 mm
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Other:
- board text added: "Buf Off"
- board text added: "EO1"
- board text added: "EO2"

Commit message: ready for ordering
Parts:
- moved hole_3mm 0.45 mm to (96.2, 83.5)
Connections:
- Q1 pad 2: /camera/E1 -> /camera/VOUT1
- Q1 pad 3: /camera/VOUT1 -> /camera/E1
- Q2 pad 2: /camera/VO1 -> /camera/12V
- Q2 pad 3: /camera/12V -> /camera/VO1
- Q3 pad 2: /camera/E2 -> /camera/VOUT2
- Q3 pad 3: /camera/VOUT2 -> /camera/E2
- Q4 pad 2: /camera/VO2 -> /camera/12V
- Q4 pad 3: /camera/12V -> /camera/VO2
Routing:
- net GND: track 231.3 -> 255.0 mm, vias 15 -> 17
- net /camera/SUB: track 2.64 -> 14.2 mm
- net /camera/12V: track 154.2 -> 164.0 mm
- net /camera/XSGV2: track 25.0 -> 19.7 mm
- net /camera/E1: track 2.31 -> 4.32 mm
- net /camera/E2: track 2.26 -> 4.27 mm
- net /camera/VO1: track 32.3 -> 34.3 mm
- net /camera/VO2: track 33.9 -> 35.6 mm
- net /camera/VOUT1: track 11.8 -> 13.2 mm
- net /camera/VOUT2: track 13.4 -> 14.6 mm
- net /camera/SCKP: track 13.1 -> 14.2 mm
- net /camera/ORG: track 19.7 -> 18.6 mm
- net /camera/VT1: track 9.27 -> 8.46 mm
- net /camera/3V3: track 65.3 -> 65.8 mm
Other:
- rule pad_to_mask_clearance: 0 -> 0.0635

Commit message: Latest, greatest.
Parts:
- removed U4: TXB0104, Housings_SSOP:TSSOP-14_4.4x5mm_Pitch0.65mm
- added ?: , xess:oshw-logo2, F.Cu at (92.9, 112.6)
- added C1: 22.0uF, Capacitors_SMD:C_1206_HandSoldering, F.Cu at (110.5, 130.0)
- added C1: 1.0uF, Capacitors_SMD:C_0805_HandSoldering, F.Cu at (65.0, 140.7)
- added C10: 0.1uF, Capacitors_SMD:C_0805_HandSoldering, F.Cu at (86.6, 138.3)
- added C11: 10uF, Capacitors_SMD:C_0805_HandSoldering, F.Cu at (76.9, 118.0)
- added C14: 10.0uF, Capacitors_SMD:C_0805_HandSoldering, F.Cu at (91.9, 119.9)
- added C15: 10.0uF, Capacitors_SMD:C_0805_HandSoldering, F.Cu at (63.1, 119.6)
- added C16: 470pF, Capacitors_SMD:C_0402, F.Cu at (65.9, 126.0)
- added C2: 47nF, Capacitors_SMD:C_0603_HandSoldering, F.Cu at (106.2, 139.8)
- added C2: 1.0uF, Capacitors_SMD:C_0805_HandSoldering, F.Cu at (90.2, 143.0)
- added C20: 0.1uF, Capacitors_SMD:C_0603_HandSoldering, F.Cu at (88.4, 122.8)
- added C21: 10.0uF, Capacitors_SMD:C_0805_HandSoldering, F.Cu at (67.7, 120.8)
- added C25: 47uF, Capacitors_SMD:C_1206_HandSoldering, F.Cu at (93.7, 124.2)
- added C3: 47nF, Capacitors_SMD:C_0603_HandSoldering, F.Cu at (110.1, 139.8)
- added C3: 47pF, Capacitors_SMD:C_0805_HandSoldering, F.Cu at (94.8, 139.9)
- added C4: 1.0uF, Capacitors_SMD:C_0603_HandSoldering, F.Cu at (114.3, 132.0)
- added C4: 2.2uF, Capacitors_SMD:C_0603_HandSoldering, F.Cu at (79.7, 121.7)
- added C5: 1.0uF, Capacitors_SMD:C_0603_HandSoldering, F.Cu at (114.3, 133.9)
- added C5: 47pF, Capacitors_SMD:C_0805_HandSoldering, F.Cu at (93.9, 135.0)
- added C6: 10.0uF, Capacitors_SMD:C_1206_HandSoldering, F.Cu at (102.6, 121.4)
- added C6: 1.0uF, Capacitors_SMD:C_0805_HandSoldering, F.Cu at (90.2, 145.4)
- added C7: 10.0uF, Capacitors_SMD:C_1206_HandSoldering, F.Cu at (109.5, 121.4)
- added C7: 100nF, Capacitors_SMD:C_0805_HandSoldering, F.Cu at (91.1, 131.3)
- added C8: 1.0uF/11mOhm, Capacitors_SMD:C_0805_HandSoldering, F.Cu at (76.7, 133.2)
- added C9: 4.7uF, Capacitors_SMD:C_1206_HandSoldering, F.Cu at (85.0, 132.4)
- added D1: <40pF@5V, camera:PowerDI_123, F.Cu at (102.0, 126.1)
- added D1: 9V/5W, Diodes_SMD:SMB_Standard, F.Cu at (74.3, 142.5)
- added D2: <40pF@5V, camera:PowerDI_123, F.Cu at (109.8, 125.9)
- added JP3: JUMPER3, xess:xess-JP2, F.Cu at (83.0, 66.7)
- added JP4: JUMPER3, xess:xess-JP2, F.Cu at (83.1, 64.2)
- added JP5: JUMPER3, xess:xess-JP2, F.Cu at (75.0, 129.0)
- added L1: 3.3uH, camera:Inductor_XAL40_SMD, F.Cu at (103.0, 131.1)
- added L1: 15uH, w_smd_inductors:inductor_smd_0805, F.Cu at (95.7, 144.1)
- added L2: 6.8uH, camera:Inductor_XAL40_SMD, F.Cu at (105.9, 126.3)
- added L2: 15uH, w_smd_inductors:inductor_smd_0805, F.Cu at (86.6, 145.9)
- added L3: 2.0uH, w_smd_inductors:inductor_smd_0805, F.Cu at (76.1, 125.5)
- added L4: 10uH, w_smd_inductors:inductor_smd_0805, F.Cu at (86.6, 142.2)
- added L8: 2.2uH, w_smd_inductors:inductor_smd_0805, F.Cu at (94.5, 120.5)
- added P1: PIN, xess:HDR_1x2, F.Cu at (113.4, 116.2)
- added P11: CONN_01X01, xess:HDR_1x1, F.Cu at (80.0, 129.0)
- added P12: CONN_01X01, xess:HDR_1x1, F.Cu at (87.2, 111.2)
- added P2: POUT, xess:HDR_1x3, F.Cu at (103.3, 116.2)
- added P8: CONN_01X06, Pin_Headers:Pin_Header_Straight_1x06, F.Cu at (71.9, 111.2)
- added P9: CONN_01X02, Pin_Headers:Pin_Header_Straight_1x02, F.Cu at (67.1, 144.0)
- added R1: 3.7k, Resistors_SMD:R_0603_HandSoldering, F.Cu at (108.0, 139.6)
- added R1: 10.0k, Resistors_SMD:R_0805_HandSoldering, F.Cu at (65.0, 138.0)
- added R16: 13.7k, Resistors_SMD:R_0402, F.Cu at (85.1, 122.5)
- added R17: 10.0k, Resistors_SMD:R_0402, F.Cu at (85.1, 120.1)
- added R2: 3.5k, Resistors_SMD:R_0603_HandSoldering, F.Cu at (111.9, 139.6)
- added R2: 324k, Resistors_SMD:R_0603_HandSoldering, F.Cu at (91.9, 134.7)
- added R28: 10.0k, Resistors_SMD:R_0603_HandSoldering, F.Cu at (76.1, 94.7)
- added R3: 100K, Resistors_SMD:R_0603_HandSoldering, F.Cu at (103.2, 137.0)
- added R3: 10.0k, Resistors_SMD:R_0603_HandSoldering, F.Cu at (64.8, 135.7)
- added R4: 100K, Resistors_SMD:R_0603_HandSoldering, F.Cu at (114.3, 135.9)
- added R4: 51.1k, Resistors_SMD:R_0603_HandSoldering, F.Cu at (76.8, 137.9)
- added R5: 1.4M, Resistors_SMD:R_0603_HandSoldering, F.Cu at (103.2, 135.1)
- added R5: 68.1k, Resistors_SMD:R_0603_HandSoldering, F.Cu at (76.8, 135.6)
- added R6: 1.07M, Resistors_SMD:R_0603_HandSoldering, F.Cu at (115.5, 138.8)
- added R6: 53.6k, Resistors_SMD:R_0603_HandSoldering, F.Cu at (64.8, 133.6)
- added R7: 324k, Resistors_SMD:R_0603_HandSoldering, F.Cu at (88.3, 134.9)
- added R8: 80.6k, Resistors_SMD:R_0402, F.Cu at (62.2, 126.1)
- added R9: 105k, Resistors_SMD:R_0402, F.Cu at (64.1, 127.8)
- added T1: NET-TIE, NetTie:NET-TIE-1mm, F.Cu at (107.6, 129.7)
- added T1: NET-TIE, Oddities:NetTie-I_Connected_SMD, B.Cu at (76.5, 125.5)
- added T2: NET-TIE, Oddities:NetTie-I_Connected_SMD, F.Cu at (65.3, 117.3)
- added U1: ADP5071, Housings_DFN_QFN:QFN-20-1EP_4x4mm_Pitch0.5mm, F.Cu at (109.0, 134.1)
- added U1: TPS2420, Housings_DFN_QFN:QFN-16-1EP_4x4mm_Pitch0.65mm, F.Cu at (71.1, 136.2)
- added U12: SN74LVC8T245, Housings_SSOP:TSSOP-24_4.4x7.8mm_Pitch0.65mm, F.Cu at (83.1, 95.3)
- added U2: LT3487, Housings_DFN_QFN:DFN-10-1EP_3x3mm_Pitch0.5mm, F.Cu at (90.5, 139.2)
- added U3: TPS63002, Housings_DFN_QFN:DFN-10-1EP_3x3mm_Pitch0.5mm, F.Cu at (76.5, 121.9)
- added U7: TPS56x200, Housings_SOT-23_SOT-143_TSOT-6:SOT-23-6, F.Cu at (88.4, 119.8)
- added U8: LMZ10500, engstad:llp-8, F.Cu at (63.6, 122.8)
- moved REF** 29.8 mm to (70.2, 102.3)
- moved R22 22.8 mm to (90.7, 96.7)
- moved G*** 21.7 mm to (101.7, 96.8)
- moved C18 19.7 mm to (70.6, 76.9)
- moved C52 19.7 mm to (66.8, 64.2)
- moved D2 19.7 mm to (93.4, 79.9)
- moved P5 19.7 mm to (103.4, 68.0)
- moved R10 19.7 mm to (99.5, 73.5)
- moved R11 19.7 mm to (94.4, 73.5)
- moved R13 19.7 mm to (99.5, 68.4)
- moved R14 19.7 mm to (68.6, 73.4)
- moved R15 19.7 mm to (63.6, 73.4)
- moved R20 19.7 mm to (63.6, 68.3)
- moved R21 19.7 mm to (68.6, 68.3)
- moved R23 19.7 mm to (88.6, 80.3)
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Connections:
- net /camera/OH1 renamed /camera/H1_5V
- net /camera/OH2 renamed /camera/H2_5V
- net /camera/OLH renamed /camera/LH_5V
- net /camera/ORG renamed /camera/RG_5V
- P4 pad 6: /camera/ENH -> /camera/~ENH~
- Q2 pad 3: /camera/VO1 -> Net-(JP3-Pad3)
- Q4 pad 3: /camera/VO2 -> Net-(JP4-Pad3)
- R13 pad 1: /camera/VO1 -> Net-(JP3-Pad3)
- R21 pad 1: /camera/VO2 -> Net-(JP4-Pad3)
- R22 pad 1: /camera/ENH -> /camera/3V3
- R22 pad 2: GND -> /camera/~ENH~
Routing:
- net GND: track 255.0 -> 539.7 mm, vias 17 -> 45
- net /power-supply/5V5: track 0.00 -> 137.3 mm, vias 0 -> 4
- net (no net): track 0.00 -> 122.6 mm
- net VIN*: track 0.00 -> 57.4 mm
- net /power-supply/PGND: track 0.00 -> 50.6 mm, vias 0 -> 7
- net /power-supply/-7V: track 0.00 -> 46.2 mm
- net Net-(JP3-Pad3): track 0.00 -> 45.0 mm
- net /power-supply/+12V: track 0.00 -> 35.7 mm, vias 0 -> 2
- net Net-(JP4-Pad3): track 0.00 -> 34.0 mm
- net /-7V: track 0.00 -> 33.8 mm, vias 0 -> 2
- net /power-supply/1V8: track 0.00 -> 32.0 mm
- net +5V: track 0.00 -> 28.7 mm, vias 0 -> 2
- net /camera/VO2: track 35.6 -> 10.3 mm
- net /0V: track 0.00 -> 24.3 mm
- net /power-supply/3V3: track 0.00 -> 24.2 mm, vias 0 -> 2
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- added copper zone on F.Cu, net +5V
- added copper zone on F.Cu, net /+12V
- added copper zone on F.Cu, net /-7V
- added copper zone on F.Cu, net /0V
- added copper zone on B.Cu, net /power-supply/PGND
- added copper zone on F.Cu, net /power-supply/PGND
- added copper zone on F.Cu, net Net-(D1-Pad2)
- added copper zone on F.Cu, net Net-(D2-Pad1)
- added copper zone on F.Cu, net Net-(L1-Pad1)
Other:
- board size 50 x 50 mm -> 61.7 x 92.1 mm
- net class Default: clearance 0.1016 -> 0.1524; trace_width 0.1524 -> 0.254; via_dia 0.4064 -> 0.604774; via_drill 0.2032 -> 0.299974
- net class Power: clearance 0.1016 -> 0.1524; trace_width 0.381 -> 0.508; via_dia 0.6096 -> 0.604774; via_drill 0.4064 -> 0.299974
- rule pad_to_mask_clearance: 0.0635 -> 0
- rule trace_clearance: 0.1016 -> 0.1524
- rule via_min_drill: 0.2032 -> 0.299974
- rule via_min_size: 0.4064 -> 0.604774
- board text added: "+"
- board text added: "-"
- board text added: "-7"
- board text added: "1.8"
- board text added: "12"
- board text added: "3.3"
- board text added: "5.0"
- board text added: "5.5"
- board text added: "Astro Power"
- board text added: "CamProto v0.1"
- board text added: "Engstad Design Studio"
- board text added: "~HEN"
- board text removed: "Buf Off"
- board text removed: "EDS CamProto v0.1"
- board text removed: "HEN"

Commit message: latest
Other:
- board text added: "JP1: [1-2] VO1 -> CCD_OUT1 [2-3] VO1 -> ADA4800 -> CCD_OUT1 JP3: [1-2] VOUT1 -> VO1 [2-3] VOUT1 -> Q1Q2 -> VO1"

Commit message: work
Other:
- board text added: "No: 22uF"
- board text added: "Soft start (short to 5V)"
Changed lines of the file:
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@@
-(kicad_pcb (version 4) (host pcbnew 0.201510170916+6271~30~ubuntu15.04.1-product)
+(kicad_pcb (version 4) (host pcbnew 0.201512191116+6384~39~ubuntu15.04.1-stable)
   (general
     (links 326)
     (no_connects 3)
-    (area 42.000001 47.6006 143.045502 162.700001)
+    (area 42.000001 40.776 143.045502 162.700001)
     (thickness 1.6)
-    (drawings 111)
+    (drawings 113)
     (tracks 1853)
     (zones 0)
@@
       (effects (font (size 1 1) (thickness 0.15)))
     )
-    (fp_text value 1.0uF (at 3.9 -1.6) (layer F.Fab)
+    (fp_text value 1.0uF (at -0.3422 14.273) (layer F.Fab)
       (effects (font (size 1 1) (thickness 0.15)))
     )
@@
       (effects (font (size 1 1) (thickness 0.15)))
     )
-    (fp_text value 47pF (at 0.228 -1.774 180) (layer F.Fab)
+    (fp_text value 47pF (at -0.1062 15.497 180) (layer F.Fab)
       (effects (font (size 1 1) (thickness 0.15)))
     )
@@
       (effects (font (size 1 1) (thickness 0.15)))
     )
-    (fp_text value 47pF (at 0.104 1.52 270) (layer F.Fab)
+    (fp_text value 47pF (at -17.643 -0.3822 270) (layer F.Fab)
       (effects (font (size 1 1) (thickness 0.15)))
     )
@@
       (effects (font (size 1 1) (thickness 0.15)))
     )
-    (fp_text value 1.0uF (at 3.9 -1.2) (layer F.Fab)
+    (fp_text value 1.0uF (at -0.3122 13.373) (layer F.Fab)
       (effects (font (size 1 1) (thickness 0.15)))
     )
@@
       (effects (font (size 1 1) (thickness 0.15)))
     )
-    (fp_text value 100nF (at -2.288 1.992 180) (layer F.Fab)
+    (fp_text value 100nF (at 0.0522 -18.563 180) (layer F.Fab)
       (effects (font (size 1 1) (thickness 0.15)))
     )
@@
       (effects (font (size 1 1) (thickness 0.15)))
     )
-    (fp_text value 1.0uF/11mOhm (at 2.82936 16.94392) (layer F.Fab)
+    (fp_text value 1.0uF/11mOhm (at -1.7252 16.818) (layer F.Fab)
       (effects (font (size 1 1) (thickness 0.15)))
     )
@@
       (effects (font (size 1 1) (thickness 0.15)))
     )
-    (fp_text value 0.1uF (at 1.422 3.372 360) (layer F.Fab)
+    (fp_text value 0.1uF (at 16.973 0.9222 450) (layer F.Fab)
       (effects (font (size 1 1) (thickness 0.15)))
     )
@@
       (effects (font (size 1 1) (thickness 0.15)))
     )
-    (fp_text value 324k (at 0 1.9 270) (layer F.Fab)
+    (fp_text value 324k (at 17.968 -0.1278 270) (layer F.Fab)
       (effects (font (size 1 1) (thickness 0.15)))
     )
@@
       (effects (font (size 1 1) (thickness 0.15)))
     )
-    (fp_text value 51.1k (at -1.16192 16.06074) (layer F.Fab)
+    (fp_text value 51.1k (at -2.5052 16.158) (layer F.Fab)
       (effects (font (size 1 1) (thickness 0.15)))
     )
@@
       (effects (font (size 1 1) (thickness 0.15)))
     )
-    (fp_text value 68.1k (at -1.21018 16.52686) (layer F.Fab)
+    (fp_text value 68.1k (at -2.5052 16.578) (layer F.Fab)
       (effects (font (size 1 1) (thickness 0.15)))
     )
@@
       (effects (font (size 1 1) (thickness 0.15)))
     )
-    (fp_text value 324k (at 0 1.9 180) (layer F.Fab)
+    (fp_text value 324k (at 0.7192 -17.768 180) (layer F.Fab)
       (effects (font (size 1 1) (thickness 0.15)))
     )
@@
       (effects (font (size 1 1) (thickness 0.15)))
     )
-    (fp_text value LT3487 (at 0 2.575 90) (layer F.Fab)
+    (fp_text value LT3487 (at -16.303 -0.9872 180) (layer F.Fab)
       (effects (font (size 1 1) (thickness 0.15)))
     )
@@
       (effects (font (size 1 1) (thickness 0.15)))
     )
-    (fp_text value 4.7uF (at 0 2.3 90) (layer F.Fab)
+    (fp_text value 4.7uF (at -19.408 -0.8052 90) (layer F.Fab)
       (effects (font (size 1 1) (thickness 0.15)))
     )
@@
       (net 126 /power-supply/PGND))
   )
+  (gr_text "Soft start (short to 5V)" (at 103.23 150.04) (layer F.Fab)
+    (effects (font (size 1 1) (thickness 0.2)))
+  )
+  (gr_text "No: 22uF" (at 98.06 155.76) (layer F.Fab)
+    (effects (font (size 1.5 1.5) (thickness 0.3)))
+  )
   (gr_text "JP1: [1-2] VO1 ->  CCD_OUT1\n     [2-3] VO1 -> ADA4800 -> CCD_OUT1\nJP3: [1-2] VOUT1 -> VO1\n     [2-3] VOUT1 -> Q1Q2 -> VO1\n\n\n" (at 70.385 45.376) (layer Eco1.User)
