File: pcb/breakout-camera.kicad_pcb (KiCad board)
At the start: 2 copper layers, 38.1 x 39.4 mm, 36 parts, among them P10 CONN_01X14, P4 CONN_01X04, P5 CONN_01X01, Q1 2SC5095, Q2 MT3S20TU, Q3 2SC5095, Q4 MT3S20TU, U10 ICX825AQA, U4 TXB0104, U9 CXD3400N

Commit message: Start up work to revive this project.
Other:
- net class Default removed
- net class Power removed
