File: pcb/camera.sch (KiCad schematic (older format))
At the start: 41 parts, among them P10 OUTP, P4 HORI, P6 POWER, P7 VERT, Q1 2SC5095, Q2 MT3S20TU, Q3 2SC5095, Q4 MT3S20TU, U10 ICX825AQA, U4 TXB0104, U5 ADDI9023

Commit message: Adding ADDI4800 to schematics
Parts:
- added C? (x3): 0.1uF, symbol C_Small
- added C?: 47uF, Capacitors_SMD:c_elec_4x5.3, symbol CP1_Small
- added R?: 96k, symbol R_Small
- added R?: 249k, symbol R_Small
- added U? (x2): ADA4800, symbol ADA4800
Connections:
- wire segments 110 -> 124
Changed lines of the file:
@@
 SCKP
 NoConn ~ 4850 50
+$Comp
+L ADA4800 U?
+U 1 1 55DCE02F
+P 4450 6700
+F 0 "U?" H 4450 6250 60  0000 C CNN
+F 1 "ADA4800" H 4450 7150 60  0000 C CNN
+F 2 "" H 5450 6300 60  0000 C CNN
+F 3 "" H 5450 6300 60  0000 C CNN
+	1    4450 6700
+	1    0    0    -1
+$EndComp
+$Comp
+L ADA4800 U?
+U 1 1 55DCE116
+P 4450 5550
+F 0 "U?" H 4450 5100 60  0000 C CNN
+F 1 "ADA4800" H 4450 6000 60  0000 C CNN
+F 2 "" H 5450 5150 60  0000 C CNN
+F 3 "" H 5450 5150 60  0000 C CNN
+	1    4450 5550
+	1    0    0    -1
+$EndComp
+Text Label 4000 5300 2    60   ~ 0
+CCD_OUT1
+$Comp
+L GND #PWR?
+U 1 1 55DCE489
+P 3950 5550
+F 0 "#PWR?" H 3950 5300 50  0001 C CNN
+F 1 "GND" H 3950 5400 50  0000 C CNN
+F 2 "" H 3950 5550 60  0000 C CNN
+F 3 "" H 3950 5550 60  0000 C CNN
+	1    3950 5550
+	0    1    1    0
+$EndComp
+Wire Wire Line
+	4000 5550 3950 5550
+$Comp
+L R_Small R?
+U 1 1 55DCE9C3
+P 5000 5100
+F 0 "R?" H 5030 5120 50  0000 L CNN
+F 1 "96k" H 5030 5060 50  0000 L CNN
+F 2 "" H 5000 5100 60  0000 C CNN
+F 3 "" H 5000 5100 60  0000 C CNN
+	1    5000 5100
+	1    0    0    -1
+$EndComp
+Wire Wire Line
+	4900 5300 5150 5300
+Wire Wire Line
+	5000 5300 5000 5200
+Wire Wire Line
+	5000 5000 5000 4900
+Text Label 5000 4900 0    60   ~ 0
+12V
+$Comp
+L C_Small C?
+U 1 1 55DCF0DB
+P 5250 5300
+F 0 "C?" H 5260 5370 50  0000 L CNN
+F 1 "0.1uF" H 5260 5220 50  0000 L CNN
+F 2 "" H 5250 5300 60  0000 C CNN
+F 3 "" H 5250 5300 60  0000 C CNN
+	1    5250 5300
+	0    1    1    0
+$EndComp
+Connection ~ 5000 5300
+Wire Wire Line
+	5350 5300 5450 5300
+$Comp
+L GND #PWR?
+U 1 1 55DCF31D
+P 5450 5300
+F 0 "#PWR?" H 5450 5050 50  0001 C CNN
+F 1 "GND" H 5450 5150 50  0000 C CNN
+F 2 "" H 5450 5300 60  0000 C CNN
+F 3 "" H 5450 5300 60  0000 C CNN
+	1    5450 5300
+	0    -1   -1   0
+$EndComp
+Wire Wire Line
+	4900 5550 5900 5550
+Text Label 5900 5550 0    60   ~ 0
+12V
+$Comp
+L R_Small R?
+U 1 1 55DCF53E
+P 5200 5700
+F 0 "R?" H 5230 5720 50  0000 L CNN
+F 1 "249k" H 5230 5660 50  0000 L CNN
+F 2 "" H 5200 5700 60  0000 C CNN
+F 3 "" H 5200 5700 60  0000 C CNN
+	1    5200 5700
+	1    0    0    -1
+$EndComp
+Wire Wire Line
+	4900 5800 5200 5800
+$Comp
+L C_Small C?
+U 1 1 55DCF845
+P 4950 5950
+F 0 "C?" H 4960 6020 50  0000 L CNN
+F 1 "0.1uF" H 4960 5870 50  0000 L CNN
+F 2 "" H 4950 5950 60  0000 C CNN
+F 3 "" H 4950 5950 60  0000 C CNN
+	1    4950 5950
+	1    0    0    -1
+$EndComp
+$Comp
+L C_Small C?
+U 1 1 55DCF919
+P 5450 5750
+F 0 "C?" H 5460 5820 50  0000 L CNN
+F 1 "0.1uF" H 5460 5670 50  0000 L CNN
+F 2 "" H 5450 5750 60  0000 C CNN
+F 3 "" H 5450 5750 60  0000 C CNN
+	1    5450 5750
+	1    0    0    -1
+$EndComp
+$Comp
+L CP1_Small C?
+U 1 1 55DCFBB7
+P 5700 5750
+F 0 "C?" H 5710 5820 50  0000 L CNN
+F 1 "47uF" H 5710 5670 50  0000 L CNN
+F 2 "Capacitors_SMD:c_elec_4x5.3" H 5700 5750 60  0001 C CNN
+F 3 "" H 5700 5750 60  0000 C CNN
+	1    5700 5750
+	1    0    0    -1
+$EndComp
+Wire Wire Line
+	5700 5550 5700 5650
+Connection ~ 5700 5550
+Wire Wire Line
+	5700 5850 5700 5900
+$Comp
+L GND #PWR?
+U 1 1 55DD024A
+P 5700 5900
+F 0 "#PWR?" H 5700 5650 50  0001 C CNN
+F 1 "GND" H 5700 5750 50  0000 C CNN
+F 2 "" H 5700 5900 60  0000 C CNN
+F 3 "" H 5700 5900 60  0000 C CNN
+	1    5700 5900
+	1    0    0    -1
+$EndComp
+Wire Wire Line
+	5450 5550 5450 5650
+Connection ~ 5450 5550
+$Comp
+L GND #PWR?
+U 1 1 55DD0507
+P 5450 5900
+F 0 "#PWR?" H 5450 5650 50  0001 C CNN
+F 1 "GND" H 5450 5750 50  0000 C CNN
+F 2 "" H 5450 5900 60  0000 C CNN
+F 3 "" H 5450 5900 60  0000 C CNN
+	1    5450 5900
+	1    0    0    -1
+$EndComp
+Wire Wire Line
+	5450 5850 5450 5900
+Wire Wire Line
+	4950 5800 4950 5850
+Connection ~ 4950 5800
+Wire Wire Line
+	4950 6050 4950 6100
+$Comp
+L GND #PWR?
+U 1 1 55DD094B
+P 4950 6100
+F 0 "#PWR?" H 4950 5850 50  0001 C CNN
+F 1 "GND" H 4950 5950 50  0000 C CNN
+F 2 "" H 4950 6100 60  0000 C CNN
+F 3 "" H 4950 6100 60  0000 C CNN
+	1    4950 6100
+	1    0    0    -1
+$EndComp
+Wire Wire Line
+	5200 5550 5200 5600
+Connection ~ 5200 5550
 $EndSCHEMATC

Commit message: More work
Parts:
- removed U?: ADA4800, symbol ADA4800
- added C26, C50, C52: 0.1uF, Capacitors_SMD:C_0603, symbol C_Small
- added C54: 47uF, Capacitors_Tantalum_SMD:TantalC_SizeA_EIA-3216_Reflow, symbol CP1_Small
- added JP1, JP2: JUMPER3, xess:xess-JP2, symbol JUMPER3
- added P5: OUTP, xess:HDR_1x2, symbol CONN_01X02
- added R26: 10K, Resistors_SMD:R_0603, symbol R_Small
- added R27: 249k, Resistors_SMD:R_0603, symbol R_Small
- added U9: ADA4800, engstad:lfcsp-cp-6-4, symbol ADA4800
- C24, C27, C51: renamed from C?; footprint (none) -> Capacitors_SMD:C_0603
- C53: renamed from C?; footprint Capacitors_SMD:c_elec_4x5.3 -> Capacitors_Tantalum_SMD:TantalC_SizeA_EIA-3216_Reflow
- R24: renamed from R?; footprint (none) -> Resistors_SMD:R_0603
- R25: renamed from R?; value 96k -> 10K; footprint (none) -> Resistors_SMD:R_0603
- U6: renamed from U?; footprint (none) -> engstad:lfcsp-cp-6-4
Connections:
- net labels added: EO1, EO2, VO1, VO2
- wire segments 124 -> 152
Other:
- moved on the sheet: C24, R10, R11, R12, R13, R14, R15, R20, R21, R24

Commit message: ready for ordering
Parts:
- Q1, Q2, Q3, Q4: symbol Q_NPN_BEC -> Q_NPN_BCE
Changed lines of the file:
@@
 $EndComp
 $Comp
-L Q_NPN_BEC Q1
+L Q_NPN_BCE Q1
 U 1 1 5590D88C
 P 7450 5150
@@
 $EndComp
 $Comp
-L Q_NPN_BEC Q2
+L Q_NPN_BCE Q2
 U 1 1 5590DA54
 P 7900 4800
@@
 $EndComp
 $Comp
-L Q_NPN_BEC Q3
+L Q_NPN_BCE Q3
 U 1 1 5590FE91
 P 9550 5150
@@
 $EndComp
 $Comp
-L Q_NPN_BEC Q4
+L Q_NPN_BCE Q4
 U 1 1 5590FF55
 P 10000 4800

Commit message: Latest, greatest.
Parts:
- removed U4: TXB0104, Housings_SSOP:TSSOP-14_4.4x5mm_Pitch0.65mm, symbol TXB0104
- added JP3, JP4: JUMPER3, xess:xess-JP2, symbol JUMPER3
- added R28: 10.0k, Resistors_SMD:R_0603_HandSoldering, symbol R
- added U12: SN74LVC8T245, Housings_SSOP:TSSOP-24_4.4x7.8mm_Pitch0.65mm, symbol SN74LVC8T245
Connections:
- net 3V3: now also R22.1, R28.1, U12.1 (VCCA)
- net 5V0: now also U12.23 (VCCB), U12.24 (VCCB)
- net GND: now also U12.11 (GND), U12.12 (GND), U12.13 (GND); no longer R22.2
- net H1: now also U12.3 (A1)
- net H2: now also U12.4 (A2)
- net HL: now also U12.5 (A3)
- net RG: now also U12.6 (A4)
- net RG_2: now also U10.27 (RG_2); no longer U10.22 (H2T_2)
- net VO1: now also JP3.2; no longer Q2.3 (E), R13.1
- net VO2: now also JP4.2; no longer Q4.3 (E), R21.1
- net VOUT1: now also JP3.1
- net VOUT2: now also JP4.1
- net ENH renamed ~ENH~
- net ~ENH~: now also R22.2, U12.22 (~OE); no longer R22.1
- net OH1 renamed H1_5V
- net H1_5V: now also U12.21 (B1)
- net OH2 renamed H2_5V
- net H2_5V: now also U10.22 (H2T_2), U10.23 (H2S_2), U12.20 (B2); no longer U10.26 (LH1_2), U10.27 (RG_2)
- net OLH renamed LH_5V
- net LH_5V: now also U10.26 (LH1_2), U12.19 (B3); no longer U10.23 (H2S_2)
- net ORG renamed RG_5V
- net RG_5V: now also U12.18 (B4)
- new net: JP3.3, Q2.3 (E), R13.1
- new net: JP4.3, Q4.3 (E), R21.1
- new net: R28.2, U12.2 (DIR)
- no-connect marks 20 -> 28
Other:
- moved on the sheet: C12, C13, C31, C32, C33, C34, C35, C36, C37, P10, P4, P5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

Commit message: latest
Other:
- note added: "JP1: [1-2] VO1 -> CCD_OUT1\n [2-3] VO1 -> ADA4800 -> CCD_OUT1\nJP3: [1-2] VOUT1 -> VO1\n [2-3] VOUT1 -> Q1Q2 -> VO1\n\n\n"
Changed lines of the file:
@@
 Text Label 5700 2350 1    60   ~ 0
 H2_5V
+Text Notes 7500 3850 0    60   ~ 0
+JP1: [1-2] VO1 ->  CCD_OUT1\n     [2-3] VO1 -> ADA4800 -> CCD_OUT1\nJP3: [1-2] VOUT1 -> VO1\n     [2-3] VOUT1 -> Q1Q2 -> VO1\n\n\n
 $EndSCHEMATC

Commit message: work
Parts:
- C100: renamed from C36; footprint Capacitors_SMD:c_elec_4x5.3 -> w_smd_cap:c_elec_4x5.3
- C101: renamed from C37; footprint Capacitors_SMD:c_elec_4x5.3 -> w_smd_cap:c_elec_4x5.3
- C77: renamed from C17; footprint Capacitors_SMD:C_0603_HandSoldering -> smd:SM0603
- C78: renamed from C12; footprint Capacitors_SMD:C_0603_HandSoldering -> smd:SM0603
- C79: renamed from C18; footprint Capacitors_SMD:C_0603_HandSoldering -> smd:SM0603
- C80: renamed from C22; footprint Capacitors_SMD:C_0603_HandSoldering -> smd:SM0603
- C81: renamed from C19; footprint Capacitors_SMD:C_0603_HandSoldering -> smd:SM0603
- C82: renamed from C23; footprint Capacitors_SMD:c_elec_4x5.3 -> w_smd_cap:c_elec_4x5.3
- C83: renamed from C13; footprint Capacitors_SMD:C_0603_HandSoldering -> smd:SM0603
- C84: renamed from C28; footprint Capacitors_SMD:c_elec_4x5.3 -> w_smd_cap:c_elec_4x5.3
- C85: renamed from C26; footprint Capacitors_SMD:C_0603 -> w_smd_cap:c_0603
- C86: renamed from C31; footprint Capacitors_SMD:C_0603 -> w_smd_cap:c_0603
- C87: renamed from C32; footprint Capacitors_SMD:C_0603 -> w_smd_cap:c_0603
- C88: renamed from C24; footprint Capacitors_SMD:C_0603 -> w_smd_cap:c_0603
- C89: renamed from C27; footprint Capacitors_SMD:C_0603 -> w_smd_cap:c_0603
- C90: renamed from C50; footprint Capacitors_SMD:C_0603 -> w_smd_cap:c_0603
- C91: renamed from C51; footprint Capacitors_SMD:C_0603 -> w_smd_cap:c_0603
- C92: renamed from C52; footprint Capacitors_SMD:C_0603 -> w_smd_cap:c_0603
- C93: renamed from C29; footprint Capacitors_SMD:C_0603 -> w_smd_cap:c_0603
- C94: renamed from C53; footprint Capacitors_Tantalum_SMD:TantalC_SizeA_EIA-3216_Reflow -> w_smd_cap:c_tant_C
- C95: renamed from C30; footprint Capacitors_SMD:C_0603 -> w_smd_cap:c_0603
- C96: renamed from C33; footprint Capacitors_SMD:C_0603_HandSolderng -> w_smd_cap:c_0603
- C97: renamed from C54; footprint Capacitors_Tantalum_SMD:TantalC_SizeA_EIA-3216_Reflow -> w_smd_cap:c_tant_C
- C98: renamed from C34; footprint Capacitors_SMD:c_elec_4x5.3 -> w_smd_cap:c_elec_4x5.3
- C99: renamed from C35; footprint Capacitors_SMD:C_0805_HandSoldering -> w_smd_cap:c_0805
- D1: renamed from D2; footprint Diodes_SMD:SOD-123 -> w_smd_diode:sod123
- R11: renamed from R23; footprint Resistors_SMD:R_0603_HandSoldering -> w_smd_resistors:r_0603
- R12: renamed from R22; footprint Resistors_SMD:R_0603_HandSoldering -> w_smd_resistors:r_0603
- R13: renamed from R28; footprint Resistors_SMD:R_0603_HandSoldering -> w_smd_resistors:r_0603
- R14: renamed from R25; footprint Resistors_SMD:R_0603 -> w_smd_resistors:r_0603
- R15: renamed from R26; footprint Resistors_SMD:R_0603 -> w_smd_resistors:r_0603
- R16: renamed from R24; footprint Resistors_SMD:R_0603 -> w_smd_resistors:r_0603
- R17: renamed from R27; footprint Resistors_SMD:R_0603 -> w_smd_resistors:r_0603
- R18, R19: footprint Resistors_SMD:R_0603_HandSoldering -> w_smd_resistors:r_0603
- R20: renamed from R10; footprint Resistors_SMD:R_0603_HandSoldering -> w_smd_resistors:r_0603
- R21: renamed from R11; footprint Resistors_SMD:R_0603_HandSoldering -> w_smd_resistors:r_0603
- R22: renamed from R12; footprint Resistors_SMD:R_0603_HandSoldering -> w_smd_resistors:r_0603
- R23: renamed from R13; footprint Resistors_SMD:R_0603_HandSoldering -> w_smd_resistors:r_0603
- R24: renamed from R14; footprint Resistors_SMD:R_0603_HandSoldering -> w_smd_resistors:r_0603
- R25: renamed from R15; footprint Resistors_SMD:R_0603_HandSoldering -> w_smd_resistors:r_0603
- R26: renamed from R20; footprint Resistors_SMD:R_0603_HandSoldering -> w_smd_resistors:r_0603
- R27: renamed from R21; footprint Resistors_SMD:R_0603_HandSoldering -> w_smd_resistors:r_0603
- U6: renamed from U12; footprint Housings_SSOP:TSSOP-24_4.4x7.8mm_Pitch0.65mm -> w_smd_dil:tssop-24
- renumbered P7 to P10, P5 to P11, P4 to P12, P6 to P8, P10 to P9, U6 to U7, U9 to U8, U10 to U9
Other:
- moved on the sheet: C79, C80, C81, C82, C84, C93, C95, C97, D1, R17, R18, R19
