File: pcb/camera.sch (KiCad schematic (older format))
At the start: 36 parts, among them P10 CONN_01X14, P4 CONN_01X04, P5 CONN_01X01, Q1 2SC5095, Q2 MT3S20TU, Q3 2SC5095, Q4 MT3S20TU, U10 ICX825AQA, U4 TXB0104, U9 CXD3400N

Commit message: Safety checkin.
Parts:
- removed C12, C13: 0.1u, Capacitors_SMD:C_0603, symbol C
- removed P10: CONN_01X14, Pin_Headers:Pin_Header_Straight_1x14, symbol CONN_01X14
- removed P4: CONN_01X04, Socket_Strips:Socket_Strip_Straight_1x04, symbol CONN_01X04
- removed P5: CONN_01X01, Socket_Strips:Socket_Strip_Straight_1x01, symbol CONN_01X01
- removed Q1, Q3: 2SC5095, w_smd_trans:sot323, symbol Q_NPN_BEC
- removed Q2, Q4: MT3S20TU, w_smd_trans:sot323, symbol Q_NPN_BEC
- removed R10, R11, R14, R15: 10K, Resistors_SMD:R_0603_HandSoldering, symbol R
- removed R12, R20: 1.17K, Resistors_SMD:R_0603_HandSoldering, symbol R
- removed R13, R21: 1.74K, Resistors_SMD:R_0603_HandSoldering, symbol R
- removed R22: 10.0k, Resistors_SMD:R_0603_HandSoldering, symbol R
- removed U4: TXB0104, Housings_SSOP:TSSOP-14_4.4x5mm_Pitch0.65mm, symbol TXB0104
- removed U9: CXD3400N, w_smd_dil:tssop-20, symbol CXD3400N
- added C12, C53, C54, C56, C57, C59: 0.1u, Capacitors_SMD:C_0603, symbol Device:C_Small
- added C55, C58: 47/20V, Capacitors_SMD:c_elec_4x5.3, symbol Device:CP1_Small
- added R15, R21: 27K, symbol Device:R_Small
- added R20, R22: 180K, symbol Device:R_Small
- added U13: LV5609LP, symbol @Engstad:LV5609LP
- added U14, U5: ADA4800, symbol @Engstad:ADA4800
- added U4: SN74LV4T125, symbol @Engstad:SN74LV4T125
- C26, C27, C29, C30, C33, C35: symbol C_Small -> Device:C_Small
- C28, C34, C36, C37: symbol CP1_Small -> Device:CP1_Small
- C31, C32: value 0.1 -> 0.1uF; symbol C_Small -> Device:C_Small
- D2: symbol D_Small -> Device:D_Small
- R18, R19: symbol R_Small -> Device:R_Small
- U10: symbol ICX825AQA -> AstroCam-rescue:ICX825AQA
Connections:
- net labels added: +12VA, +3.3V, +5VA, CCD_12VA, CCD_3V3, CCD_5V0A, CCD_H1, CCD_H2, CCD_HL, CCD_N7VA, CCD_RG, SHT
- net labels removed: 12V, 3V3, 5V0, B1, B2, E1, E2, ENH, H1, H1S_1, H1S_2, H1T_1, H1T_2, H2, H2S_1, H2S_2, H2T_1, H2T_2, HL, LH1_1, LH1_2, RG
- wire segments 107 -> 169
- no-connect marks 2 -> 0
Other:
- note added: "196K"
- note added: "Converts 3.3V input signals into \nVL (-7V), VM (0V) and VH (12V).\n\nSHT => SHT\n L. => 12V\n H. => -7V\n\nXV2/4 => V2/4\n L => 0V\n H => -7V\n\nXV1/3, SG1/3 => V1/3\n L L => 12V\n L H =>. 0V\n H - => -7V"
- moved on the sheet: U10

Commit message: A little more work.
Parts:
- C12, C26, C27, C29, C30, C31, C32, C33, C35, C53, C54, C56, C57, C59: footprint Capacitors_SMD:C_0603 -> Capacitor_SMD:C_0603_1608Metric
- C28: footprint Capacitors_SMD:c_elec_4x5.3 -> Capacitor_SMD:C_1210_3225Metric; symbol Device:CP1_Small -> Device:C_Small
- C34, C36, C37, C55, C58: footprint Capacitors_SMD:c_elec_4x5.3 -> Capacitor_SMD:CP_Elec_4x5.3
- D2: footprint Diodes_SMD:SOD-123 -> Diode_SMD:D_SOD-123
- R15, R20, R21, R22: footprint (none) -> Resistor_SMD:R_0603_1608Metric
- R18, R19: footprint Resistors_SMD:R_0603_HandSoldering -> Resistor_SMD:R_0603_1608Metric
- U13: footprint (none) -> Engstad:ON_Semiconductor-VCT24-3.5x3.5mm
- U14, U5: footprint (none) -> Engstad:lfcsp-cp-6-4
- U4: footprint (none) -> Engstad:Texas_R-PDSO-G14
Connections:
- net +12VA: now also C33.1, C35.1; no longer C33.2, C35.2
- net CCD_H1: now also U4.5 (2A); no longer U4.2 (1A)
- net CCD_H2: now also U4.2 (1A); no longer U4.5 (2A)
- net GND: now also C33.2, C35.2; no longer C33.1, C35.1
- net OH1: now also U4.6 (2Y); no longer U4.3 (1Y)
- net OH2: now also U4.3 (1Y); no longer U4.6 (2Y)
- net -7V renamed -7V0A
Other:
- moved on the sheet: C12, C29, C30, D2, R18, R19
