File: pcb/u-ctrl.sch (KiCad schematic (older format))
At the start: 62 parts, among them P1 CONN_01X02, P13 CONN_01X06, P14 LEDS, P15 ADJ, P16 CONN_01X02, Q5 VEC2611, Q6 VEC2607, T3 NET-TIE, U11 TPS65530

Commit message: latest
Parts:
- removed P1: CONN_01X02, xess:HDR_1x2, symbol CONN_01X02
- added CON1: BARREL_JACK, w_conn_misc:dc_socket, symbol BARREL_JACK
- added P1: USB_OTG, w_conn_pc:conn_usb_B_mini_smd, symbol USB_OTG
- L10, L9: value 4.7 -> 4.7u
- L11: footprint w_smd_inductors:inductor_smd_4.8x2.8mm -> w_smd_inductors:inductor_smd_1008
Connections:
- net GND: now also CON1.2
- net GNDA: now also P1.5 (GND), P1.6 (shield)
- net VBATT: now also CON1.1, P1.1 (VCC)
- net SW4S: now reaches L11.1, U11.1 (SW4S)
- net SW4I: now reaches L11.2, U11.3 (SW4I)
- net VOUT_AFE renamed VOUT_AFE_3V3
- net VOUT_BACKL renamed VOUT_BACKL_5V
- net VOUT_CORE renamed VOUT_CORE_1V2
- net VOUT_IO renamed VOUT_IO_3V3
- net VOUT_MEM renamed VOUT_MEM_1V8
- net VOUT_MOTOR renamed VOUT_MOTOR_5V
- no-connect marks 0 -> 4
Changed lines of the file:
@@
 $EndComp
 Text Label 5850 2650 0    60   ~ 0
-VOUT_AFE
+VOUT_AFE_3V3
 $Comp
 L GND #PWR040
@@
 $EndComp
 Text Label 5850 4700 0    60   ~ 0
-VOUT_IO
+VOUT_IO_3V3
 $Comp
 L GND #PWR044
@@
 P 4900 5650
 F 0 "L10" H 4930 5690 50  0000 L CNN
-F 1 "4.7" H 4930 5610 50  0000 L CNN
+F 1 "4.7u" H 4930 5610 50  0000 L CNN
 F 2 "w_smd_inductors:inductor_smd_4.8x2.8mm" H 4900 5650 60  0001 C CNN
 F 3 "" H 4900 5650 60  0000 C CNN
@@
 $EndComp
 Text Label 5850 5650 0    60   ~ 0
-VOUT_CORE
+VOUT_CORE_1V2
 $Comp
 L R_Small R39
@@
 $EndComp
 Text Label 3400 7250 0    60   ~ 0
-VOUT_MEM
+VOUT_MEM_1V8
 $Comp
 L R_Small R38
@@
 P 3400 6900
 F 0 "L9" H 3430 6940 50  0000 L CNN
-F 1 "4.7" H 3430 6860 50  0000 L CNN
+F 1 "4.7u" H 3430 6860 50  0000 L CNN
 F 2 "w_smd_inductors:inductor_smd_4.8x2.8mm" H 3400 6900 60  0001 C CNN
 F 3 "" H 3400 6900 60  0000 C CNN
@@
 F 0 "L11" H 5030 2190 50  0000 L CNN
 F 1 "4.7uH" H 5030 2110 50  0000 L CNN
-F 2 "w_smd_inductors:inductor_smd_4.8x2.8mm" H 5000 2150 60  0001 C CNN
+F 2 "w_smd_inductors:inductor_smd_1008" H 5000 2150 60  0001 C CNN
 F 3 "" H 5000 2150 60  0000 C CNN
 F 4 "TOKO DE2812C-1098AS-4R7M" H 5000 2150 60  0001 C CNN "Part"
@@
 $EndComp
 Text Label 1150 5100 2    60   ~ 0
-VOUT_MOTOR
+VOUT_MOTOR_5V
 $Comp
 L C C56
@@
 	9200 3550 9200 3350
 Connection ~ 9200 3350
-Text Label 8050 1000 2    60   ~ 0
+Text Label 8200 1050 0    60   ~ 0
 VBATT
 Text Label 9050 950  0    60   ~ 0
@@
 VBATT
 Text Label 9050 1050 0    60   ~ 0
-VOUT_AFE
+VOUT_AFE_3V3
 Text Label 9050 1150 0    60   ~ 0
-VOUT_IO
+VOUT_IO_3V3
 Text Label 9050 1350 0    60   ~ 0
-VOUT_MEM
+VOUT_MEM_1V8
 Text Label 9050 1450 0    60   ~ 0
-VOUT_MOTOR
+VOUT_MOTOR_5V
 Text Label 10250 950  0    60   ~ 0
 VOUT_CCD+
@@
 VOUT_CCD-
 Text Label 9050 1250 0    60   ~ 0
-VOUT_CORE
-$Comp
-L CONN_01X02 P1
-U 1 1 55EBECB5
-P 8250 1050
-F 0 "P1" H 8250 1200 50  0000 C CNN
-F 1 "CONN_01X02" V 8350 1050 50  0000 C CNN
-F 2 "xess:HDR_1x2" H 8250 1050 60  0001 C CNN
-F 3 "" H 8250 1050 60  0000 C CNN
-	1    8250 1050
-	1    0    0    -1
-$EndComp
-Text Label 8050 1100 2    60   ~ 0
-AGND
+VOUT_CORE_1V2
+Text Label 8200 1250 0    60   ~ 0
+GND
 Wire Wire Line
 	1900 4900 2700 4900
@@
 	2250 4650 2700 4650
 Text Label 1150 4100 2    60   ~ 0
-VOUT_BACKL
+VOUT_BACKL_5V
 $Comp
 L INDUCTOR L13
@@
 Wire Wire Line
 	10250 5800 10500 5800
+$Comp
+L BARREL_JACK CON1
+U 1 1 561CDE36
+P 7900 1150
+F 0 "CON1" H 7900 1400 60  0000 C CNN
+F 1 "BARREL_JACK" H 7900 950 60  0000 C CNN
+F 2 "w_conn_misc:dc_socket" H 7900 1600 60  0000 C CNN
+F 3 "" H 7900 1150 60  0000 C CNN
+	1    7900 1150
+	1    0    0    -1
+$EndComp
+NoConn ~ 8200 1150
+$Comp
+L USB_OTG P1
+U 1 1 5620D209
+P 10400 4500
+F 0 "P1" H 10725 4375 50  0000 C CNN
+F 1 "USB_OTG" H 10400 4700 50  0000 C CNN
+F 2 "w_conn_pc:conn_usb_B_mini_smd" V 10350 4400 60  0000 C CNN
+F 3 "" V 10350 4400 60  0000 C CNN
+	1    10400 4500
+	0    1    1    0
+$EndComp
+NoConn ~ 10100 4400
+NoConn ~ 10100 4500
+NoConn ~ 10100 4600
+Wire Wire Line
+	10100 4300 9450 4300
+Text Label 9450 4300 2    60   ~ 0
+VBATT
+$Comp
+L GNDA #PWR077
+U 1 1 5620F8D1
+P 10500 4900
+F 0 "#PWR077" H 10500 4650 50  0001 C CNN
+F 1 "GNDA" H 10500 4750 50  0000 C CNN
+F 2 "" H 10500 4900 60  0000 C CNN
+F 3 "" H 10500 4900 60  0000 C CNN
+	1    10500 4900
+	1    0    0    -1
+$EndComp
+$Comp
+L GNDA #PWR078
+U 1 1 5620F999
+P 10100 4700
+F 0 "#PWR078" H 10100 4450 50  0001 C CNN
+F 1 "GNDA" H 10100 4550 50  0000 C CNN
+F 2 "" H 10100 4700 60  0000 C CNN
+F 3 "" H 10100 4700 60  0000 C CNN
+	1    10100 4700
+	1    0    0    -1
+$EndComp
+Text Label 5000 1900 0    60   ~ 0
+SW4S
+Text Label 5000 2400 0    60   ~ 0
+SW4I
 $EndSCHEMATC

Commit message: work
Parts:
- removed C55, C72: 10uF, Capacitors_SMD:C_1206, symbol C_Small
- removed C56, C58, C75: 10uF, Capacitors_SMD:C_1206, symbol C
- removed C57: 1.0u, Capacitors_SMD:C_0603, symbol C_Small
- removed C59: 10u, Capacitors_SMD:C_1206, symbol C_Small
- removed C60: 3.3uF, Capacitors_SMD:C_0805, symbol C_Small
- removed C61: 4.7u, Capacitors_SMD:C_0805, symbol C_Small
- removed C62, C65: 10.0u, Capacitors_SMD:C_1206, symbol C_Small
- removed C63, C64: 0.1u, Capacitors_SMD:C_0603, symbol C_Small
- removed C66, C67: 47.0u, Capacitors_SMD:C_1206, symbol C_Small
- removed C68, C69, C70, C71: 22u, Capacitors_SMD:C_1206, symbol C_Small
- removed C73, C74: 22uF, Capacitors_SMD:C_1206, symbol C_Small
- removed C76: 10uF, Capacitors_SMD:C_0805, symbol C_Small
- removed CON1: BARREL_JACK, w_conn_misc:dc_socket, symbol BARREL_JACK
- removed D3, D5: 30V/0.5A, Diodes_SMD:SOD-123, symbol D_Small
- removed D4: 30V/.5A, Diodes_SMD:SOD-123, symbol D_Small
- removed L10, L9: 4.7u, w_smd_inductors:inductor_smd_4.8x2.8mm, symbol L_Small
- removed L11: 4.7uH, w_smd_inductors:inductor_smd_1008, symbol L_Small
- removed L12: 2.7uH, w_smd_inductors:inductor_smd_4.8x2.8mm, symbol L_Small
- removed L13: 12uH, w_smd_inductors:inductor_smd_4.8x2.8mm, symbol INDUCTOR
- removed L5: 4.3uH, w_smd_inductors:inductor_smd_4.8x2.8mm, symbol INDUCTOR
- removed L6, L7: 12uH, w_smd_inductors:inductor_smd_4.8x2.8mm, symbol L_Small
- removed P1: USB_OTG, w_conn_pc:conn_usb_B_mini_smd, symbol USB_OTG
- removed P13: CONN_01X06, xess:HDR_1x6, symbol CONN_01X06
- removed P14: LEDS, xess:HDR_1x2, symbol CONN_01X02
- removed P15: ADJ, xess:HDR_1x1, symbol CONN_01X01
- removed P16: CONN_01X02, xess:HDR_1x2, symbol CONN_01X02
- removed Q5: VEC2611, w_smd_trans:sc70, symbol VEC2611
- removed Q6: VEC2607, w_smd_trans:sc70, symbol VEC2607
- removed R29: 11.0k, Resistors_SMD:R_0603, symbol R_Small
- removed R30, R40, R42: 5.6k, Resistors_SMD:R_0603, symbol R_Small
- removed R31, R32, R39, R41, R43, R44, R45: 1.0k, Resistors_SMD:R_0603, symbol R_Small
- removed R33: 3.0k, Resistors_SMD:R_0603, symbol R
- removed R34, R35, R36: 0.6k, Resistors_SMD:R_0603, symbol R
- removed R37, R48: 1.0k, Resistors_SMD:R_0603, symbol R
- removed R38: 2.0k, Resistors_SMD:R_0603, symbol R_Small
- removed R46: 10, Resistors_SMD:R_0603, symbol R
- removed R47: 5.0k, Resistors_SMD:R_0603, symbol R
- removed T3: NET-TIE, Oddities:NetTie-I_Connected_SMD, symbol NET-TIE
- removed U11: TPS65530, Housings_DFN_QFN:UQFN-48-1EP_6x6mm_Pitch0.4mm, symbol TPS65530
- added C17, C22: 10pF, smd:SM0603, symbol C_Small
- added C19, C23: 22uF, smd:SM0805, symbol C
- added C24: 1.0uF, smd:SM0603, symbol C
- added C25, C26, C30, C31: 0.1uF, smd:SM0603, symbol C
- added CON1: SDMMC_Card, engstad:SCHD3A0100, symbol SDMMC_Card
- added L1, L3: Bead, smd:SM0805, symbol L_Small
- added L2: 0.47uH, smd:SM0603, symbol L_Small
- added P10: JLINK-SWD, engstad:pin-strip-6, symbol CONN_01X06
- added P2: USB_OTG, engstad:usb-otg-short, symbol USB_OTG
- added P4: BATT, engstad:pin-socket-2, symbol CONN_01X02
- added P7: RTC, engstad:pin-socket-1, symbol CONN_01X01
- added P9: CORTEX-JTAG, engstad:conn-jtag-0.05, symbol CONN_02X05
- added R1: 10k, smd:SM0603, symbol R
- added SW1: spdp-2x, engstad:slide-switch-smd-cas-220-d20, symbol spdp-2x
- added SW2: RST, engstad:tactile-switch-te-147873-2, symbol SW_PUSH_NO
- added U2: RClamp0504S, w_smd_trans:sot23-6, symbol RClamp0504S
- added U5: APX823, w_smd_trans:sot23-5, symbol APX823
- added X1: XTAL, engstad:cstce-v-c, symbol crystal-resonator-smd
- added Y1: Crystal, armory:CRYSTAL-32k-B, symbol Crystal
Connections:
- net labels added: ADC-SCK, ADC-SDATA, ADC-SL, BOOT0, JTCK/SWCLK, JTDI, JTDO/SWO, JTMS/SWDIO, OSC_IN, OSC_OUT, OTG_5V, OTG_FS_D+, OTG_FS_D-, OTG_FS_ID, RTC, RTC_OSC_IN, RTC_OSC_OUT, SDMMC_CK, SDMMC_CMD, SDMMC_D0, SDMMC_D1, SDMMC_D2, SDMMC_D3, VBAT, VCC-3V3, VDD, VDDA, VDDSD, ~RST
- net labels removed: AGND, EN_AFE, EN_CCD, EN_LGT, EN_SEQ, GNDA, PGND, REF, SW4I, SW4S, VBATT, VCC1, VCC2, VCC3, VCC4, VCC5, VCC6, VCC7, VCC8, VOUT_AFE_3V3, VOUT_BACKL_5V, VOUT_CCD+, VOUT_CCD-, VOUT_CORE_1V2, VOUT_IO_3V3, VOUT_MEM_1V8, VOUT_MOTOR_5V, V_BADJ, XSLEEP
- wire segments 133 -> 77
- no-connect marks 4 -> 3
Other:
- note removed: "CH1: 0.9-2.5 [V] (Engine Core)\nCH2: 2.5-3.6 [V] (Engine I/O)\nCH3: 0.9-2.5 [V] (External Memory)\nCH4: 2.2-3.6 [V] (AFE)\nCH5: 0-18.0 [V] (CCD+)\nCH6: -10-(-5) [V] (CCD-)\nCH7: 3-20 [V] (Backlight LED)\nCH8: 3.3-5.5 [V] (Motor Ctrl & IC drive)\nREF: 2.8 [V] (Internal supply for logic)\n"
- note removed: "Control signals: LOW < 0.4 V, HIGH > 1.4 V\nSEQ56 *not* higher than REF (2.5V)\nVCC max 5.5V\nVCC min 1.5V (except VCC3 & VCC6 2.5V)"
- note removed: "I_out = (0.2 * V_BADJ + 0.05)/R_sense"
- note removed: "PS: Power input for IC"
- note removed: "T_SS [ms] = C_SS [uF] x 60"
- note removed: "T_SS56 [ms] = C_SS56 [uF] x 6.25 = 6.25 [ms]\n"
- note removed: "VOUT = (1 + R1/R2) × 1.25 [V] = 5.0 [V]"
- note removed: "VOUT = (1 + R2/R1) * 0.6 [V] = 1.2 [V]\nRange: 0.9-2.5 [V]"
- note removed: "VOUT = (1 + R2/R1) * 0.6 [V] = 1.8 [V]\nRange: 0.9-2.5V"
- note removed: "VOUT = (1 + R2/R1) * 0.6 [V] = 3.3 [V]\nRange: 2.2-3.6 [V]"
- note removed: "VOUT = (1 + R2/R1) * 0.6 [V] = 3.3 [V]\nRange: 2.5-3.6 [V]"
- note removed: "VOUT=(1+R2/R1) [V]"
- note removed: "VOUT=\n1.25-(1+R2/R1)*1.25 [V]"
- note removed: "VOUTMAX=(1+R2/R1)*1.25 [V]"
