File: pcb/AstroCam.kicad_pcb (KiCad board)
At the start: 2 copper layers, 40 x 40 mm, 93 parts, among them P1 CONN_01X02, P10 CONN_01X14, P2 CONN_01X18, P3 CONN_01X18, P4 CONN_01X04, P5 CONN_01X01, P8 CONN_01X06, P9 CONN_01X02, Q1 2SC5095, Q2 MT3S20TU, Q3 2SC5095, Q4 MT3S20TU, U1 TPS2420, U10 ICX825AQA, U11 ADDI7013, U2 LT3487, U3 TPS63002, U4 TXB0104, U7 TPS56x200, U8 LMZ10500, U9 CXD3400N

Commit message: Cleanups
Parts:
- removed C12, C13, C26, C27: 0.1u, Capacitors_SMD:C_0603
- removed C28: 1u/35V, Capacitors_SMD:c_elec_4x5.3
- removed C29: 0.1uF, Capacitors_SMD:C_0603
- removed C30: 2200pF, Capacitors_SMD:C_0603
- removed C31, C32: 0.1, Capacitors_SMD:C_0603
- removed C33, C35: 0.01, Capacitors_SMD:C_0603
- removed C34, C36, C37: 3.3/20V, Capacitors_SMD:c_elec_4x5.3
- removed C38, C39, C40, C41, C42, C43, C44, C45, C46: 0.1uF, Capacitors_SMD:C_0603_HandSoldering
- removed C47: 4.7uF, Capacitors_SMD:C_0603_HandSoldering
- removed C48, C49: 0.1u, Capacitors_SMD:C_0603_HandSoldering
- removed D2: D, Diodes_SMD:SOD-123
- removed P1: CONN_01X02, Pin_Headers:Pin_Header_Straight_1x02
- removed P10: CONN_01X14, Pin_Headers:Pin_Header_Straight_1x14
- removed P2, P3: CONN_01X18, Pin_Headers:Pin_Header_Straight_1x18
- removed P4: CONN_01X04, Socket_Strips:Socket_Strip_Straight_1x04
- removed P5: CONN_01X01, Socket_Strips:Socket_Strip_Straight_1x01
- removed Q1, Q3: 2SC5095, w_smd_trans:sot323
- removed Q2, Q4: MT3S20TU, w_smd_trans:sot323
- removed R10, R11, R14, R15: 10K, Resistors_SMD:R_0603_HandSoldering
- removed R12, R20: 1.17K, Resistors_SMD:R_0603_HandSoldering
- removed R13, R21: 1.74K, Resistors_SMD:R_0603_HandSoldering
- removed R18: 100k, Resistors_SMD:R_0603_HandSoldering
- removed R19: 1M0, Resistors_SMD:R_0603_HandSoldering
- removed R22: 10.0k, Resistors_SMD:R_0603_HandSoldering
- removed U10: ICX825AQA, camera:ICX825
- removed U11: ADDI7013, camera:csp-bga-bc-76-3
- removed U4: TXB0104, Housings_SSOP:TSSOP-14_4.4x5mm_Pitch0.65mm
- removed U9: CXD3400N, w_smd_dil:tssop-20

Commit message: Latest, greatest.
Parts:
- added ?: , xess:oshw-logo2, F.Cu at (179.6, 68.6)
- added JP5: JUMPER3, xess:xess-JP2, F.Cu at (161.7, 85.0)
- added P11: CONN_01X01, xess:HDR_1x1, F.Cu at (166.8, 85.0)
- added P12: CONN_01X01, xess:HDR_1x1, F.Cu at (173.9, 67.2)
- added T1: NET-TIE, Oddities:NetTie-I_Connected_SMD, B.Cu at (163.2, 81.5)
- added T2: NET-TIE, Oddities:NetTie-I_Connected_SMD, F.Cu at (152.0, 73.3)
- C9: footprint Capacitors_SMD:C_0805_HandSoldering -> Capacitors_SMD:C_1206_HandSoldering
- D1: footprint Diodes_SMD:Diode-SMB_Handsoldering -> Diodes_SMD:SMB_Standard
- U2: footprint w_smd_qfn:dfn10-3x3 -> Housings_DFN_QFN:DFN-10-1EP_3x3mm_Pitch0.5mm
- U8: footprint camera:llp-8 -> engstad:llp-8
- moved C4 64.3 mm to (166.4, 77.7)
- moved U3 64.3 mm to (163.2, 77.9)
- moved C11 64.3 mm to (163.6, 74.0)
- moved L3 64.3 mm to (162.8, 81.5)
- moved D1 57.1 mm to (161.0, 98.5)
- moved P8 57.1 mm to (158.7, 67.2)
- moved L1 55.2 mm to (182.4, 100.2), turned to 270 degrees
- moved P9 54.7 mm to (153.8, 100.1), turned to 270 degrees
- moved L8 54.5 mm to (181.3, 76.5), turned to 270 degrees
- moved C14 53.4 mm to (178.6, 75.9), turned to 270 degrees
- moved R6 53.3 mm to (151.5, 89.7)
- moved R3 52.9 mm to (151.5, 91.7)
- moved R1 52.9 mm to (151.8, 94.0)
- moved U1 52.6 mm to (157.8, 92.2)
- moved C8 52.6 mm to (163.5, 89.2)
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Connections:
- net /power-supply/V_BAT renamed VIN*
- C11 pad 2: GND -> /power-supply/PGND
- C21 pad 2: GND -> /power-supply/PGND
- P8 pad 4: /power-supply/-7V -> /power-supply/+12V
- P8 pad 5: /power-supply/+12V -> /power-supply/-7V
- U1 pad 10: /power-supply/5V5 -> /power-supply/OUT_5V5
- U1 pad 11: /power-supply/5V5 -> /power-supply/OUT_5V5
- U1 pad 12: /power-supply/5V5 -> /power-supply/OUT_5V5
- U3 pad 11: GND -> /power-supply/PGND
- U3 pad 3: GND -> /power-supply/PGND
- U8 pad 4: GND -> /power-supply/PGND
- U8 pad 9: GND -> Net-(U8-Pad9)
Routing:
- net /power-supply/PGND: track 0.00 -> 50.6 mm, vias 0 -> 7
- net /power-supply/5V0: track 63.0 -> 14.1 mm
- net (no net): track 0.00 -> 40.0 mm
- net VIN*: track 33.7 -> 57.4 mm
- net /power-supply/5V5: track 160.3 -> 137.3 mm, vias 7 -> 4
- net /power-supply/OUT_5V5: track 0.00 -> 17.7 mm
- net /power-supply/-7V: track 29.2 -> 46.2 mm, vias 2 -> 0
- net GND: track 164.6 -> 172.2 mm, vias 25 -> 20
- net /power-supply/1V8: track 27.5 -> 32.0 mm
- net /power-supply/3V3: track 19.8 -> 24.2 mm
- net Net-(R6-Pad1): track 8.25 -> 6.45 mm
- net Net-(U8-Pad9): track 0.00 -> 1.70 mm
- net /power-supply/+12V: track 34.3 -> 35.7 mm, vias 4 -> 2
- net Net-(R3-Pad2): track 4.23 -> 3.27 mm
- net /power-supply/CAP: track 9.31 -> 9.98 mm
- added copper zone on B.Cu, net /power-supply/PGND
- added copper zone on F.Cu, net /power-supply/PGND
- removed copper zone on F.Cu, net /power-supply/+12V
- removed copper zone on F.Cu, net /power-supply/-7V
- removed copper zone on F.Cu, net /power-supply/3V3
- removed copper zone on F.Cu, net /power-supply/5V5
- removed copper zone on F.Cu, net VIN*
Other:
- outline, holes or cut-outs redrawn
- net class Power added: clearance 0.1524, trace_width 0.508, via_dia 0.604774, via_drill 0.299974
- board text added: "-7"
- board text added: "1.8"
- board text added: "12"
- board text added: "3.3"
- board text added: "5.0"
- board text added: "5.5"
- board text added: "Astro Power"
- board text added: "GND"
- board text removed: "-7.0V"
- board text removed: "1.8V"
- board text removed: "12.0V"
- board text removed: "3.3V"
- board text removed: "5.0V"
- board text removed: "5.5V"

Commit message: More fiddling
Parts:
- added C12, C13, C48, C49: 0.1u, Capacitors_SMD:C_0603_HandSoldering, F.Cu at (165.0, 115.1)
- added C17, C38, C39, C40, C41, C42, C43, C44, C45, C46: 0.1uF, Capacitors_SMD:C_0603_HandSoldering, F.Cu at (165.0, 115.1)
- added C18: 0.1uF/25V, Capacitors_SMD:C_0603_HandSoldering, F.Cu at (165.0, 115.1)
- added C19: 0.1uF/10V, Capacitors_SMD:C_0603_HandSoldering, F.Cu at (165.0, 115.1)
- added C22: 1.0uF/25V, Capacitors_SMD:C_0603_HandSoldering, F.Cu at (165.0, 115.1)
- added C23: 4.7uF/10V, Capacitors_SMD:c_elec_4x5.3, F.Cu at (165.0, 115.1)
- added C24, C26, C27, C29, C50, C51, C52: 0.1uF, Capacitors_SMD:C_0603, F.Cu at (165.0, 115.1)
- added C28: 1u/35V, Capacitors_SMD:c_elec_4x5.3, F.Cu at (165.0, 115.1)
- added C30: 2200pF, Capacitors_SMD:C_0603, F.Cu at (165.0, 115.1)
- added C31, C32: 0.1, Capacitors_SMD:C_0603, F.Cu at (165.0, 115.1)
- added C34, C36, C37: 3.3/20V, Capacitors_SMD:c_elec_4x5.3, F.Cu at (165.0, 115.1)
- added C35: 0.01, Capacitors_SMD:C_0805_HandSoldering, F.Cu at (165.0, 115.1)
- added C47: 4.7uF, Capacitors_SMD:C_0603_HandSoldering, F.Cu at (165.0, 115.1)
- added C53, C54: 47uF, Capacitors_Tantalum_SMD:TantalC_SizeA_EIA-3216_Reflow, F.Cu at (165.0, 115.1)
- added C55, C56, C58, C72, C75: 10uF, Capacitors_SMD:C_1206, F.Cu at (165.0, 115.1)
- added C57: 1.0u, Capacitors_SMD:C_0603, F.Cu at (165.0, 115.1)
- added C59: 10u, Capacitors_SMD:C_1206, F.Cu at (165.0, 115.1)
- added C60: 3.3uF, Capacitors_SMD:C_0805, F.Cu at (165.0, 115.1)
- added C61: 4.7u, Capacitors_SMD:C_0805, F.Cu at (165.0, 115.1)
- added C62, C65: 10.0u, Capacitors_SMD:C_1206, F.Cu at (165.0, 115.1)
- added C63, C64: 0.1u, Capacitors_SMD:C_0603, F.Cu at (165.0, 115.1)
- added C66, C67: 47.0u, Capacitors_SMD:C_1206, F.Cu at (165.0, 115.1)
- added C68, C69, C70, C71: 22u, Capacitors_SMD:C_1206, F.Cu at (165.0, 115.1)
- added C73, C74: 22uF, Capacitors_SMD:C_1206, F.Cu at (165.0, 115.1)
- added C76: 10uF, Capacitors_SMD:C_0805, F.Cu at (165.0, 115.1)
- added D2: D, Diodes_SMD:SOD-123, F.Cu at (165.0, 115.1)
- added D3, D5: 30V/0.5A, Diodes_SMD:SOD-123, F.Cu at (165.0, 115.1)
- added D4: 30V/.5A, Diodes_SMD:SOD-123, F.Cu at (165.0, 115.1)
- added JP1, JP2, JP3, JP4: JUMPER3, xess:xess-JP2, F.Cu at (165.0, 115.1)
- added L10, L9: 4.7, w_smd_inductors:inductor_smd_4.8x2.8mm, F.Cu at (165.0, 115.1)
- added L11: 4.7uH, w_smd_inductors:inductor_smd_4.8x2.8mm, F.Cu at (165.0, 115.1)
- added L12: 2.7uH, w_smd_inductors:inductor_smd_4.8x2.8mm, F.Cu at (165.0, 115.1)
- added L13, L6, L7: 12uH, w_smd_inductors:inductor_smd_4.8x2.8mm, F.Cu at (165.0, 115.1)
- added L5: 4.3uH, w_smd_inductors:inductor_smd_4.8x2.8mm, F.Cu at (165.0, 115.1)
- added P1, P16: CONN_01X02, xess:HDR_1x2, F.Cu at (165.0, 115.1)
- added P10, P5: OUTP, xess:HDR_1x2, F.Cu at (165.0, 115.1)
- added P13: CONN_01X06, xess:HDR_1x6, F.Cu at (165.0, 115.1)
- added P14: LEDS, xess:HDR_1x2, F.Cu at (165.0, 115.1)
- added P15: ADJ, xess:HDR_1x1, F.Cu at (165.0, 115.1)
- added P2, P3: CONN_01X18, Pin_Headers:Pin_Header_Straight_1x18, F.Cu at (165.0, 115.1)
- added P4: HORI, xess:HDR_1x6, F.Cu at (165.0, 115.1)
- added P6: POWER, xess:HDR_1x6, F.Cu at (165.0, 115.1)
- added P7: VERT, xess:HDR_1x8, F.Cu at (165.0, 115.1)
- added Q1, Q3: 2SC5095, w_smd_trans:sot323, F.Cu at (165.0, 115.1)
- added Q2, Q4: MT3S20TU, w_smd_trans:sot323, F.Cu at (165.0, 115.1)
- added Q5: VEC2611, w_smd_trans:sc70, F.Cu at (165.0, 115.1)
- added Q6: VEC2607, w_smd_trans:sc70, F.Cu at (165.0, 115.1)
- added R10, R11, R14, R15: 10K, Resistors_SMD:R_0603_HandSoldering, F.Cu at (165.0, 115.1)
- added R12, R20: 1.17K, Resistors_SMD:R_0603_HandSoldering, F.Cu at (165.0, 115.1)
- added R13, R21: 1.74K, Resistors_SMD:R_0603_HandSoldering, F.Cu at (165.0, 115.1)
- added R18: 100k, Resistors_SMD:R_0603_HandSoldering, F.Cu at (165.0, 115.1)
- added R19: 1M0, Resistors_SMD:R_0603_HandSoldering, F.Cu at (165.0, 115.1)
- added R22, R23, R28: 10.0k, Resistors_SMD:R_0603_HandSoldering, F.Cu at (165.0, 115.1)
- added R24, R27: 249k, Resistors_SMD:R_0603, F.Cu at (165.0, 115.1)
- added R25, R26: 10K, Resistors_SMD:R_0603, F.Cu at (165.0, 115.1)
- added R29: 11.0k, Resistors_SMD:R_0603, F.Cu at (165.0, 115.1)
- added R30, R40, R42: 5.6k, Resistors_SMD:R_0603, F.Cu at (165.0, 115.1)
- added R31, R32, R37, R39, R41, R43, R44, R45, R48: 1.0k, Resistors_SMD:R_0603, F.Cu at (165.0, 115.1)
- added R33: 3.0k, Resistors_SMD:R_0603, F.Cu at (165.0, 115.1)
- added R34, R35, R36: 0.6k, Resistors_SMD:R_0603, F.Cu at (165.0, 115.1)
- added R38: 2.0k, Resistors_SMD:R_0603, F.Cu at (165.0, 115.1)
- added R46: 10, Resistors_SMD:R_0603, F.Cu at (165.0, 115.1)
- added R47: 5.0k, Resistors_SMD:R_0603, F.Cu at (165.0, 115.1)
- added T3: NET-TIE, Oddities:NetTie-I_Connected_SMD, F.Cu at (165.0, 115.1)
- added U11: TPS65530, Housings_DFN_QFN:UQFN-48-1EP_6x6mm_Pitch0.4mm, F.Cu at (165.0, 115.1)
- added U12: SN74LVC8T245, Housings_SSOP:TSSOP-24_4.4x7.8mm_Pitch0.65mm, F.Cu at (165.0, 115.1)
- added U4: ADDI7013, engstad:csp-bga-bc-76-3, F.Cu at (165.0, 115.1)
- added U5: ADDI9023, engstad:csp-bga-bc-40-1, F.Cu at (165.0, 115.1)
- added U6, U9: ADA4800, engstad:lfcsp-cp-6-4, F.Cu at (165.0, 115.1)
Connections:
- U8 pad 9: Net-(U8-Pad9) -> /power-supply/PGND
Routing:
- net /power-supply/PGND: track 50.6 -> 58.7 mm, vias 7 -> 13
- net Net-(U8-Pad9): track 1.70 -> 0.00 mm

Commit message: More.
Parts:
- removed C12, C13, C48, C49: 0.1u, Capacitors_SMD:C_0603_HandSoldering
- removed C17, C38, C39, C40, C41, C42, C43, C44, C45, C46: 0.1uF, Capacitors_SMD:C_0603_HandSoldering
- removed C18: 0.1uF/25V, Capacitors_SMD:C_0603_HandSoldering
- removed C19: 0.1uF/10V, Capacitors_SMD:C_0603_HandSoldering
- removed C22: 1.0uF/25V, Capacitors_SMD:C_0603_HandSoldering
- removed C23: 4.7uF/10V, Capacitors_SMD:c_elec_4x5.3
- removed C24, C26, C27, C29, C50, C51, C52: 0.1uF, Capacitors_SMD:C_0603
- removed C28: 1u/35V, Capacitors_SMD:c_elec_4x5.3
- removed C30: 2200pF, Capacitors_SMD:C_0603
- removed C31, C32: 0.1, Capacitors_SMD:C_0603
- removed C34, C36, C37: 3.3/20V, Capacitors_SMD:c_elec_4x5.3
- removed C35: 0.01, Capacitors_SMD:C_0805_HandSoldering
- removed C47: 4.7uF, Capacitors_SMD:C_0603_HandSoldering
- removed C53, C54: 47uF, Capacitors_Tantalum_SMD:TantalC_SizeA_EIA-3216_Reflow
- removed C55, C56, C58, C72, C75: 10uF, Capacitors_SMD:C_1206
- removed C57: 1.0u, Capacitors_SMD:C_0603
- removed C59: 10u, Capacitors_SMD:C_1206
- removed C60: 3.3uF, Capacitors_SMD:C_0805
- removed C61: 4.7u, Capacitors_SMD:C_0805
- removed C62, C65: 10.0u, Capacitors_SMD:C_1206
- removed C63, C64: 0.1u, Capacitors_SMD:C_0603
- removed C66, C67: 47.0u, Capacitors_SMD:C_1206
- removed C68, C69, C70, C71: 22u, Capacitors_SMD:C_1206
- removed C73, C74: 22uF, Capacitors_SMD:C_1206
- removed C76: 10uF, Capacitors_SMD:C_0805
- removed D2: D, Diodes_SMD:SOD-123
- removed D3, D5: 30V/0.5A, Diodes_SMD:SOD-123
- removed D4: 30V/.5A, Diodes_SMD:SOD-123
- removed JP1, JP2, JP3, JP4: JUMPER3, xess:xess-JP2
- removed L10, L9: 4.7, w_smd_inductors:inductor_smd_4.8x2.8mm
- removed L11: 4.7uH, w_smd_inductors:inductor_smd_4.8x2.8mm
- removed L12: 2.7uH, w_smd_inductors:inductor_smd_4.8x2.8mm
- removed L13, L6, L7: 12uH, w_smd_inductors:inductor_smd_4.8x2.8mm
- removed L5: 4.3uH, w_smd_inductors:inductor_smd_4.8x2.8mm
- removed P1, P16: CONN_01X02, xess:HDR_1x2
- removed P10, P5: OUTP, xess:HDR_1x2
- removed P13: CONN_01X06, xess:HDR_1x6
- removed P14: LEDS, xess:HDR_1x2
- removed P15: ADJ, xess:HDR_1x1
- removed P2, P3: CONN_01X18, Pin_Headers:Pin_Header_Straight_1x18
- removed P4: HORI, xess:HDR_1x6
- removed P6: POWER, xess:HDR_1x6
- removed P7: VERT, xess:HDR_1x8
- removed Q1, Q3: 2SC5095, w_smd_trans:sot323
- removed Q2, Q4: MT3S20TU, w_smd_trans:sot323
- removed Q5: VEC2611, w_smd_trans:sc70
- removed Q6: VEC2607, w_smd_trans:sc70
- removed R10, R11, R14, R15: 10K, Resistors_SMD:R_0603_HandSoldering
- removed R12, R20: 1.17K, Resistors_SMD:R_0603_HandSoldering
- removed R13, R21: 1.74K, Resistors_SMD:R_0603_HandSoldering
- removed R18: 100k, Resistors_SMD:R_0603_HandSoldering
- removed R19: 1M0, Resistors_SMD:R_0603_HandSoldering
- removed R22, R23, R28: 10.0k, Resistors_SMD:R_0603_HandSoldering
- removed R24, R27: 249k, Resistors_SMD:R_0603
- removed R25, R26: 10K, Resistors_SMD:R_0603
- removed R29: 11.0k, Resistors_SMD:R_0603
- removed R30, R40, R42: 5.6k, Resistors_SMD:R_0603
- removed R31, R32, R37, R39, R41, R43, R44, R45, R48: 1.0k, Resistors_SMD:R_0603
- removed R33: 3.0k, Resistors_SMD:R_0603
- removed R34, R35, R36: 0.6k, Resistors_SMD:R_0603
- removed R38: 2.0k, Resistors_SMD:R_0603
- removed R46: 10, Resistors_SMD:R_0603
- removed R47: 5.0k, Resistors_SMD:R_0603
- removed T3: NET-TIE, Oddities:NetTie-I_Connected_SMD
- removed U11: TPS65530, Housings_DFN_QFN:UQFN-48-1EP_6x6mm_Pitch0.4mm
- removed U12: SN74LVC8T245, Housings_SSOP:TSSOP-24_4.4x7.8mm_Pitch0.65mm
- removed U4: ADDI7013, engstad:csp-bga-bc-76-3
- removed U5: ADDI9023, engstad:csp-bga-bc-40-1
- removed U6, U9: ADA4800, engstad:lfcsp-cp-6-4

Commit message: work
Parts:
- removed ?: , xess:oshw-logo2
- removed C1, C2, C6: 1.0uF, Capacitors_SMD:C_0805_HandSoldering
- removed C10: 0.1uF, Capacitors_SMD:C_0805_HandSoldering
- removed C11: 10uF, Capacitors_SMD:C_0805_HandSoldering
- removed C14, C15, C21: 10.0uF, Capacitors_SMD:C_0805_HandSoldering
- removed C16: 470pF, Capacitors_SMD:C_0402
- removed C20: 0.1uF, Capacitors_SMD:C_0603_HandSoldering
- removed C25: 47uF, Capacitors_SMD:C_1206_HandSoldering
- removed C3, C5: 47pF, Capacitors_SMD:C_0805_HandSoldering
- removed C4: 2.2uF, Capacitors_SMD:C_0603_HandSoldering
- removed C7: 100nF, Capacitors_SMD:C_0805_HandSoldering
- removed C8: 1.0uF/11mOhm, Capacitors_SMD:C_0805_HandSoldering
- removed C9: 4.7uF, Capacitors_SMD:C_1206_HandSoldering
- removed D1: 9V/5W, Diodes_SMD:SMB_Standard
- removed JP5: JUMPER3, xess:xess-JP2
- removed L1, L2: 15uH, w_smd_inductors:inductor_smd_0805
- removed L3: 2.0uH, w_smd_inductors:inductor_smd_0805
- removed L4: 10uH, w_smd_inductors:inductor_smd_0805
- removed L8: 2.2uH, w_smd_inductors:inductor_smd_0805
- removed P11, P12: CONN_01X01, xess:HDR_1x1
- removed P8: CONN_01X06, Pin_Headers:Pin_Header_Straight_1x06
- removed P9: CONN_01X02, Pin_Headers:Pin_Header_Straight_1x02
- removed R1: 10.0k, Resistors_SMD:R_0805_HandSoldering
- removed R16: 13.7k, Resistors_SMD:R_0402
- removed R17: 10.0k, Resistors_SMD:R_0402
- removed R2, R7: 324k, Resistors_SMD:R_0603_HandSoldering
- removed R3: 10.0k, Resistors_SMD:R_0603_HandSoldering
- removed R4: 51.1k, Resistors_SMD:R_0603_HandSoldering
- removed R5: 68.1k, Resistors_SMD:R_0603_HandSoldering
- removed R6: 53.6k, Resistors_SMD:R_0603_HandSoldering
- removed R8: 80.6k, Resistors_SMD:R_0402
- removed R9: 105k, Resistors_SMD:R_0402
- removed T1, T2: NET-TIE, Oddities:NetTie-I_Connected_SMD
- removed U1: TPS2420, Housings_DFN_QFN:QFN-16-1EP_4x4mm_Pitch0.65mm
- removed U2: LT3487, Housings_DFN_QFN:DFN-10-1EP_3x3mm_Pitch0.5mm
- removed U3: TPS63002, Housings_DFN_QFN:DFN-10-1EP_3x3mm_Pitch0.5mm
- removed U7: TPS56x200, Housings_SOT-23_SOT-143_TSOT-6:SOT-23-6
- removed U8: LMZ10500, engstad:llp-8
Routing:
- net GND: track 172.2 -> 0.00 mm, vias 20 -> 0
- net /power-supply/5V5: track 137.3 -> 0.00 mm, vias 4 -> 0
- net /power-supply/PGND: track 58.7 -> 0.00 mm, vias 13 -> 0
- net VIN*: track 57.4 -> 0.00 mm
- net /power-supply/-7V: track 46.2 -> 0.00 mm
- net (no net): track 40.0 -> 0.00 mm
- net /power-supply/+12V: track 35.7 -> 0.00 mm, vias 2 -> 0
- net /power-supply/1V8: track 32.0 -> 0.00 mm
- net /power-supply/3V3: track 24.3 -> 0.00 mm, vias 2 -> 0
- net /power-supply/OUT_5V5: track 17.7 -> 0.00 mm
- net /power-supply/5V0: track 14.1 -> 0.00 mm
- net /power-supply/DN: track 10.2 -> 0.00 mm
- net /power-supply/CAP: track 9.98 -> 0.00 mm
- net Net-(C20-Pad2): track 9.05 -> 0.00 mm, vias 2 -> 0
- net Net-(C6-Pad1): track 9.00 -> 0.00 mm
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- removed copper zone on B.Cu, net /power-supply/PGND
- removed copper zone on F.Cu, net /power-supply/PGND
- removed copper zone on B.Cu, net GND
- removed copper zone on F.Cu, net GND
Other:
- board size 40 x 40 mm -> 50 x 50 mm
- net class Default: clearance 0.1524 -> 0.15
- rule trace_clearance: 0.1524 -> 0.15
- rule trace_min: 0.1524 -> 0.1
- rule via_min_drill: 0.299974 -> 0.254
- rule via_min_size: 0.604774 -> 0.4572
- board text removed: "+"
- board text removed: "-"
- board text removed: "-7"
- board text removed: "1.8"
- board text removed: "12"
- board text removed: "3.3"
- board text removed: "5.0"
- board text removed: "5.5"
- board text removed: "Astro Power"
- board text removed: "GND"
