File: pcb/AstroCam.kicad_pcb (KiCad board)
At the start: 2 copper layers, 40 x 40 mm, 93 parts, among them P1 CONN_01X02, P10 CONN_01X14, P2 CONN_01X18, P3 CONN_01X18, P4 CONN_01X04, P5 CONN_01X01, P8 CONN_01X06, P9 CONN_01X02, Q1 2SC5095, Q2 MT3S20TU, Q3 2SC5095, Q4 MT3S20TU, U1 TPS2420, U10 ICX825AQA, U11 ADDI7013, U2 LT3487, U3 TPS63002, U4 TXB0104, U7 TPS56x200, U8 LMZ10500, U9 CXD3400N

Commit message: Safety checkin.
Parts:
- moved C27 99.5 mm to (146.8, 151.1)
- moved C26 97.4 mm to (146.8, 147.5)
- moved C29 96.5 mm to (150.5, 151.1)
- moved C12 95.6 mm to (146.7, 144.0)
- moved C30 94.3 mm to (150.5, 147.4)
- moved C32 93.6 mm to (154.2, 151.0)
- moved C31 92.3 mm to (150.6, 144.0)
- moved C33 90.7 mm to (157.9, 151.0)
- moved R10 90.1 mm to (144.2, 127.3)
- moved R12 88.9 mm to (143.7, 122.6)
- moved C35 88.1 mm to (158.2, 147.3)
- moved C39 87.4 mm to (162.2, 150.9)
- moved C41 85.8 mm to (158.3, 143.6)
- moved R13 85.1 mm to (150.0, 128.1)
- moved D2 85.1 mm to (152.1, 132.3)
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
Commit message: A little more work.
Parts:
- removed C1: 1.0uF, Capacitors_SMD:C_0805_HandSoldering
- removed D1: 9V/5W, Diodes_SMD:Diode-SMB_Handsoldering
- removed L3: 2.0uH, w_smd_inductors:inductor_smd_0805
- removed P1, P9: CONN_01X02, Pin_Headers:Pin_Header_Straight_1x02
- removed P10: CONN_01X14, Pin_Headers:Pin_Header_Straight_1x14
- removed P2, P3: CONN_01X18, Pin_Headers:Pin_Header_Straight_1x18
- removed P4: CONN_01X04, Socket_Strips:Socket_Strip_Straight_1x04
- removed P5: CONN_01X01, Socket_Strips:Socket_Strip_Straight_1x01
- removed P8: CONN_01X06, Pin_Headers:Pin_Header_Straight_1x06
- removed Q1, Q3: 2SC5095, w_smd_trans:sot323
- removed Q2, Q4: MT3S20TU, w_smd_trans:sot323
- added C17: 10.0uF, Capacitor_SMD:C_1206_3216Metric, F.Cu at (123.9, 72.3)
- added C18: 10.0uF, Capacitor_SMD:C_1206_3216Metric, F.Cu at (126.4, 72.3)
- added C19: 10.0uF, Capacitor_SMD:C_1206_3216Metric, F.Cu at (104.3, 101.1)
- added C22: 10uF, Capacitor_SMD:C_1206_3216Metric, F.Cu at (83.7, 83.5)
- added C23: 10uF, Capacitor_SMD:C_1206_3216Metric, F.Cu at (108.1, 85.8)
- added C24: 0.47uF, Capacitor_SMD:C_0603_1608Metric, F.Cu at (103.4, 97.5)
- added C50: 10nF, Capacitor_SMD:C_0603_1608Metric, F.Cu at (85.6, 92.5)
- added C51: 4.7uF, Capacitor_SMD:C_0805_2012Metric, F.Cu at (107.0, 97.5)
- added C52: 10uF, Capacitor_SMD:C_1206_3216Metric, F.Cu at (86.3, 96.7)
- added C53: 0.1u, Capacitor_SMD:C_0603_1608Metric, F.Cu at (163.8, 105.3)
- added C54: 0.1u, Capacitor_SMD:C_0603_1608Metric, F.Cu at (174.2, 89.7)
- added C55: 47/20V, Capacitor_SMD:CP_Elec_4x5.3, F.Cu at (145.0, 80.0)
- added C56: 0.1u, Capacitor_SMD:C_0603_1608Metric, F.Cu at (174.2, 95.8)
- added C57: 0.1u, Capacitor_SMD:C_0603_1608Metric, F.Cu at (145.0, 94.5)
- added C58: 47/20V, Capacitor_SMD:CP_Elec_4x5.3, F.Cu at (179.0, 97.8)
- added C59: 0.1u, Capacitor_SMD:C_0603_1608Metric, F.Cu at (145.0, 88.5)
- added C60: 2.2uF, Capacitor_SMD:C_0603_1608Metric, F.Cu at (107.3, 79.7)
- added C61: 2.2uF, Capacitor_SMD:C_0603_1608Metric, F.Cu at (115.4, 80.4)
- added C62: 2.2uF, Capacitor_SMD:C_0603_1608Metric, F.Cu at (115.4, 77.3)
- added NT1: Net-Tie_3, NetTie:NetTie-3_SMD_Pad0.5mm, F.Cu at (86.8, 77.8)
- added NT2: Net-Tie_2, NetTie:NetTie-2_THT_Pad0.3mm, F.Cu at (104.2, 74.2)
- added U12: LT3042, Package_DFN_QFN:DFN-10-1EP_3x3mm_P0.5mm_EP1.65x2.38mm_ThermalVias, F.Cu at (98.8, 99.7)
- added U13: LV5609LP, Engstad:ON_Semiconductor-VCT24-3.5x3.5mm, F.Cu at (164.2, 100.8)
- added U14: ADA4800, Engstad:lfcsp-cp-6-4, F.Cu at (146.8, 91.7)
- added U5: ADA4800, Engstad:lfcsp-cp-6-4, F.Cu at (172.2, 92.7)
- added U6: AD9978, Engstad:qfn-40, F.Cu at (182.1, 80.0)
- C10, C2, C5, C6: footprint Capacitors_SMD:C_0805_HandSoldering -> Capacitor_SMD:C_0603_1608Metric
- C11: value 10uF -> 0.1uF; footprint Capacitors_SMD:C_0805_HandSoldering -> Capacitor_SMD:C_0603_1608Metric
- C12, C26, C27, C29, C30, C33, C35: footprint Capacitors_SMD:C_0603 -> Capacitor_SMD:C_0603_1608Metric
- C13: value 0.1u -> 10.0uF; footprint Capacitors_SMD:C_0603 -> Capacitor_SMD:C_1206_3216Metric
- C14: value 10.0uF -> 10uF; footprint Capacitors_SMD:C_0805_HandSoldering -> Capacitor_SMD:C_0805_2012Metric
- C15, C21, C9: footprint Capacitors_SMD:C_0805_HandSoldering -> Capacitor_SMD:C_0805_2012Metric
- C16: footprint Capacitors_SMD:C_0402 -> Capacitor_SMD:C_0603_1608Metric
- C20, C38, C39, C40, C41, C42, C43, C45, C48, C49: footprint Capacitors_SMD:C_0603_HandSoldering -> Capacitor_SMD:C_0603_1608Metric
- C25: value 47uF -> 10uF; footprint Capacitors_SMD:C_1206_HandSoldering -> Capacitor_SMD:C_1206_3216Metric
- C28: footprint Capacitors_SMD:c_elec_4x5.3 -> Capacitor_SMD:C_1210_3225Metric
- C3: value 47pF -> 22uF; footprint Capacitors_SMD:C_0805_HandSoldering -> Capacitor_SMD:C_1206_3216Metric
- C31, C32: value 0.1 -> 0.1uF; footprint Capacitors_SMD:C_0603 -> Capacitor_SMD:C_0603_1608Metric
- C34, C36, C37: footprint Capacitors_SMD:c_elec_4x5.3 -> Capacitor_SMD:CP_Elec_4x5.3
- C4: value 2.2uF -> 10uF; footprint Capacitors_SMD:C_0603_HandSoldering -> Capacitor_SMD:C_0805_2012Metric
- C44, C46: value 0.1uF -> 4.7uF; footprint Capacitors_SMD:C_0603_HandSoldering -> Capacitor_SMD:C_0805_2012Metric
- C47: value 4.7uF -> 0.1uF; footprint Capacitors_SMD:C_0603_HandSoldering -> Capacitor_SMD:C_0603_1608Metric
- C7: value 100nF -> 0.1uF; footprint Capacitors_SMD:C_0805_HandSoldering -> Capacitor_SMD:C_0603_1608Metric
- C8: value 1.0uF/11mOhm -> 1.0uF; footprint Capacitors_SMD:C_0805_HandSoldering -> Capacitor_SMD:C_0603_1608Metric
- D2: footprint Diodes_SMD:SOD-123 -> Diode_SMD:D_SOD-123
- L1, L2, L4: footprint w_smd_inductors:inductor_smd_0805 -> Engstad:L_Wurth-4018
- L8: footprint w_smd_inductors:inductor_smd_0805 -> Inductor_SMD:L_0805_2012Metric
- R1: footprint Resistors_SMD:R_0805_HandSoldering -> Resistor_SMD:R_0603_1608Metric
- R10: value 10K -> 200K; footprint Resistors_SMD:R_0603_HandSoldering -> Resistor_SMD:R_0603_1608Metric
- R11: value 10K -> 49K9; footprint Resistors_SMD:R_0603_HandSoldering -> Resistor_SMD:R_0603_1608Metric
- R12: value 1.17K -> 499R; footprint Resistors_SMD:R_0603_HandSoldering -> Resistor_SMD:R_0603_1608Metric
- R13: value 1.74K -> 487K; footprint Resistors_SMD:R_0603_HandSoldering -> Resistor_SMD:R_0603_1608Metric
- R14: value 10K -> 100K; footprint Resistors_SMD:R_0603_HandSoldering -> Resistor_SMD:R_0603_1608Metric
- R15: value 10K -> 27K; footprint Resistors_SMD:R_0603_HandSoldering -> Resistor_SMD:R_0603_1608Metric
- R16, R17, R8, R9: footprint Resistors_SMD:R_0402 -> Resistor_SMD:R_0603_1608Metric
- R18, R19, R3, R4, R5, R6: footprint Resistors_SMD:R_0603_HandSoldering -> Resistor_SMD:R_0603_1608Metric
- R2: value 324k -> 324K; footprint Resistors_SMD:R_0603_HandSoldering -> Resistor_SMD:R_0603_1608Metric
- R20: value 1.17K -> 180K; footprint Resistors_SMD:R_0603_HandSoldering -> Resistor_SMD:R_0603_1608Metric
- R21: value 1.74K -> 27K; footprint Resistors_SMD:R_0603_HandSoldering -> Resistor_SMD:R_0603_1608Metric
- R22: value 10.0k -> 180K; footprint Resistors_SMD:R_0603_HandSoldering -> Resistor_SMD:R_0603_1608Metric
- R7: value 324k -> 487K; footprint Resistors_SMD:R_0603_HandSoldering -> Resistor_SMD:R_0603_1608Metric
- U1: footprint Housings_DFN_QFN:QFN-16-1EP_4x4mm_Pitch0.65mm -> Package_DFN_QFN:QFN-16-1EP_4x4mm_P0.65mm_EP2.7x2.7mm_ThermalVias
- U11: value ADDI7013 -> MIC5355-SGYMME; footprint camera:csp-bga-bc-76-3 -> Package_SO:MSOP-8-1EP_3x3mm_P0.65mm_EP2.5x3mm_Mask1.73x2.36mm_ThermalVias
- U2: footprint w_smd_qfn:dfn10-3x3 -> Package_DFN_QFN:DFN-10-1EP_3x3mm_P0.5mm_EP1.7x2.5mm
- U3: value TPS63002 -> TPS7A3401; footprint Housings_DFN_QFN:DFN-10-1EP_3x3mm_Pitch0.5mm -> Engstad:VSSOP-8_3.0x3.0mm_P0.65mm
- U4: value TXB0104 -> SN74LV4T125; footprint Housings_SSOP:TSSOP-14_4.4x5mm_Pitch0.65mm -> Engstad:Texas_R-PDSO-G14
- U7: footprint Housings_SOT-23_SOT-143_TSOT-6:SOT-23-6 -> Package_TO_SOT_SMD:SOT-23-6
- U8: footprint camera:llp-8 -> Engstad:Texas_Instruments-LLP-8
- U9: value CXD3400N -> RT9069-C0GB; footprint w_smd_dil:tssop-20 -> Package_TO_SOT_SMD:SOT-23-5
- moved R11 168.2 mm to (93.7, 98.0), turned to 180 degrees
- moved C34 118.1 mm to (148.6, 71.3)
- moved U11 116.8 mm to (111.3, 79.9)
- moved C13 112.1 mm to (121.5, 72.3), turned to 270 degrees
- moved U9 110.0 mm to (111.2, 85.9), turned to 270 degrees
- moved C28 103.9 mm to (148.9, 100.2), turned to 270 degrees
- moved C37 103.8 mm to (159.7, 102.1), turned to 90 degrees
- moved C36 92.1 mm to (171.4, 71.3), turned to 180 degrees
- moved U10 91.9 mm to (160.0, 85.0)
- moved C12 80.0 mm to (160.4, 65.2), turned to 180 degrees
- moved C43 78.4 mm to (185.6, 74.5), turned to 180 degrees
- moved C39 78.1 mm to (178.6, 74.5), turned to 180 degrees
- moved C42 76.1 mm to (176.4, 80.8), turned to 180 degrees
- moved C33 76.0 mm to (152.0, 75.2), turned to 90 degrees
- moved C32 75.9 mm to (153.9, 75.2), turned to 90 degrees
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Connections:
- net /power-supply/V_BAT renamed VIN*
- net Net-(C6-Pad1) renamed /power-supply/SW-
- net Net-(L4-Pad2) renamed /power-supply/SW+
- C10 pad 2: /power-supply/+12V -> /power-supply/13V5
- C11 pad 1: /power-supply/5V0 -> /power-supply/5V5
- C11 pad 2: GND -> GNDPWR
- C12 pad 1: /camera/3V3 -> +5VA
- C13 pad 1: /camera/5V0 -> +1V8
- C13 pad 2: GND -> GNDPWR
- C14 pad 2: GND -> GNDPWR
- C15 pad 2: GND -> /power-supply/LMZ_PGND
- C2 pad 2: GND -> GNDPWR
- C21 pad 1: /power-supply/3V3 -> +3V3
- C21 pad 2: GND -> /power-supply/LMZ_PGND
- C25 pad 1: /power-supply/1V8 -> +12VA
- C26 pad 1: /camera/-7V -> GND
- C26 pad 2: GND -> -7V0A
- C27 pad 1: /camera/12V -> +12VA
- C28 pad 2: Net-(C28-Pad2) -> /camera/SHT
- C3 pad 1: /power-supply/-7V -> /power-supply/-8V
- C3 pad 2: GND -> GNDPWR
- C33 pad 1: GND -> +12VA
- C33 pad 2: /camera/12V -> GND
- C34 pad 1: /camera/12V -> +12VA
- C35 pad 1: GND -> +12VA
- C35 pad 2: /camera/12V -> GND
- C36 pad 1: /camera/12V -> +12VA
- C37 pad 2: /camera/-7V -> -7V0A
- C38 pad 1: /h-driver/3V3 -> +3V3
- C39 pad 1: /h-driver/1V8 -> +1V8A
- C4 pad 2: GND -> GNDPWR
- C40 pad 1: /h-driver/3V3 -> +3V3
- C41 pad 1: /h-driver/1V8 -> +1V8A
- C42 pad 1: /h-driver/3V3 -> +3V3
- C43 pad 1: /h-driver/1V8 -> +1V8A
- C44 pad 1: /h-driver/3V3 -> +3V3
- C45 pad 1: /h-driver/1V8 -> +1V8A
- C46 pad 1: /h-driver/3V3 -> +1V8A
- C47 pad 1: /h-driver/3V3 -> +1V8A
- C48 pad 1: /h-driver/IN_A+ -> /h-driver/ADC_INA
- C49 pad 1: /h-driver/IN_B+ -> /h-driver/ADC_INB
- C5 pad 1: /power-supply/-7V -> /power-supply/-8V
- C7 pad 2: GND -> GNDPWR
- C9 pad 2: GND -> GNDPWR
- D2 pad 2: /camera/12V -> +12VA
- L1 pad 1: /power-supply/-7V -> /power-supply/-8V
- L8 pad 2: /power-supply/1V8 -> +1V8
- R10 pad 1: /camera/12V -> /power-supply/5V5
- R10 pad 2: /camera/B1 -> Net-(R10-Pad2)
- R11 pad 1: /camera/B1 -> Net-(C24-Pad1)
- R12 pad 1: /camera/E1 -> Net-(R12-Pad1)
- R13 pad 1: /camera/CCD_OUT1 -> -7V0A
- R13 pad 2: GND -> /power-supply/SENSE
- R14 pad 1: /camera/12V -> /power-supply/SENSE
- R14 pad 2: /camera/B2 -> GND
- R15 pad 1: /camera/B2 -> Net-(C54-Pad1)
- R15 pad 2: GND -> +5VA
- R16 pad 1: /power-supply/1V8 -> +1V8
- R17 pad 2: GND -> GNDPWR
- R2 pad 2: /power-supply/-7V -> /power-supply/-8V
- R20 pad 1: /camera/E2 -> +12VA
- R20 pad 2: GND -> Net-(C56-Pad1)
- R21 pad 1: /camera/CCD_OUT2 -> Net-(C57-Pad1)
- R21 pad 2: GND -> +5VA
- R22 pad 1: /camera/ENH -> +12VA
- R22 pad 2: GND -> Net-(C59-Pad1)
- U1 pad 5: GND -> (no net)
- U10 pad 15: /camera/12V -> +12VA
- U10 pad 17: /camera/LH1_1 -> /camera/OHL
- U10 pad 18: /camera/H1S_1 -> /camera/OH1
- U10 pad 19: /camera/H1S_1 -> /camera/OH1
- U10 pad 20: /camera/H2S_1 -> /camera/OH2
- U10 pad 21: /camera/H2S_1 -> /camera/OH2
- U10 pad 22: /camera/H2S_1 -> /camera/OH2
- U10 pad 23: /camera/H2S_1 -> /camera/OH2
- U10 pad 24: /camera/H1S_1 -> /camera/OH1
- U10 pad 25: /camera/H1S_1 -> /camera/OH1
- U10 pad 26: /camera/LH1_1 -> /camera/OHL
- U10 pad 28: /camera/12V -> +12VA
- U10 pad 7: /camera/-7V -> -7V0A
- U2 pad 10: /power-supply/+12V -> /power-supply/13V5
- U2 pad 11: GND -> GNDPWR
- U3 pad 1: /power-supply/5V0 -> -7V0A
- U3 pad 2: Net-(L3-Pad2) -> /power-supply/SENSE
- U3 pad 4: Net-(L3-Pad1) -> GND
- U3 pad 5: /power-supply/5V5 -> /power-supply/-8V
- U3 pad 6: /power-supply/5V5 -> GND
- U3 pad 7: /power-supply/5V5 -> GND
- U3 pad 8: /power-supply/5V5 -> /power-supply/-8V
- U4 pad 1: /camera/3V3 -> GND
- U4 pad 10: /camera/ORG -> GND
- U4 pad 11: /camera/LH1_1 -> /camera/ORG
- U4 pad 12: /camera/H2S_1 -> (no net)
- U4 pad 13: /camera/H1S_1 -> GND
- U4 pad 14: /camera/5V0 -> +5VA
- U4 pad 2: /camera/H1 -> (no net)
- U4 pad 3: /camera/H2 -> /camera/OH2
- U4 pad 4: /camera/HL -> GND
- U4 pad 5: /camera/RG -> (no net)
- U4 pad 6: (no net) -> /camera/OH1
- U4 pad 8: /camera/ENH -> /camera/OHL
- U7 pad 1: GND -> GNDPWR
- U8 pad 1: Net-(U8-Pad1) -> (no net)
- U8 pad 3: /power-supply/3V3 -> +3V3
- U8 pad 5: /power-supply/3V3 -> +3V3
- U8 pad 6: GND -> /power-supply/LMZ_PGND
- U9 pad 1: /camera/3V3 -> /power-supply/13V5
- U9 pad 2: /camera/XSHT -> GND
- U9 pad 3: /camera/XV2 -> (no net)
- U9 pad 4: GND -> /power-supply/13V5
- U9 pad 5: /camera/XSGV2 -> +12VA
Routing:
- net /power-supply/5V5: track 160.3 -> 13.9 mm, vias 7 -> 0
- net GND: track 164.6 -> 38.5 mm, vias 25 -> 0
- net /power-supply/5V0: track 63.0 -> 0.00 mm
- net /power-supply/+12V: track 34.3 -> 0.00 mm, vias 4 -> 0
- net VIN*: track 33.7 -> 0.00 mm
- net /power-supply/-7V: track 29.2 -> 0.00 mm, vias 2 -> 0
- net /power-supply/1V8: track 27.5 -> 0.00 mm
- net /camera/OH1: track 0.00 -> 23.2 mm, vias 0 -> 2
- net /camera/ORG: track 0.00 -> 21.7 mm, vias 0 -> 2
- net /camera/SHT: track 0.00 -> 21.6 mm, vias 0 -> 2
- net /camera/OH2: track 0.00 -> 21.3 mm, vias 0 -> 2
- net /camera/OHL: track 0.00 -> 21.3 mm, vias 0 -> 2
- net /power-supply/3V3: track 19.8 -> 0.00 mm, vias 2 -> 0
- net /power-supply/13V5: track 0.00 -> 14.1 mm
- net /power-supply/LMZ_PGND: track 0.00 -> 10.6 mm, vias 0 -> 1
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- removed copper zone on F.Cu, net /power-supply/+12V
- removed copper zone on F.Cu, net /power-supply/-7V
- removed copper zone on F.Cu, net /power-supply/3V3
- removed copper zone on F.Cu, net /power-supply/5V5
- removed copper zone on B.Cu, net GND
- removed copper zone on F.Cu, net GND
- removed copper zone on F.Cu, net VIN*
Other:
- board size 40 x 40 mm -> 105 x 50 mm
- board text removed: "+"
- board text removed: "-"
- board text removed: "-7.0V"
- board text removed: "1.8V"
- board text removed: "12.0V"
- board text removed: "3.3V"
- board text removed: "5.0V"
- board text removed: "5.5V"

Commit message: Work on power system and horizontal driver.
Parts:
- added J2: PMOD, Connector_PinHeader_2.54mm:PinHeader_2x06_P2.54mm_Horizontal, F.Cu at (201.6, 43.3)
- added J3: PMOD, Connector_PinHeader_2.54mm:PinHeader_2x06_P2.54mm_Horizontal, F.Cu at (200.8, 97.4)
- added J4: PMOD, Connector_PinHeader_2.54mm:PinHeader_2x06_P2.54mm_Horizontal, F.Cu at (200.7, 79.7)
- added J5: PMOD, Connector_PinHeader_2.54mm:PinHeader_2x06_P2.54mm_Horizontal, F.Cu at (200.9, 61.9)
Connections:
- U1 pad 5: (no net) -> /power-supply/IGND
- U11 pad 3: (no net) -> Net-(U11-Pad3)
- U11 pad 6: (no net) -> Net-(U11-Pad6)
- U12 pad 4: (no net) -> Net-(U12-Pad4)
- U13 pad 12: (no net) -> /XV2
- U13 pad 13: (no net) -> /XSGV2
- U13 pad 14: (no net) -> /XV1
- U13 pad 15: (no net) -> /XV3
- U13 pad 16: (no net) -> /XSGV3
- U13 pad 17: (no net) -> /XV4
- U13 pad 18: (no net) -> /XSHT
- U4 pad 12: (no net) -> /CCD_RG
- U4 pad 2: (no net) -> /CCD_H2
- U4 pad 5: (no net) -> /CCD_H1
- U4 pad 9: (no net) -> /CCD_HL
- U6 pad 11: (no net) -> /h-driver/ADC_OUT_A0+
- U6 pad 12: (no net) -> /h-driver/ADC_OUT_A0-
- U6 pad 13: (no net) -> /h-driver/ADC_OUT_A1+
- U6 pad 14: (no net) -> /h-driver/ADC_OUT_A1-
- U6 pad 15: (no net) -> /h-driver/ADC_OUT_TCLK+
- U6 pad 16: (no net) -> /h-driver/ADC_OUT_TCKL-
- U6 pad 17: (no net) -> /h-driver/ADC_OUT_B0+
- U6 pad 18: (no net) -> /h-driver/ADC_OUT_B0-
- U6 pad 19: (no net) -> /h-driver/ADC_OUT_B1+
- U6 pad 2: (no net) -> /ADC_SL
- U6 pad 20: (no net) -> /h-driver/ADC_OUT_B1-
- U6 pad 23: (no net) -> Net-(U6-Pad23)
- U6 pad 25: (no net) -> Net-(U6-Pad25)
- U6 pad 26: (no net) -> /ADC_CLI
- U6 pad 29: (no net) -> Net-(U6-Pad29)
- U6 pad 3: (no net) -> /ADC_SDATA
- U6 pad 4: (no net) -> /ADC_SCK
- U6 pad 7: (no net) -> /ADC_VD
- U6 pad 8: (no net) -> /ADC_HD
- U8 pad 1: (no net) -> Net-(U8-Pad1)

Commit message: Start up work to revive this project.
Parts:
- added C1: 0.01, Capacitor_SMD:C_0603_1608Metric, F.Cu at (154.8, 97.2)
- added C63: 3.3/20V, Capacitor_Tantalum_SMD:CP_EIA-1608-08_AVX-J, F.Cu at (157.0, 97.2)
- added J1: Barrel_Jack_Switch, Connector_BarrelJack:BarrelJack_Wuerth_6941xx301002, F.Cu at (94.0, 46.2)
- added REF**: PT-LH030CSM, Engstad:PT-LH030CSM, F.Cu at (160.0, 85.0)
- C28: value 1u/35V -> 1uF/35V; footprint Capacitor_SMD:C_1210_3225Metric -> Capacitor_Tantalum_SMD:CP_EIA-1608-08_AVX-J
- C29: value 0.1uF -> 0.1uF/35V; footprint Capacitor_SMD:C_0603_1608Metric -> Capacitor_SMD:C_0805_2012Metric
- C30: value 2200pF -> 2.2uF/50V; footprint Capacitor_SMD:C_0603_1608Metric -> Capacitor_SMD:C_0805_2012Metric
- C34: footprint Capacitor_SMD:CP_Elec_4x5.3 -> Capacitor_Tantalum_SMD:CP_EIA-3528-12_Kemet-T
- C36, C37: footprint Capacitor_SMD:CP_Elec_4x5.3 -> Capacitor_Tantalum_SMD:CP_EIA-1608-08_AVX-J
- C55, C58: value 47/20V -> 47u/20V; footprint Capacitor_SMD:CP_Elec_4x5.3 -> Capacitor_SMD:C_1206_3216Metric
- NT2: value Net-Tie_2 -> NetTie_2
- moved C52 36.1 mm to (122.0, 91.5), turned to 90 degrees
- moved J3 35.6 mm to (234.9, 107.5)
- moved J4 34.6 mm to (234.9, 84.6)
- moved C38 34.2 mm to (216.1, 88.5), turned to -90 degrees
- moved J5 34.0 mm to (234.9, 61.7)
- moved C39 33.8 mm to (212.4, 76.0), turned to 90 degrees
- moved J2 33.6 mm to (234.9, 38.9)
- moved C41 33.5 mm to (218.9, 87.7), turned to 90 degrees
- moved C47 33.4 mm to (210.5, 87.0), turned to 180 degrees
- moved R13 32.7 mm to (119.5, 90.9), turned to 90 degrees
- moved U6 32.6 mm to (214.6, 82.1)
- moved C40 32.2 mm to (214.3, 76.0), turned to 90 degrees
- moved C50 32.2 mm to (117.8, 92.2), turned to 90 degrees
- moved C45 31.4 mm to (207.6, 79.2), turned to 180 degrees
- moved C42 31.3 mm to (207.6, 82.8)
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Connections:
- net /camera/OH1 renamed /camera/O_H1
- net /camera/OH2 renamed /camera/O_H2
- net /camera/OHL renamed /camera/O_HL
- net /camera/ORG renamed /camera/O_RG
- net /h-driver/ADC_INA renamed /camera/CCD_OUT1
- net /h-driver/ADC_INB renamed /camera/CCD_OUT2
- net /h-driver/ADC_OUT_TCKL- renamed /h-driver/ADC_OUT_TCLK-
- net Net-(C28-Pad1) renamed /camera/SH_DEL
- net Net-(C48-Pad2) renamed /h-driver/IN_A-
- net Net-(C49-Pad2) renamed /h-driver/IN_B-
- net Net-(C54-Pad1) renamed /camera/ISF1
- net Net-(C56-Pad1) renamed /camera/IDRV1
- net Net-(C57-Pad1) renamed /camera/ISF2
- net Net-(C59-Pad1) renamed /camera/IDRV2
- C39 pad 1: +1V8A -> +1V8
- C41 pad 1: +1V8A -> +1V8
- C43 pad 1: +1V8A -> +1V8
- C45 pad 1: +1V8A -> +1V8
- C46 pad 1: +1V8A -> +1V8
- C47 pad 1: +1V8A -> +1V8
- C53 pad 1: +3V3 -> +3.3VA
- J2 pad 10: /ADC_SDATA -> /CCD_H2
- J2 pad 11: Net-(J2-Pad11) -> unconnected-(J2-Pin_11-Pad11)
- J2 pad 12: Net-(J2-Pad12) -> /CCD_H1
- J2 pad 5: Net-(J2-Pad5) -> unconnected-(J2-Pin_5-Pad5)
- J2 pad 6: /ADC_SL -> /CCD_RG
- J2 pad 7: Net-(J2-Pad7) -> unconnected-(J2-Pin_7-Pad7)
- J2 pad 8: /ADC_SCK -> /CCD_HL
- J2 pad 9: Net-(J2-Pad9) -> unconnected-(J2-Pin_9-Pad9)
- J3 pad 10: /XSGV1 -> /XSGV3
- J3 pad 6: /ADC_VD -> unconnected-(J3-Pin_6-Pad6)
- J4 pad 10: /CCD_H2 -> /ADC_SCK
- J4 pad 12: /CCD_H1 -> /ADC_SDATA
- J5 pad 6: /CCD_RG -> /ADC_SL
- J5 pad 8: /CCD_HL -> /ADC_VD
- U10 pad 5: GND -> +12VA
- U11 pad 3: Net-(U11-Pad3) -> unconnected-(U11-NC-Pad3)
- U11 pad 6: Net-(U11-Pad6) -> unconnected-(U11-NC-Pad6)
- U12 pad 4: Net-(U12-Pad4) -> unconnected-(U12-PG-Pad4)
- U13 pad 20: +3V3 -> +3.3VA
- U6 pad 1: +1V8A -> +1V8
- U6 pad 21: +1V8A -> +1V8
- U6 pad 23: Net-(U6-Pad23) -> unconnected-(U6-NC1-Pad23)
- U6 pad 25: Net-(U6-Pad25) -> unconnected-(U6-CLK_OUT-Pad25)
- U6 pad 29: Net-(U6-Pad29) -> unconnected-(U6-NC2-Pad29)
- U6 pad 30: +1V8A -> +1V8
- U6 pad 32: +1V8A -> +1V8
- U6 pad 9: +1V8A -> +1V8
- U8 pad 1: Net-(U8-Pad1) -> unconnected-(U8-EN-Pad1)
Routing:
- net +3V3: track 8.10 -> 103.6 mm, vias 2 -> 7
- net /ADC_SL: track 0.00 -> 55.8 mm, vias 0 -> 1
- net +1V8: track 0.00 -> 53.7 mm, vias 0 -> 5
- net GND: track 38.5 -> 88.5 mm, vias 0 -> 17
- net /ADC_VD: track 0.00 -> 36.2 mm, vias 0 -> 1
- net /ADC_SDATA: track 0.00 -> 35.5 mm, vias 0 -> 1
- net /h-driver/ADC_OUT_A1-: track 0.00 -> 35.3 mm
- net /h-driver/ADC_OUT_A1+: track 0.00 -> 35.2 mm
- net /h-driver/ADC_OUT_TCLK-: track 0.00 -> 33.9 mm
- net /h-driver/ADC_OUT_B1-: track 0.00 -> 33.9 mm
- net /h-driver/ADC_OUT_A0-: track 0.00 -> 33.9 mm
- net /h-driver/ADC_OUT_B0-: track 0.00 -> 33.8 mm
- net /h-driver/ADC_OUT_A0+: track 0.00 -> 33.8 mm
- net /h-driver/ADC_OUT_B1+: track 0.00 -> 33.7 mm
- net /h-driver/ADC_OUT_B0+: track 0.00 -> 33.7 mm
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- added copper zone on B.Cu, net GND
Other:
- board size 105 x 50 mm -> 161.3 x 91.4 mm
- net class Default removed
