File: pcb/fpga.sch (KiCad schematic (older format))
At the start: 26 parts, among them P4 CONN_02X02, P5 VDRV, P6 HDRV, U2 XILINX-6SLX16-CSG225

Commit message: lastest at home
Parts:
- removed P4: CONN_02X02, w_pin_strip:pin_strip_2x2, symbol CONN_02X02
- added JP1: Jumper_NO_Small, engstad:pin-socket-2, symbol Jumper_NO_Small
- C13: footprint engstad:0805 -> engstad:C0603
- C14, C15, C16, C17, C18: footprint (none) -> engstad:C0603
- C19, C20, C21, C22, C23, C24, C25, C31, C33: footprint engstad:0805 -> engstad:0402
Connections:
- net FPGA-COMP is gone; now on net +3V3: U2.L10 (CMPCS_B_2)
- net +3V3: now also JP1.1; no longer C16.1, C22.1, C28.1, U2.D14 (VCCO_1[4]), U2.H14 (VCCO_1[4]), U2.J12 (VCCO_1[4]), U2.M14 (VCCO_1[4])
- net FPGA-A0+: now also U2.M11 (IO_L12P_D1_MISO2_2); no longer U2.P11 (IO_L3P_D0_DIN_MISO_MISO1_2)
- net FPGA-A0-: now also U2.N11 (IO_L12N_D2_MISO3_2); no longer U2.R11 (IO_L3N_MOSI_CSI_B_MISO0_2)
- net GND: no longer U2.R13 (IO_L2N_CMPMOSI_2)
- net HEN#: now also U2.J3 (IO_L43N_GCLK22_IRDY2_M3CASN_3); no longer U2.K1 (IO_L40N_M3DQ7_3)
- net at U2.K4 (IO_L43P_GCLK23_M3RASN_3): now also P6.5 (P5)
- net CCLK: now reaches U2.N12 (IO_L1P_CCLK_2)
- net FPGA-CLKIN: no longer names the net of U2.N7 (IO_L30N_GCLK0_USERCCLK_2)
- net FPGA-DONE renamed DONE
- net FPGA-INIT-B renamed INIT-B
- net FPGA-PROG-B renamed PROG-B
- new net DIN: U2.P11 (IO_L3P_D0_DIN_MISO_MISO1_2)
- new net VCC1: C16.1, C22.1, C28.1, JP1.2, U2.D14 (VCCO_1[4]), U2.H14 (VCCO_1[4]), U2.J12 (VCCO_1[4]), U2.M14 (VCCO_1[4])
- no-connect marks 113 -> 111
Other:
- note added: "DOUT (not used)"
- note added: "reserved"
- moved on the sheet: P5, P6, U2D
