File: pcb/h-driver.sch (KiCad schematic (older format))
At the start: 15 parts, among them P2 CONN_01X18, P3 CONN_01X18, U11 ADDI7013

Commit message: Cleanups
Connections:
- net labels added: INP_A+, INP_B+
Changed lines of the file:
@@
 	0    -1   -1   0
 $EndComp
+Text Label 7200 2500 0    60   ~ 0
+INP_A+
+Text Label 7200 2600 0    60   ~ 0
+INP_B+
 $EndSCHEMATC

Commit message: More work
Parts:
- U11: footprint camera:csp-bga-bc-76-3 -> engstad:csp-bga-bc-76-3
Changed lines of the file:
@@
 LIBS:contrib
 LIBS:valves
-LIBS:camera
+LIBS:engstad
+LIBS:sony
 LIBS:AstroCam-cache
 EELAYER 25 0
@@
 F 0 "U11" H 2100 2950 60  0000 C CNN
 F 1 "ADDI7013" H 2100 2200 60  0000 C CNN
-F 2 "camera:csp-bga-bc-76-3" H 2200 2150 60  0001 C CNN
+F 2 "engstad:csp-bga-bc-76-3" H 2200 2150 60  0001 C CNN
 F 3 "" H 2200 2150 60  0000 C CNN
 	1    2100 2200
@@
 F 0 "U11" H 6450 2950 60  0000 C CNN
 F 1 "ADDI7013" H 6450 2200 60  0000 C CNN
-F 2 "camera:csp-bga-bc-76-3" H 6550 2150 60  0001 C CNN
+F 2 "engstad:csp-bga-bc-76-3" H 6550 2150 60  0001 C CNN
 F 3 "" H 6550 2150 60  0000 C CNN
 	2    6450 2200
@@
 F 0 "U11" H 2100 5300 60  0000 C CNN
 F 1 "ADDI7013" H 2100 4550 60  0000 C CNN
-F 2 "camera:csp-bga-bc-76-3" H 2200 4500 60  0001 C CNN
+F 2 "engstad:csp-bga-bc-76-3" H 2200 4500 60  0001 C CNN
 F 3 "" H 2200 4500 60  0000 C CNN
 	3    2100 4550
@@
 F 0 "U11" H 4950 5250 60  0000 C CNN
 F 1 "ADDI7013" H 4950 4500 60  0000 C CNN
-F 2 "camera:csp-bga-bc-76-3" H 5050 4450 60  0001 C CNN
+F 2 "engstad:csp-bga-bc-76-3" H 5050 4450 60  0001 C CNN
 F 3 "" H 5050 4450 60  0000 C CNN
 	4    4950 4500

Commit message: Adding ADDI4800 to schematics
Parts:
- U11: symbol ADDI7013 -> ADDI7013-RESCUE-AstroCam
Changed lines of the file:
@@
 $EndDescr
 $Comp
-L ADDI7013 U?
+L ADDI7013-RESCUE-AstroCam U?
 U 1 1 557AD8F3
 P 2100 2200
@@
 $EndComp
 $Comp
-L ADDI7013 U?
+L ADDI7013-RESCUE-AstroCam U?
 U 2 1 557B0AAF
 P 6450 2200
@@
 $EndComp
 $Comp
-L ADDI7013 U?
+L ADDI7013-RESCUE-AstroCam U?
 U 3 1 557B0FDF
 P 2100 4550
@@
 1V8
 $Comp
-L ADDI7013 U?
+L ADDI7013-RESCUE-AstroCam U?
 U 4 1 557B715D
 P 4950 4500

Commit message: Latest, greatest.
Parts:
- removed U11: ADDI7013, engstad:csp-bga-bc-76-3, symbol ADDI7013-RESCUE-AstroCam
- added U4: ADDI7013, engstad:csp-bga-bc-76-3, symbol ADDI7013
Connections:
- net labels added: INP_A-, INP_B-
- wire segments 83 -> 45
Other:
- note added: "Power Ground\n"
- note added: "Power Input"
- moved on the sheet: C38, C39, C40, C41, C42, C43, C44, C45, C46, C47, C48, C49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

Commit message: work
Parts:
- removed P2, P3: CONN_01X18, Pin_Headers:Pin_Header_Straight_1x18, symbol CONN_01X18
- added P1: CONN_02X04, w_pin_strip:pin_strip_4x2, symbol CONN_02X04
- added P2, P3: CONN_01X04, w_pin_strip:pin_strip_4, symbol CONN_01X04
- added T1: NET-TIE, engstad:net-tie-0.5mm, symbol NET-TIE
- C1: renamed from C47; footprint Capacitors_SMD:C_0603_HandSoldering -> smd:SM0603
- C10: renamed from C43; footprint Capacitors_SMD:C_0603_HandSoldering -> smd:SM0603
- C11: renamed from C48; footprint Capacitors_SMD:C_0603_HandSoldering -> smd:SM0603
- C12: renamed from C49; footprint Capacitors_SMD:C_0603_HandSoldering -> smd:SM0603
- C2: renamed from C42; footprint Capacitors_SMD:C_0603_HandSoldering -> smd:SM0603
- C3: renamed from C46; footprint Capacitors_SMD:C_0603_HandSoldering -> smd:SM0603
- C4: renamed from C44; footprint Capacitors_SMD:C_0603_HandSoldering -> smd:SM0603
- C5: renamed from C45; footprint Capacitors_SMD:C_0603_HandSoldering -> smd:SM0603
- C6: renamed from C38; footprint Capacitors_SMD:C_0603_HandSoldering -> smd:SM0603
- C7: renamed from C41; footprint Capacitors_SMD:C_0603_HandSoldering -> smd:SM0603
- C8: renamed from C39; footprint Capacitors_SMD:C_0603_HandSoldering -> smd:SM0603
- C9: renamed from C40; footprint Capacitors_SMD:C_0603_HandSoldering -> smd:SM0603
- renumbered U4 to U1
Connections:
- net labels added: +3V3, 1V8A, 3V3A, ADC-SCK, ADC-SDATA, ADC-SL, ADC-SYNC/RESET#, FPGA-A0+, FPGA-A0-, FPGA-A1+, FPGA-A1-, FPGA-B0+, FPGA-B0-, FPGA-B1+, FPGA-B1-, FPGA-CLK+, FPGA-CLK-, FPGA-CLKOUT, FV, GNDA, LV
- net labels removed: 1V8, 3V3, A0+, A0-, A1+, A1-, B0+, B0-, B1+, B1-, H3, H4, SYNC, TCLK+, TCLK-
- wire segments 45 -> 109
- no-connect marks 0 -> 2
Other:
- note added: "Can be 1.8V"
- moved on the sheet: C1, C10, C2, C3, C4, C5, C6, C7, C8, C9, U1A, U1C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

Commit message: lastest at home
Parts:
- removed T1: NET-TIE, engstad:net-tie-0.5mm, symbol NET-TIE
- C1, C10, C11, C12, C2, C3, C4, C5, C6, C7, C8, C9: footprint smd:SM0603 -> engstad:C0603
Changed lines of the file:
@@
 F 0 "C11" V 6750 1500 50  0000 L CNN
 F 1 "0.1u" V 7050 1500 50  0000 L CNN
-F 2 "smd:SM0603" H 6938 1450 30  0001 C CNN
+F 2 "engstad:C0603" H 6938 1450 30  0001 C CNN
 F 3 "" H 6900 1600 60  0000 C CNN
 	1    6900 1600
@@
 F 0 "C12" V 6750 2400 50  0000 L CNN
 F 1 "0.1u" V 7050 2400 50  0000 L CNN
-F 2 "smd:SM0603" H 6938 2350 30  0001 C CNN
+F 2 "engstad:C0603" H 6938 2350 30  0001 C CNN
 F 3 "" H 6900 2500 60  0000 C CNN
 	1    6900 2500
@@
 F 0 "C6" H 4610 3870 50  0000 L CNN
 F 1 "0.1uF" H 4610 3720 50  0000 L CNN
-F 2 "smd:SM0603" H 4600 3800 60  0001 C CNN
+F 2 "engstad:C0603" H 4600 3800 60  0001 C CNN
 F 3 "" H 4600 3800 60  0000 C CNN
 	1    4600 3800
@@
 F 0 "C9" H 4860 3870 50  0000 L CNN
 F 1 "0.1uF" H 4860 3720 50  0000 L CNN
-F 2 "smd:SM0603" H 4850 3800 60  0001 C CNN
+F 2 "engstad:C0603" H 4850 3800 60  0001 C CNN
 F 3 "" H 4850 3800 60  0000 C CNN
 	1    4850 3800
@@
 F 0 "C8" H 4675 4225 50  0000 R CNN
 F 1 "0.1uF" H 4675 4375 50  0000 R CNN
-F 2 "smd:SM0603" H 4700 4300 60  0001 C CNN
+F 2 "engstad:C0603" H 4700 4300 60  0001 C CNN
 F 3 "" H 4700 4300 60  0000 C CNN
 	1    4700 4300
@@
 F 0 "C7" H 4625 5075 50  0000 L CNN
 F 1 "0.1uF" H 4625 4925 50  0000 L CNN
-F 2 "smd:SM0603" H 4600 5000 60  0001 C CNN
+F 2 "engstad:C0603" H 4600 5000 60  0001 C CNN
 F 3 "" H 4600 5000 60  0000 C CNN
 	1    4600 5000
@@
 F 0 "C10" H 4910 5070 50  0000 L CNN
 F 1 "0.1uF" H 4910 4920 50  0000 L CNN
-F 2 "smd:SM0603" H 4900 5000 60  0001 C CNN
+F 2 "engstad:C0603" H 4900 5000 60  0001 C CNN
 F 3 "" H 4900 5000 60  0000 C CNN
 	1    4900 5000
@@
 F 0 "C2" H 2660 3870 50  0000 L CNN
 F 1 "0.1uF" H 2660 3720 50  0000 L CNN
-F 2 "smd:SM0603" H 2650 3800 60  0001 C CNN
+F 2 "engstad:C0603" H 2650 3800 60  0001 C CNN
 F 3 "" H 2650 3800 60  0000 C CNN
 	1    2650 3800
@@
 F 0 "C1" H 2410 4320 50  0000 L CNN
 F 1 "4.7uF" H 2410 4170 50  0000 L CNN
-F 2 "smd:SM0603" H 2400 4250 60  0001 C CNN
+F 2 "engstad:C0603" H 2400 4250 60  0001 C CNN
 F 3 "" H 2400 4250 60  0000 C CNN
 	1    2400 4250
@@
 F 0 "C3" H 2660 4320 50  0000 L CNN
 F 1 "0.1uF" H 2660 4170 50  0000 L CNN
-F 2 "smd:SM0603" H 2650 4250 60  0001 C CNN
+F 2 "engstad:C0603" H 2650 4250 60  0001 C CNN
 F 3 "" H 2650 4250 60  0000 C CNN
 	1    2650 4250
@@
 F 0 "C5" V 2550 5100 50  0000 C CNN
 F 1 "0.1uF" V 2750 5100 50  0000 C CNN
-F 2 "smd:SM0603" H 2650 5100 60  0001 C CNN
+F 2 "engstad:C0603" H 2650 5100 60  0001 C CNN
 F 3 "" H 2650 5100 60  0000 C CNN
 	1    2650 5100
@@
 F 0 "C4" V 2550 4750 50  0000 C CNN
 F 1 "0.1uF" V 2750 4750 50  0000 C CNN
-F 2 "smd:SM0603" H 2650 4750 60  0001 C CNN
+F 2 "engstad:C0603" H 2650 4750 60  0001 C CNN
 F 3 "" H 2650 4750 60  0000 C CNN
 	1    2650 4750
@@
 	0    1    1    0
 $EndComp
-$Comp
-L GNDA #PWR014
-U 1 1 56AD6585
-P 7850 5850
-F 0 "#PWR014" H 7850 5600 50  0001 C CNN
-F 1 "GNDA" V 7850 5650 50  0000 C CNN
-F 2 "" H 7850 5850 50  0000 C CNN
-F 3 "" H 7850 5850 50  0000 C CNN
-	1    7850 5850
-	0    -1   -1   0
-$EndComp
-$Comp
-L GND #PWR015
-U 1 1 56AD6618
-P 7350 5850
-F 0 "#PWR015" H 7350 5600 50  0001 C CNN
-F 1 "GND" V 7350 5650 50  0000 C CNN
-F 2 "" H 7350 5850 50  0000 C CNN
-F 3 "" H 7350 5850 50  0000 C CNN
-	1    7350 5850
-	0    1    1    0
-$EndComp
-$Comp
-L NET-TIE T1
-U 1 1 56AD6658
-P 7600 5850
-F 0 "T1" H 7600 6103 60  0000 C CNN
-F 1 "NET-TIE" H 7600 5997 60  0000 C CNN
-F 2 "engstad:net-tie-0.5mm" H 7600 6000 60  0001 C CNN
-F 3 "" H 7600 6000 60  0000 C CNN
-	1    7600 5850
-	1    0    0    -1
-$EndComp
 Text Notes 1800 4600 2    50   ~ 0
 Can be 1.8V
@@
 HD
 $Comp
-L +3V3 #PWR016
+L +3V3 #PWR014
 U 1 1 56FB3873
 P 2300 3650
-F 0 "#PWR016" H 2300 3500 50  0001 C CNN
+F 0 "#PWR014" H 2300 3500 50  0001 C CNN
 F 1 "+3V3" V 2318 3777 50  0000 L CNN
 F 2 "" H 2300 3650 50  0000 C CNN
@@
 $EndComp
 $Comp
-L +3V3 #PWR017
+L +3V3 #PWR015
 U 1 1 56FB38D5
 P 2300 4100
-F 0 "#PWR017" H 2300 3950 50  0001 C CNN
+F 0 "#PWR015" H 2300 3950 50  0001 C CNN
 F 1 "+3V3" V 2318 4227 50  0000 L CNN
 F 2 "" H 2300 4100 50  0000 C CNN
@@
 $EndComp
 $Comp
-L +3V3 #PWR018
+L +3V3 #PWR016
 U 1 1 56FB3A6D
 P 2300 4600
-F 0 "#PWR018" H 2300 4450 50  0001 C CNN
+F 0 "#PWR016" H 2300 4450 50  0001 C CNN
 F 1 "+3V3" V 2318 4727 50  0000 L CNN
 F 2 "" H 2300 4600 50  0000 C CNN
