File: pcb/h-driver.sch (KiCad schematic (older format))
At the start: 15 parts, among them P2 CONN_01X18, P3 CONN_01X18, U11 ADDI7013

Commit message: Safety checkin.
Parts:
- removed P2, P3: CONN_01X18, Pin_Headers:Pin_Header_Straight_1x18, symbol CONN_01X18
- removed unit 1 of U11
- removed unit 2 of U11
- added U6: ADDI7013, symbol @Engstad:ADDI7013
- C38, C39, C40, C41, C42, C43, C44, C45, C46, C47: symbol C_Small -> Device:C_Small
- C48, C49: symbol C -> Device:C
- U11: symbol ADDI7013 -> AstroCam-rescue:ADDI7013
Connections:
- net labels added: +1V8, +1V8A, +3V3, ADC_1V8, ADC_1V8A, ADC_3V3, ADC_HD, ADC_HOR_H1, ADC_HOR_H2, ADC_HOR_H3, ADC_HOR_H4, ADC_HOR_HL1, ADC_HOR_HL2, ADC_HOR_RG1, ADC_HOR_RG2, ADC_INA, ADC_INB, ADC_OUT_A0+, ADC_OUT_A0-, ADC_OUT_A1+, ADC_OUT_A1-, ADC_OUT_B0+, ADC_OUT_B0-, ADC_OUT_B1+, ADC_OUT_B1-, ADC_OUT_TCKL-, ADC_OUT_TCLK+, ADC_SCK, ADC_SDATA, ADC_SL, ADC_SYNC, ADC_VD
- net labels removed: 3V3, A0+, A0-, A1+, A1-, B0+, B0-, B1+, B1-, CLI, GP01, GP02, GP03, GP04, H1, H2, H3, H4, HD, HL1, HL2, IN_A+, IN_A-, IN_B+, IN_B-, RG1, RG2, SCK, SDATA, SL, SYNC, TCLK+, TCLK-, VD
- wire segments 83 -> 141
Other:
- moved on the sheet: U11C, U11D

Commit message: A little more work.
Parts:
- removed U11: ADDI7013, camera:csp-bga-bc-76-3, symbol AstroCam-rescue:ADDI7013
- removed U6: ADDI7013, symbol @Engstad:ADDI7013
- added U6: AD9978, Engstad:qfn-40, symbol @Engstad:AD9978
- C38, C39, C40, C41, C42, C43, C45: footprint Capacitors_SMD:C_0603_HandSoldering -> Capacitor_SMD:C_0603_1608Metric
- C44, C46: value 0.1uF -> 4.7uF; footprint Capacitors_SMD:C_0603_HandSoldering -> Capacitor_SMD:C_0805_2012Metric
- C47: value 4.7uF -> 0.1uF; footprint Capacitors_SMD:C_0603_HandSoldering -> Capacitor_SMD:C_0603_1608Metric
- C48, C49: footprint Capacitors_SMD:C_0603_HandSoldering -> Capacitor_SMD:C_0603_1608Metric; symbol Device:C -> Device:C_Small
Connections:
- net +1V8 is gone; now on net +1V8A: C43.1, C45.1
- net +1V8A: now also C46.1, C47.1, U6.1 (AVDD1), U6.21 (LVDD), U6.30 (AVDD2), U6.32 (AVDD3), U6.9 (DVDD)
- net +3V3: now also U6.27 (INVDD1), U6.36 (INVDD2), U6.6 (IOVDD); no longer C46.1, C47.1
- net ADC_HD: now also U6.8 (HD)
- net ADC_OUT_A0+: now also U6.11 (DOUT0+)
- net ADC_OUT_A0-: now also U6.12 (DOUT0-)
- net ADC_OUT_A1+: now also U6.13 (DOUT1+)
- net ADC_OUT_A1-: now also U6.14 (DOUT1-)
- net ADC_OUT_B0+: now also U6.17 (DOUT2+)
- net ADC_OUT_B0-: now also U6.18 (DOUT2-)
- net ADC_OUT_B1+: now also U6.19 (DOUT3+)
- net ADC_OUT_B1-: now also U6.20 (DOUT3-)
- net ADC_OUT_TCKL-: now also U6.16 (TCKL-)
- net ADC_OUT_TCLK+: now also U6.15 (TCLK+)
- net ADC_SCK: now also U6.4 (SCK)
- net ADC_SDATA: now also U6.3 (SDATA)
- net ADC_SL: now also U6.2 (SL)
- net ADC_VD: now also U6.7 (VD)
- net GND: now also U6.10 (DVSS), U6.22 (LVSS), U6.24 (LVSS), U6.28 (INVSS1), U6.31 (AVSS2), U6.33 (AVSS3), U6.35 (IN_A+), U6.37 (INVSS2), U6.39 (IN_B+), U6.40 (AVSS1), U6.41 (GND-PAD), U6.5 (IOVSS)
- net at C48.2: now also U6.34 (IN_A-)
- net at C49.2: now also U6.38 (IN_B-)
- new net ADC_CLI: U6.26 (CLI)
- no-connect marks 0 -> 1
Other:
- note added: "Near INVDD1"
- note added: "Near INVDD2"
- note added: "Near IOVDD\n"
- note removed: "Analog Differential \nPair Outputs"
- note removed: "Control\n"
- moved on the sheet: C38, C39, C40, C41, C42, C43, C45, C48, C49

Commit message: Work on power system and horizontal driver.
Connections:
- net +1V8A: no longer U6.21 (LVDD), U6.9 (DVDD)
- net GND: no longer U6.31 (AVSS2), U6.33 (AVSS3), U6.35 (IN_A+), U6.39 (IN_B+), U6.40 (AVSS1)
- new net +1V8: U6.21 (LVDD), U6.9 (DVDD)
- new net GNDA: U6.31 (AVSS2), U6.33 (AVSS3), U6.35 (IN_A+), U6.39 (IN_B+), U6.40 (AVSS1)
Other:
- moved on the sheet: C48, C49
Changed lines of the file:
@@
 L Device:C_Small C48
 U 1 1 557B103C
-P 3700 2700
-F 0 "C48" V 3650 2750 50  0000 L CNN
-F 1 "0.1u" V 3650 2450 50  0000 L CNN
-F 2 "Capacitor_SMD:C_0603_1608Metric" H 3738 2550 30  0001 C CNN
-F 3 "" H 3700 2700 60  0000 C CNN
-	1    3700 2700
+P 3650 2700
+F 0 "C48" V 3600 2750 50  0000 L CNN
+F 1 "0.1u" V 3600 2450 50  0000 L CNN
+F 2 "Capacitor_SMD:C_0603_1608Metric" H 3688 2550 30  0001 C CNN
+F 3 "" H 3650 2700 60  0000 C CNN
+	1    3650 2700
 	0    -1   1    0
 $EndComp
@@
 L Device:C_Small C49
 U 1 1 557B105D
-P 3700 2900
-F 0 "C49" V 3650 2950 50  0000 L CNN
-F 1 "0.1u" V 3650 2650 50  0000 L CNN
-F 2 "Capacitor_SMD:C_0603_1608Metric" H 3738 2750 30  0001 C CNN
-F 3 "" H 3700 2900 60  0000 C CNN
-	1    3700 2900
+P 3650 2900
+F 0 "C49" V 3600 2950 50  0000 L CNN
+F 1 "0.1u" V 3600 2650 50  0000 L CNN
+F 2 "Capacitor_SMD:C_0603_1608Metric" H 3688 2750 30  0001 C CNN
+F 3 "" H 3650 2900 60  0000 C CNN
+	1    3650 2900
 	0    -1   1    0
 $EndComp
@@
 $EndComp
 Wire Wire Line
-	4350 2700 3800 2700
+	4350 2700 3750 2700
 Wire Wire Line
 	1950 3800 1950 3850
@@
 ADC_SL
 Wire Wire Line
-	3800 2900 4350 2900
+	3750 2900 4350 2900
 Wire Wire Line
 	4350 2800 4250 2800
-$Comp
-L power:GND #PWR0121
-U 1 1 5FCA6F27
-P 4250 2800
-F 0 "#PWR0121" H 4250 2550 50  0001 C CNN
-F 1 "GND" H 4255 2627 50  0000 C CNN
-F 2 "" H 4250 2800 50  0001 C CNN
-F 3 "" H 4250 2800 50  0001 C CNN
-	1    4250 2800
-	0    1    1    0
-$EndComp
-$Comp
-L power:GND #PWR0122
-U 1 1 5FCA71BA
-P 4250 3000
-F 0 "#PWR0122" H 4250 2750 50  0001 C CNN
-F 1 "GND" H 4255 2827 50  0000 C CNN
-F 2 "" H 4250 3000 50  0001 C CNN
-F 3 "" H 4250 3000 50  0001 C CNN
-	1    4250 3000
-	0    1    1    0
-$EndComp
 Wire Wire Line
 	4250 3000 4350 3000
 Wire Wire Line
-	3400 2700 3600 2700
+	3400 2700 3550 2700
 Text HLabel 3400 2700 0    50   Input ~ 0
 ADC_INA
@@
 Connection ~ 4300 3250
 Wire Wire Line
-	3400 2900 3600 2900
+	3400 2900 3550 2900
 Wire Wire Line
 	3400 1900 4350 1900
@@
 Wire Wire Line
 	3800 3850 4350 3850
-Connection ~ 3800 3750
 Wire Wire Line
 	4100 3650 4100 4050
@@
 	1500 4650 1900 4650
 $Comp
-L power:GND #PWR0133
-U 1 1 5FAD9C0F
-P 6000 3350
-F 0 "#PWR0133" H 6000 3100 50  0001 C CNN
-F 1 "GND" H 6005 3177 50  0000 C CNN
-F 2 "" H 6000 3350 50  0001 C CNN
-F 3 "" H 6000 3350 50  0001 C CNN
-	1    6000 3350
-	1    0    0    -1
-$EndComp
-Wire Wire Line
-	3550 3150 3800 3150
-Wire Wire Line
-	3800 3150 3800 3750
-Connection ~ 3800 3150
-Wire Wire Line
-	3800 3150 4300 3150
-$Comp
 L Device:C_Small C47
 U 1 1 5FAE1501
@@
 $EndComp
 NoConn ~ 5750 3000
+$Comp
+L power:GNDA #PWR?
+U 1 1 60C9F0F8
+P 6000 3350
+F 0 "#PWR?" H 6000 3100 50  0001 C CNN
+F 1 "GNDA" H 6005 3177 50  0000 C CNN
+F 2 "" H 6000 3350 50  0001 C CNN
+F 3 "" H 6000 3350 50  0001 C CNN
+	1    6000 3350
+	1    0    0    -1
+$EndComp
+$Comp
+L power:GNDA #PWR?
+U 1 1 60CA7B63
+P 4250 3000
+F 0 "#PWR?" H 4250 2750 50  0001 C CNN
+F 1 "GNDA" V 4255 2873 50  0000 R CNN
+F 2 "" H 4250 3000 50  0001 C CNN
+F 3 "" H 4250 3000 50  0001 C CNN
+	1    4250 3000
+	0    1    1    0
+$EndComp
+$Comp
+L power:GNDA #PWR?
+U 1 1 60CA8403
+P 4250 2800
+F 0 "#PWR?" H 4250 2550 50  0001 C CNN
+F 1 "GNDA" V 4255 2673 50  0000 R CNN
+F 2 "" H 4250 2800 50  0001 C CNN
+F 3 "" H 4250 2800 50  0001 C CNN
+	1    4250 2800
+	0    1    1    0
+$EndComp
+Wire Wire Line
+	3550 3150 4300 3150
+$Comp
+L power:+1V8 #PWR?
+U 1 1 60CB3D35
+P 3800 3600
+F 0 "#PWR?" H 3800 3450 50  0001 C CNN
+F 1 "+1V8" H 3815 3773 50  0000 C CNN
+F 2 "" H 3800 3600 50  0001 C CNN
+F 3 "" H 3800 3600 50  0001 C CNN
+	1    3800 3600
+	1    0    0    -1
+$EndComp
+Wire Wire Line
+	3800 3600 3800 3750
+Connection ~ 3800 3750
 $EndSCHEMATC
