File: pcb/usb-ctrl.sch (KiCad schematic (older format))
At the start: 64 parts, among them CON1 USB3, P7 CONN_02X10, U3 CYUSB303X, U4 MTFC4GLDDQ-4M IT, Y1 19.2 MHz

Commit message: lastest at home
Parts:
- removed RP2, RP3: 22R, w_smd_resistors:r_cat16-8, symbol R_PACK8
- added P8: UART, w_pin_strip:pin_socket_4, symbol CONN_01X04
- added R8: 47K, engstad:R0603, symbol R
- C35: footprint smd:SM0805 -> engstad:C0603
- C36, C37, C38, C39, C40, C41, C42, C43, C44, C45, C53, C54, C55, C56, C57, C58, C59, C60, C61, C62, C69: footprint smd:SM0603 -> engstad:0402
- C46, C47: footprint smd:SM0603 -> engstad:C0603
- C48: renamed from C50; footprint smd:SM0805 -> engstad:0805
- C49: renamed from C51; footprint smd:SM0805 -> engstad:0805
- C50: renamed from C52; footprint smd:SM0805 -> engstad:0805
- C51: renamed from C48; footprint smd:SM0603 -> engstad:0402
- C52: renamed from C49; footprint smd:SM0603 -> engstad:0402
- C63: renamed from C64; footprint smd:SM0603 -> engstad:0402
- C64: renamed from C65; footprint smd:SM0603 -> engstad:0402
- C65: renamed from C66; footprint smd:SM0603 -> engstad:0402
- C66: renamed from C67; footprint smd:SM0603 -> engstad:0402
- C67: renamed from C68; footprint smd:SM0603 -> engstad:0402
- C68: renamed from C63; footprint smd:SM0603 -> engstad:0402
- C70: renamed from C76; footprint smd:SM0603 -> engstad:C0603
- C71: renamed from C70; footprint smd:SM0603 -> engstad:C0603
- C72: renamed from C71; footprint smd:SM0603 -> engstad:C0603
- C73: renamed from C72; footprint smd:SM0603 -> engstad:C0603
- C74: renamed from C73; footprint smd:SM0603 -> engstad:C0603
- C75: renamed from C74; footprint smd:SM0603 -> engstad:C0603
- C76: renamed from C75; footprint smd:SM0603 -> engstad:C0603
- L1, L2, L3, L4: footprint (none) -> w_smd_inductors:inductor_smd_0805
- R1, R2, R3, R4, R5, R6, R7: footprint engstad:0603 -> engstad:R0603
- R10: renamed from R9; footprint engstad:0603 -> engstad:R0603
- R11: renamed from R10; footprint engstad:0603 -> engstad:R0603
- R9: renamed from R8; footprint engstad:0603 -> engstad:R0603
Connections:
- net 3.3V is gone; now on net +3V3: R4.2, R5.2, RP1.10 (R7), RP1.11 (R6), RP1.12 (R5), RP1.13 (R4), RP1.14 (R3), RP1.15 (R2), RP1.16 (R1), RP1.9 (R8), U3.E10 (VBATT)
- net VDD is gone; now on net +3V3: C70.2, P7.1 (P1), R10.1, R11.1, R6.1, R7.1, R9.1
- net +3V3: now also U3.B11 (TRST#), R8.1
- net DQ0: now also U3.F10 (GPIO_0/DQ0/MMC_D0/A0)
- net DQ1: now also U3.F9 (GPIO_1/DQ1/MMC_D1/A1)
- net DQ10: now also U3.K11 (GPIO_10/DQ10/A10)
- net DQ11: now also U3.L10 (GPIO_11/DQ11/A11)
- net DQ12: now also U3.K10 (GPIO_12/DQ12/A12)
- net DQ13: now also U3.K9 (GPIO_13/DQ13/A13)
- net DQ14: now also U3.J8 (GPIO_14/DQ14/A14)
- net DQ15: now also U3.G8 (GPIO_15/DQ15/A15)
- net DQ2: now also U3.F7 (GPIO_2/DQ2/MMC_D2/A2)
- net DQ3: now also U3.G10 (GPIO_3/DQ3/MMC_D3/A3)
- net DQ4: now also U3.G9 (GPIO_4/DQ4/MMC_D4/A4)
- net DQ5: now also U3.F8 (GPIO_5/DQ5/MMC_D5/A5)
- net DQ6: now also U3.H10 (GPIO_6/DQ6/MMC_D6/A6)
- net DQ7: now also U3.H9 (GPIO_7/DQ7/A7)
- net DQ8: now also U3.J10 (GPIO_8/DQ8/A8)
- net DQ9: now also U3.J9 (GPIO_9/DQ9/A9)
- net TRST#: no longer U3.B11 (TRST#)
- net UART_CTS: now also P8.2 (P2)
- net UART_RTS: now also P8.1 (P1)
- net UART_RX: now also P8.4 (P4)
- net UART_TX: now also P8.3 (P3)
- net RXVDD: now reaches C49.1, C55.1, L2.2, U3.A2 (U3RXVDDQ)
- net AVDD: now reaches C48.1, C54.1, L1.2, U3.A7 (AVDD)
- net TXVDD: now reaches C50.1, C56.1, L3.2, U3.B5 (U3TXVDDQ)
- net CVDD: now reaches C62.1, C68.1, L4.1, U3.B6 (CVDDQ)
- net RESET#: now reaches U3.C5 (RESET#)
- net RESET#: now also R8.2
- net FPGA-DONE renamed DONE
- net FPGA-INIT-B renamed INIT-B
- net FPGA-PROG-B renamed PROG-B
- net I2C_SCL: no longer names the net of U3.D9 (GPIO_58/I2C_SCL)
- net I2C_SDA: no longer names the net of U3.D10 (GPIO_59/I2C_SDA)
- net TCK renamed FPGA-TCK
- net TDI renamed FPGA-TDI
- net FPGA-TDI: no longer U3.E7 (TDI)
- net TDO renamed EZ-TDO
- net TMS renamed FPGA-TMS
- net VUSB renamed VBUS
- new net FPGA-TDO: U3.E7 (TDI)
- no-connect marks 11 -> 26
Other:
- moved on the sheet: C48, C49, C50, C54, C55, C56, C57, C58, C59, C60, C61, C62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
